Commit message: modified SRDF and controllers

File: src/igus_rebel_description_ros2/urdf/igus_rebel_mod.description.xacro (robot description, xacro)
@@ -97,5 +97,5 @@
 			<parent link="link_3" />
 			<child link="link_4" />
-			<origin rpy="0.0 -1.0 0.0" xyz="-0.035 0.003 0.055"/>
+			<origin rpy="0.0 -1.0 0.0" xyz="-0.035 0.003 0.055" />
 			<dynamics damping="0.0" friction="0.0" />
 		</joint>
@@ -123,5 +123,5 @@
 			<origin rpy="0.0 0 0.0" xyz="0.005 0.015 0.096" />
 			<axis xyz="0 -1 0" />
-			<limit effort="330.0" lower="${-pi*11/18}" upper="${pi*11/18}" velocity="${pi*45/180}"/>
+			<limit effort="330.0" lower="${-pi*11/18}" upper="${pi*11/18}" velocity="${pi*45/180}" />
 			<dynamics damping="0.0" friction="0.0" />
 		</joint>
@@ -149,5 +149,5 @@
 			<origin rpy="-0.05 0.0 0.0" xyz="0.0 -0.025 0.145" />
 			<axis xyz="0 0 1" />
-			<limit effort="330.0" lower="${-pi*179/180}" upper="${pi*179/180}" velocity="${pi*45/180}"/>
+			<limit effort="330.0" lower="${-pi*179/180}" upper="${pi*179/180}" velocity="${pi*45/180}" />
 			<dynamics damping="0.0" friction="0.0" />
 		</joint>
@@ -175,5 +175,5 @@
 			<origin rpy="0.0 0.0 0.0" xyz="0.0 0.029 0.143" />
 			<axis xyz="0 -1 0" />
-			<limit effort="330.0" lower="${-pi*19/36}" upper="${pi*19/36}" velocity="${pi*45/180}"/>
+			<limit effort="330.0" lower="${-pi*19/36}" upper="${pi*19/36}" velocity="${pi*45/180}" />
 			<dynamics damping="0.0" friction="0.0" />
 		</joint>
@@ -201,5 +201,5 @@
 			<origin rpy="0.0 0.0 0.0" xyz="0.0 -0.029 0.11" />
 			<axis xyz="0 0 1" />
-			<limit effort="330.0" lower="${-pi*179/180}" upper="${pi*179/180}" velocity="${pi*45/180}"/>
+			<limit effort="330.0" lower="${-pi*179/180}" upper="${pi*179/180}" velocity="${pi*45/180}" />
 			<dynamics damping="0.0" friction="0.0" />
 		</joint>
@@ -225,5 +225,5 @@
 			<parent link="link_8" />
 			<child link="flange" />
-			<origin rpy="0.0 ${-pi/2} 0.0" xyz="0.0 0 0.0012"/>
+			<origin rpy="0.0 ${-pi/2} 0.0" xyz="0.0 0 0.0012" />
 			<axis xyz="0 0 0" />
 		</joint>
@@ -237,4 +237,8 @@
 		</joint>
 		<link name="tool0">
+			<inertial>
+				<mass value="0.1" />
+				<inertia ixx="0.03" ixy="0.0" ixz="0.0" iyy="0.03" iyz="0.0" izz="0.03" />
+			</inertial>
 		</link>
 	</xacro:macro>
