Commit message: bug fixes and more organized moveit folder

File: src/igus_rebel_description_ros2/urdf/igus_rebel_mod.control.xacro (robot description, xacro)
@@ -31,6 +31,4 @@
 						<param name="max">${pi/4}</param>
 					</command_interface>
-					<!--<command_interface
-					name="effort" />-->
 					<state_interface name="position">
 						<param name="initial_value">0.0</param>
@@ -40,9 +38,4 @@
 						<param name="initial_value">0.0</param>
 					</state_interface>
-					<!--
-					<state_interface name="effort">
-						<param name="initial_value">0.0</param>
-					</state_interface>
-					-->
 					<!-- CRI specific parameters -->
 					<param name="cri_joint_offset">${cri_joint_offset}</param>
@@ -54,5 +47,5 @@
 			<xacro:rebel_joint name="joint3" position_min="${-pi*2/3}" position_max="${pi*2/3}" cri_joint_offset="${-pi/6.0}" />
 			<xacro:rebel_joint name="joint4" position_min="${-pi*179/180}" position_max="${pi*179/180}" />
-			<xacro:rebel_joint name="joint5" position_min="${-pi*19/36}" position_max="${pi*19/36}" cri_joint_offset="0" />
+			<xacro:rebel_joint name="joint5" position_min="${-pi*19/36}" position_max="${pi*19/36}" />
 			<xacro:rebel_joint name="joint6" position_min="${-pi*179/180}" position_max="${pi*179/180}" />
 			<!--

File: src/igus_rebel_description_ros2/urdf/igus_rebel_mod.description.xacro (robot description, xacro)
@@ -22,5 +22,5 @@
 			<child link="link_1" />
 			<origin rpy="0.0 0.0 ${pi}" xyz="0.0 0 0.126" />
-			<axis xyz="0 0 -1" />
+			<axis xyz="0 0 1" />
 			<limit effort="330.0" lower="${-pi*179/180}" upper="${pi*179/180}" velocity="${pi*45/180}" />
 			<dynamics damping="0.0" friction="0.0" />
