Commit message: fixed bugs, added camera and mount URDF visualizations

File: igus_rebel_description_ros2/urdf/igus_rebel.description.xacro (robot description, xacro)
@@ -13,7 +13,4 @@
 				</geometry>
 			</collision>
-			<material name="black">
-				<color rgba="${0/255} ${0/255} ${0/255} 1.0" />
-			</material>
 			<inertial>
 				<mass value="1.0" />
@@ -25,5 +22,5 @@
 			<child link="link_1" />
 			<origin rpy="0.0 0.0 0.0" xyz="0.0 0 0.100" />
-			<axis xyz="0 0 -1" />
+			<axis xyz="0 0 1" />
 			<limit effort="330.0" lower="${-pi*179/180}" upper="${pi*179/180}" velocity="${pi*45/180}" />
 		</joint>
@@ -183,12 +180,4 @@
 		<link name="flange">
 		</link>
-		<joint name="flange_to_tool0" type="fixed">
-			<parent link="flange" />
-			<child link="tool0" />
-			<origin rpy="0.0 0.0 0.0" xyz="0.0 0.0 0.0" />
-			<axis xyz="0 0 0" />
-		</joint>
-		<link name="tool0">
-		</link>
 	</xacro:macro>
 </robot>

File: igus_rebel_description_ros2/urdf/igus_rebel.urdf.xacro (robot description, xacro)
@@ -19,5 +19,5 @@
 	</joint>
 	<!-- Grippers -->
-	<!--<xacro:include filename="$(find igus_rebel_description_ros2)/urdf/grippers/grippers.macro.xacro" />-->
-	<!--<xacro:gripper gripper_type="$(arg gripper)" parent_link="flange" hardware_protocol="$(arg hardware_protocol)" /> -->
+	<xacro:include filename="$(find igus_rebel_description_ros2)/urdf/grippers/grippers.xacro" />
+	<xacro:gripper gripper_type="$(arg gripper)" />
 </robot>
