Commit message: bug fixes, corrected aruco pose follower and xacro descriptions

File: igus_rebel_description_ros2/urdf/igus_rebel.control.xacro (robot description, xacro)
@@ -47,5 +47,5 @@
 			<xacro:rebel_joint name="joint3" position_min="${-pi*2/3}" position_max="${pi*2/3}" cri_joint_offset="${-pi/6.0}" />
 			<xacro:rebel_joint name="joint4" position_min="${-pi*179/180}" position_max="${pi*179/180}" />
-			<xacro:rebel_joint name="joint5" position_min="${-pi*19/36}" position_max="${pi*19/36}" />
+			<xacro:rebel_joint name="joint5" position_min="${-pi*19/36}" position_max="${pi*19/36}" cri_joint_offset="${pi/24.0}" />
 			<xacro:rebel_joint name="joint6" position_min="${-pi*179/180}" position_max="${pi*179/180}" />
 			<!--

File: igus_rebel_description_ros2/urdf/mobile_robot/castle.xacro (robot description, xacro)
@@ -4,5 +4,5 @@
 		<parent link="mobile_robot_base_link" />
 		<child link="tower_link" />
-		<origin rpy="0.0 0.0 0" xyz="0.15 0 0.1" />
+		<origin rpy="0.0 0.0 0" xyz="0.13 0 0.1" />
 		<axis xyz="0 0 -1" />
 	</joint>
@@ -13,7 +13,7 @@
 		</inertial>
 		<visual>
-			<origin xyz="0.0 0 0.3" rpy="0 0 0" />
+			<origin xyz="0.0 0 0.33" rpy="0 0 0" />
 			<geometry>
-				<box size="0.55 0.3 0.65" />
+				<box size="0.55 0.3 0.69" />
 			</geometry>
 			<material name="dark_blue">
@@ -24,5 +24,5 @@
 			<origin xyz="0.0 0 0.3" rpy="0 0 0" />
 			<geometry>
-				<box size="0.55 0.3 0.65" />
+				<box size="0.55 0.3 0.69" />
 			</geometry>
 		</collision>
