Commit message: xacro macro for SRDF definition and correct collision checking

File: igus_rebel_description_ros2/urdf/mobile_robot/scout_wheel_type1.xacro (robot description, xacro)
@@ -26,5 +26,5 @@
 			</collision>
 		</link>
-		<joint name="${wheel_prefix}_wheel" type="continuous">
+		<joint name="${wheel_prefix}_wheel" type="fixed">
 			<parent link="mobile_robot_base_link" />
 			<child link="${wheel_prefix}_wheel_link" />

File: igus_rebel_description_ros2/urdf/mobile_robot/scout_wheel_type2.xacro (robot description, xacro)
@@ -26,5 +26,5 @@
 			</collision>
 		</link>
-		<joint name="${wheel_prefix}_wheel" type="continuous">
+		<joint name="${wheel_prefix}_wheel" type="fixed">
 			<parent link="mobile_robot_base_link" />
 			<child link="${wheel_prefix}_wheel_link" />
