Commit message: corrected srdf xacro for collision bugs

File: igus_rebel_description_ros2/urdf/mobile_robot/castle.xacro (robot description, xacro)
@@ -4,5 +4,5 @@
 		<parent link="mobile_robot_base_link" />
 		<child link="tower_link" />
-		<origin rpy="0.0 0.0 0" xyz="0.13 0 0.1" />
+		<origin rpy="0.0 0.0 0" xyz="0.13 0.0 0.1" />
 		<axis xyz="0 0 -1" />
 	</joint>
@@ -13,5 +13,5 @@
 		</inertial>
 		<visual>
-			<origin xyz="0.0 0 0.33" rpy="0 0 0" />
+			<origin xyz="0.0 0.0 0.33" rpy="0.0 0.0 0.0" />
 			<geometry>
 				<box size="0.55 0.3 0.69" />
@@ -22,5 +22,5 @@
 		</visual>
 		<collision>
-			<origin xyz="0.0 0 0.3" rpy="0 0 0" />
+			<origin xyz="0.0 0.0 0.33" rpy="0.0 0.0 0.0" />
 			<geometry>
 				<box size="0.55 0.3 0.69" />

File: igus_rebel_description_ros2/urdf/mobile_robot/scout_v2.xacro (robot description, xacro)
@@ -61,5 +61,5 @@
 	<link name="front_mount" />
 	<joint name="front_mount_joint" type="fixed">
-		<origin xyz="0.325 0 0.112701" rpy="0 0 0" />
+		<origin xyz="0.325 0.0 0.112701" rpy="0 0 0" />
 		<parent link="mobile_robot_base_link" />
 		<child link="front_mount" />
@@ -67,5 +67,5 @@
 	<link name="rear_mount" />
 	<joint name="rear_mount_joint" type="fixed">
-		<origin xyz="-0.325 0 0.112701" rpy="0 0 0" />
+		<origin xyz="-0.325 0.0 0.112701" rpy="0 0 0" />
 		<parent link="mobile_robot_base_link" />
 		<child link="rear_mount" />

File: igus_rebel_moveit_config/config/igus_rebel.srdf.xacro (robot description, xacro)
@@ -9,6 +9,4 @@
 		<disable_collisions link1="${link}" link2="rear_right_wheel_link" reason="Never" />
 		<disable_collisions link1="${link}" link2="rear_left_wheel_link" reason="Never" />
-		<disable_collisions link1="${link}" link2="front_mount" reason="Never" />
-		<disable_collisions link1="${link}" link2="rear_mount" reason="Never" />
 	</xacro:macro>
 	<!-- disable collision between a link and the camera links-->
@@ -16,7 +14,5 @@
 		<disable_collisions link1="${link}" link2="camera_link" reason="Never" />
 		<disable_collisions link1="${link}" link2="camera_mount" reason="Never" />
-		<disable_collisions link1="${link}" link2="camera_insert" reason="Never" />
 		<disable_collisions link1="${link}" link2="toucher" reason="Never" />
-		<disable_collisions link1="${link}" link2="flange" reason="Never" />
 		<disable_collisions link1="${link}" link2="camera_usb_plug_link" reason="Never" />
 	</xacro:macro>
@@ -57,5 +53,5 @@
 			</group>
 			<end_effector name="manipulator" parent_link="toucher" group="chain_arm_manipulator"
-				parent_group="rebel_arm_manipulator" />
+				parent_group="camera" />
 		</xacro:if>
 		<!-- default positions common for every configuration -->
@@ -76,4 +72,20 @@
 			<joint name="joint6" value="0" />
 		</group_state>
+		<group_state name="zero" group="chain_arm_manipulator">
+			<joint name="joint1" value="0" />
+			<joint name="joint2" value="0" />
+			<joint name="joint3" value="0" />
+			<joint name="joint4" value="0" />
+			<joint name="joint5" value="0" />
+			<joint name="joint6" value="0" />
+		</group_state>
+		<group_state name="home" group="chain_arm_manipulator">
+			<joint name="joint1" value="0" />
+			<joint name="joint2" value="${-pi/6.0}" />
+			<joint name="joint3" value="${-pi/6.0}" />
+			<joint name="joint4" value="0" />
+			<joint name="joint5" value="${pi/24.0}" />
+			<joint name="joint6" value="0" />
+		</group_state>
 		<!--TODO:
 		add parking position -->
@@ -81,4 +93,5 @@
 		<!-- default collision checks for base robot -->
 		<disable_collisions link1="base_link" link2="link_1" reason="Adjacent" />
+		<disable_collisions link1="base_link" link2="link_2" reason="Never" />
 		<disable_collisions link1="link_1" link2="link_2" reason="Adjacent" />
 		<disable_collisions link1="link_2" link2="link_5" reason="Adjacent" />
@@ -94,19 +107,10 @@
 		<!-- additional collision checks due to the presence of the camera mount -->
 		<xacro:if value="${gripper == 'camera'}">
-			<disable_collisions link1="link_8" link2="flange" reason="Adjacent" />
-			<disable_collisions link1="link_8" link2="camera_mount" reason="Never" />
-			<disable_collisions link1="link_8" link2="camera_insert" reason="Never" />
-			<disable_collisions link1="link_8" link2="toucher" reason="Adjacent" />
-			<disable_collisions link1="flange" link2="camera_mount" reason="Adjacent" />
-			<disable_collisions link1="flange" link2="toucher" reason="Adjacent" />
-			<disable_collisions link1="flange" link2="camera_insert" reason="Never" />
-			<disable_collisions link1="flange" link2="camera_link" reason="Never" />
+			<disable_collisions link1="camera_link" link2="camera_mount" reason="Adjacent" />
+			<disable_collisions link1="camera_link" link2="camera_usb_plug_link" reason="Adjacent" />
+			<disable_collisions link1="camera_mount" link2="camera_usb_plug_link" reason="Never" />
+			<disable_collisions link1="camera_link" link2="toucher" reason="Never" />
 			<disable_collisions link1="camera_mount" link2="toucher" reason="Never" />
-			<disable_collisions link1="camera_mount" link2="camera_insert" reason="Adjacent" />
-			<disable_collisions link1="camera_insert" link2="toucher" reason="Never" />
-			<disable_collisions link1="camera_link" link2="camera_usb_plug_link" reason="Adjacent" />
-			<disable_collisions link1="camera_link" link2="camera_insert" reason="Adjacent" />
-			<disable_collisions link1="camera_link" link2="camera_mount" reason="Adjacent" />
-			<disable_collisions link1="camera_link" link2="toucher" reason="Never" />
+			<xacro:no_collision_camera link="base_link" />
 			<xacro:no_collision_camera link="link_1" />
 			<xacro:no_collision_camera link="link_2" />
@@ -114,34 +118,54 @@
 			<xacro:no_collision_camera link="link_6" />
 			<xacro:no_collision_camera link="link_7" />
+			<xacro:no_collision_camera link="link_8" />
 		</xacro:if>
 		<!-- when the robot scout is loaded define the collision checks -->
 		<xacro:if value="${load_base}">
-			<disable_collision link1="base_link" link2="mobile_robot_base_link" reason="Adjacent" />
-			<disable_collision link1="base_link" link2="inertial_link" reason="Adjacent" />
-			<disable_collision link1="base_link" link2="rebel_support" reason="Adjacent" />
-			<disable_collision link1="base_link" link2="front_mount" reason="Adjacent" />
-			<disable_collision link1="base_link" link2="rear_mount" reason="Adjacent" />
-			<disable_collision link1="base_link" link2="tower_link" reason="Never" />
-			<disable_collision link1="mobile_robot_base_link" link2="inertial_link" reason="Adjacent" />
-			<disable_collision link1="mobile_robot_base_link" link2="front_mount" reason="Adjacent" />
-			<disable_collision link1="mobile_robot_base_link" link2="rear_mount" reason="Adjacent" />
-			<disable_collision link1="mobile_robot_base_link" link2="rebel_support" reason="Adjacent" />
-			<disable_collision link1="mobile_robot_base_link" link2="front_right_wheel_link" reason="Adjacent" />
-			<disable_collision link1="mobile_robot_base_link" link2="front_left_wheel_link" reason="Adjacent" />
-			<disable_collision link1="mobile_robot_base_link" link2="rear_right_wheel_link" reason="Adjacent" />
-			<disable_collision link1="mobile_robot_base_link" link2="rear_left_wheel_link" reason="Adjacent" />
-			<disable_collision link1="mobile_robot_base_link" link2="tower_link" reason="Adjacent" />
-			<xacro:no_collision_scout link="link_1" />
-			<xacro:no_collision_scout link="link_2" />
-			<xacro:no_collision_scout link="link_5" />
-			<xacro:no_collision_scout link="link_6" />
-			<xacro:no_collision_scout link="link_7" />
-			<xacro:no_collision_scout link="link_8" />
-			<xacro:no_collision_scout link="flange" />
-			<xacro:no_collision_scout link="camera_mount" />
-			<xacro:no_collision_scout link="camera_insert" />
-			<xacro:no_collision_scout link="toucher" />
-			<xacro:no_collision_scout link="camera_link" />
-			<xacro:no_collision_scout link="camera_usb_plug_link" />
+			<group name="mobile_robot">
+				<link name="mobile_robot_base_link" />
+				<link name="front_right_wheel_link" />
+				<link name="front_left_wheel_link" />
+				<link name="rear_right_wheel_link" />
+				<link name="rear_left_wheel_link" />
+				<link name="inertial_link" />
+				<link name="front_mount" />
+				<link name="rear_mount" />
+				<link name="rebel_support" />
+				<link name="tower_link" />
+			</group>
+			<disable_collisions link1="base_link" link2="front_left_wheel_link" reason="Never" />
+			<disable_collisions link1="base_link" link2="front_right_wheel_link" reason="Never" />
+			<disable_collisions link1="base_link" link2="mobile_robot_base_link" reason="Adjacent" />
+			<disable_collisions link1="base_link" link2="rear_left_wheel_link" reason="Never" />
+			<disable_collisions link1="base_link" link2="rear_right_wheel_link" reason="Never" />
+			<disable_collisions link1="base_link" link2="tower_link" reason="Never" />
+			<disable_collisions link1="front_left_wheel_link" link2="front_right_wheel_link" reason="Never" />
+			<disable_collisions link1="front_left_wheel_link" link2="link_1" reason="Never" />
+			<disable_collisions link1="front_left_wheel_link" link2="link_2" reason="Never" />
+			<disable_collisions link1="front_left_wheel_link" link2="link_5" reason="Never" />
+			<disable_collisions link1="front_left_wheel_link" link2="mobile_robot_base_link" reason="Adjacent" />
+			<disable_collisions link1="front_left_wheel_link" link2="rear_left_wheel_link" reason="Never" />
+			<disable_collisions link1="front_left_wheel_link" link2="rear_right_wheel_link" reason="Never" />
+			<disable_collisions link1="front_left_wheel_link" link2="tower_link" reason="Never" />
+			<disable_collisions link1="front_right_wheel_link" link2="link_1" reason="Never" />
+			<disable_collisions link1="front_right_wheel_link" link2="link_2" reason="Never" />
+			<disable_collisions link1="front_right_wheel_link" link2="link_5" reason="Never" />
+			<disable_collisions link1="front_right_wheel_link" link2="mobile_robot_base_link" reason="Adjacent" />
+			<disable_collisions link1="front_right_wheel_link" link2="rear_left_wheel_link" reason="Never" />
+			<disable_collisions link1="front_right_wheel_link" link2="rear_right_wheel_link" reason="Never" />
+			<disable_collisions link1="front_right_wheel_link" link2="tower_link" reason="Never" />
+			<disable_collisions link1="link_1" link2="mobile_robot_base_link" reason="Never" />
+			<disable_collisions link1="link_1" link2="rear_left_wheel_link" reason="Never" />
+			<disable_collisions link1="link_1" link2="rear_right_wheel_link" reason="Never" />
+			<disable_collisions link1="link_1" link2="tower_link" reason="Never" />
+			<disable_collisions link1="link_2" link2="mobile_robot_base_link" reason="Never" />
+			<disable_collisions link1="link_2" link2="rear_left_wheel_link" reason="Never" />
+			<disable_collisions link1="link_2" link2="rear_right_wheel_link" reason="Never" />
+			<disable_collisions link1="mobile_robot_base_link" link2="rear_left_wheel_link" reason="Adjacent" />
+			<disable_collisions link1="mobile_robot_base_link" link2="rear_right_wheel_link" reason="Adjacent" />
+			<disable_collisions link1="mobile_robot_base_link" link2="tower_link" reason="Adjacent" />
+			<disable_collisions link1="rear_left_wheel_link" link2="rear_right_wheel_link" reason="Never" />
+			<disable_collisions link1="rear_left_wheel_link" link2="tower_link" reason="Never" />
+			<disable_collisions link1="rear_right_wheel_link" link2="tower_link" reason="Never" />
 		</xacro:if>
 	</xacro:macro>
