Commit message: created searching movement and updated castle definition

File: igus_rebel_description_ros2/urdf/mobile_robot/castle.urdf (robot description, URDF)
Before this commit: robot scout_v2, 1 links, 1 joints
Links:
- link tower_link: geometry collision box size=0.17 0.28 0.2; collision box size=0.38 0.28 0.69
Joints:
- joint tower: origin xyz=0.13 0.0 0.1 rpy=0.0 0.0 0 -> xyz=0.0 0.0 0.1 rpy=0.0 0.0 0

File: igus_rebel_description_ros2/urdf/robot.urdf.xacro (robot description, xacro)
@@ -21,5 +21,5 @@
 			<parent link="base_link" />
 			<child link="rebel_support" />
-			<origin xyz="-0.26 0.0 0.1" rpy="0 0 ${pi}" />
+			<origin xyz="-0.27 0.0 0.135" rpy="0 0 ${pi}" />
 		</joint>
 		<link name="rebel_support" />

Commit message: updated robot setup with new batteries

File: igus_rebel_description_ros2/urdf/mobile_robot/castle.urdf (robot description, URDF)
Before this commit: robot scout_v2, 1 links, 1 joints
Links:
- link tower_link: geometry collision box size=0.18 0.28 0.2; collision box size=0.38 0.28 0.69

File: igus_rebel_description_ros2/urdf/robot.urdf.xacro (robot description, xacro)
@@ -47,5 +47,5 @@
 			<parent link="base_link" />
 			<child link="rebel_support" />
-			<origin xyz="-0.27 0.0 0.135" rpy="0 0 ${pi}" />
+			<origin xyz="-0.28 0.0 0.135" rpy="0 0 ${pi}" />
 		</joint>
 		<link name="rebel_support" />

Commit message: fixes and adjustments

File: igus_rebel_description_ros2/urdf/mobile_robot/castle.urdf (robot description, URDF)
Before this commit: robot scout_v2, 1 links, 1 joints
Links:
- link tower_link: geometry collision box size=0.18 0.32 0.22; collision box size=0.38 0.32 0.69

File: igus_rebel_moveit_config/config/igus_rebel.srdf.xacro (robot description, xacro)
@@ -73,8 +73,8 @@
 			<joint name="joint1" value="${-42.0 * pi / 180.0}" />
 			<joint name="joint2" value="${70.0 * pi / 180.0}" />
-			<joint name="joint3" value="${103.0 * pi / 180.0}" />
+			<joint name="joint3" value="${102.0 * pi / 180.0}" />
 			<joint name="joint4" value="${82.0 * pi / 180.0}" />
-			<joint name="joint5" value="${-86.0 * pi / 180.0}" />
-			<joint name="joint6" value="${-95.0 * pi / 180.0}" />
+			<joint name="joint5" value="${-90.0 * pi / 180.0}" />
+			<joint name="joint6" value="${-90.0 * pi / 180.0}" />
 		</group_state>
 		<group_state name="stand" group="rebel_arm">

Commit message: few corrections and adjustments

File: igus_rebel_description_ros2/urdf/mobile_robot/castle.urdf (robot description, URDF)
Before this commit: robot scout_v2, 1 links, 1 joints
Links:
- link tower_link: geometry collision box size=0.18 0.32 0.21; collision box size=0.38 0.32 0.69

File: igus_rebel_moveit_config/config/igus_rebel.srdf.xacro (robot description, xacro)
@@ -81,7 +81,7 @@
 			<joint name="joint1" value="${61.0 * pi / 180.0}" />
 			<joint name="joint2" value="${-60.0 * pi / 180.0}" />
-			<joint name="joint3" value="${66.0 * pi / 180.0}" />
+			<joint name="joint3" value="${72.0 * pi / 180.0}" />
 			<joint name="joint4" value="0" />
-			<joint name="joint5" value="${87.0 * pi / 180.0}" />
+			<joint name="joint5" value="${90.0 * pi / 180.0}" />
 			<joint name="joint6" value="${5.0 * pi / 180.0}" />
 		</group_state>

Commit message: added basket to mobile robot

File: igus_rebel_description_ros2/urdf/mobile_robot/castle.urdf (robot description, URDF)
Before this commit: robot scout_v2, 1 links, 1 joints
Links:
- removed link tower_link
Joints:
- removed joint tower

File: igus_rebel_description_ros2/urdf/robot.urdf.xacro (robot description, xacro)
@@ -37,4 +37,5 @@
 		to mobile_robot_base_link-->
 		<xacro:include filename="$(find igus_rebel_description_ros2)/urdf/mobile_robot/castle.urdf" />
+		<xacro:castle with_basket="true" />
 		<!-- load scout robot -->
 		<xacro:include
