Commit message: bug fixes, added SRDF definition for robot + camera

File: igus_rebel_description_ros2/urdf/grippers/grippers.xacro (robot description, xacro)
@@ -37,12 +37,19 @@
 				</collision>
 			</link>
+			<joint name="flange_to_toucher" type="fixed">
+				<parent link="flange" />
+				<child link="toucher" />
+				<origin rpy="0.0 0.0 0.0" xyz="0.1 0.0 0.0" /> <!-- 10 cm in front of the flange origin -->
+				<axis xyz="0 0 0" />
+			</joint>
+			<link name="toucher" />
 			<!-- positions the camera inside the structure -->
 			<joint name="mount_to_cam" type="fixed">
 				<parent link="camera_mount" />
 				<child link="camera_insert" />
-				<origin rpy="0.0 0.0 0.0" xyz="0.04 0.0 0.065" />
+				<origin rpy="0.0 0.0 0.0" xyz="0.038 0.0 0.065" />
 				<axis xyz="0 0 0" />
 			</joint>
-			<link name="camera_insert"/>
+			<link name="camera_insert" />
 			<!-- includes the realsense D435 ros2 description file and its collision box-->
 			<xacro:arg name="use_nominal_extrinsics" default="false" />

File: igus_rebel_description_ros2/urdf/igus_rebel.control.xacro (robot description, xacro)
@@ -1,6 +1,6 @@
 <?xml version="1.0"?>
-<robot xmlns:xacro="http://www.ros.org/wiki/xacro" name="igus_rebel_mod">
-	<xacro:macro name="igus_rebel_mod_control" params="hardware_protocol">
-		<ros2_control name="igus_rebel_mod" type="system">
+<robot xmlns:xacro="http://www.ros.org/wiki/xacro" name="igus_rebel">
+	<xacro:macro name="igus_rebel_control" params="hardware_protocol">
+		<ros2_control name="igus_rebel" type="system">
 			<hardware>
 				<xacro:if value="${hardware_protocol == 'mock_hardware'}">

File: igus_rebel_description_ros2/urdf/igus_rebel.urdf.xacro (robot description, xacro)
@@ -9,6 +9,6 @@
 	<xacro:igus_rebel_description  />
 	<!-- controller macro -->
-	<xacro:include filename="$(find igus_rebel_description_ros2)/urdf/igus_rebel_mod.control.xacro" />
-	<xacro:igus_rebel_mod_control hardware_protocol="$(arg hardware_protocol)"/>
+	<xacro:include filename="$(find igus_rebel_description_ros2)/urdf/igus_rebel.control.xacro" />
+	<xacro:igus_rebel_control hardware_protocol="$(arg hardware_protocol)"/>
 	<!-- Add world link -->
 	<link name="world" />

File: igus_rebel_description_ros2/urdf/igus_rebel_mod.urdf.xacro (robot description, xacro)
@@ -9,6 +9,6 @@
 	<xacro:igus_rebel_mod_description hardware_protocol="$(arg hardware_protocol)" />
 	<!-- controller macro -->
-	<xacro:include filename="$(find igus_rebel_description_ros2)/urdf/igus_rebel_mod.control.xacro" />
-	<xacro:igus_rebel_mod_control hardware_protocol="$(arg hardware_protocol)"/>
+	<xacro:include filename="$(find igus_rebel_description_ros2)/urdf/igus_rebel.control.xacro" />
+	<xacro:igus_rebel_control hardware_protocol="$(arg hardware_protocol)"/>
 	<!-- Add world link -->
 	<link name="world" />

File: igus_rebel_moveit_config/config/igus_rebel.urdf.xacro (robot description, xacro)
@@ -1,23 +1,5 @@
 <?xml version="1.0"?>
 <robot xmlns:xacro="http://www.ros.org/wiki/xacro" name="igus_rebel">
-	<!-- Controller settings, only enable a single one in the launch file -->
-	<xacro:arg name="hardware_protocol" default="cri" />
-	<!-- Gripper selection -->
-	<xacro:arg name="gripper" default="none" />
-	<!-- Include and call rebel macro -->
-	<xacro:include filename="$(find igus_rebel_description_ros2)/urdf/igus_rebel.description.xacro" />
-	<xacro:igus_rebel_description />
-	<!-- controller macro -->
-	<xacro:include filename="$(find igus_rebel_description_ros2)/urdf/igus_rebel_mod.control.xacro" />
-	<xacro:igus_rebel_mod_control hardware_protocol="$(arg hardware_protocol)"/>
-	<!-- Add world link -->
-	<link name="world" />
-	<joint name="world_to_base" type="fixed">
-		<parent link="world" />
-		<child link="base_link" />
-		<origin xyz="0.0 0.0 0.0" rpy="0.0 0.0 0.0" />
-	</joint>
-	<!-- Grippers -->
-	<!--<xacro:include filename="$(find igus_rebel_description_ros2)/urdf/grippers/grippers.macro.xacro" />-->
-	<!--<xacro:gripper gripper_type="$(arg gripper)" parent_link="flange" hardware_protocol="$(arg hardware_protocol)" /> -->
+	<!-- include igus_rebel.urdf.xacro from the description package -->
+	<xacro:include filename="$(find igus_rebel_description_ros2)/urdf/igus_rebel.urdf.xacro" />
 </robot>

Commit message: modified base end effector

File: igus_rebel_description_ros2/urdf/grippers/grippers.xacro (robot description, xacro)
@@ -39,9 +39,37 @@
 			<joint name="flange_to_toucher" type="fixed">
 				<parent link="flange" />
-				<child link="toucher" />
-				<origin rpy="0.0 0.0 0.0" xyz="0.1 0.0 0.0" /> <!-- 10 cm in front of the flange origin -->
+				<child link="toucher_cylinder" />
+				<origin rpy="0.0 0.0 0.0" xyz="0.0 0.0 0.0" />
 				<axis xyz="0 0 0" />
 			</joint>
-			<link name="toucher" />
+			<!-- toucher is a cylindrical approximation of the pointer for touching objects -->
+			<!-- 22.5 cm = length of cylinder -->
+			<link name="toucher_cylinder">
+				<inertial>
+					<origin xyz="0.1125 0.0 0.0" rpy="0.0 ${pi/2.0} 0.0" />
+					<mass value="0.1" />
+					<inertia ixx="0.0001" iyy="0.0001" izz="0.0001" ixy="0" iyz="0" ixz="0" />
+				</inertial>
+				<visual>
+					<origin xyz="0.1125 0.0 0.0" rpy="0.0 ${pi/2.0} 0.0" />
+					<geometry>
+						<cylinder length="0.225" radius="0.015" />
+					</geometry>
+					<material name="dark_green" />
+				</visual>
+				<collision>
+					<origin xyz="0.1125 0.0 0.0" rpy="0.0 ${pi/2.0} 0.0" />
+					<geometry>
+						<cylinder length="0.225" radius="0.015" />
+					</geometry>
+				</collision>
+			</link>
+			<joint name="flange_to_point" type="fixed">
+				<parent link="flange" />
+				<child link="tip_link" />
+				<origin xyz="0.225 0.0 0.0" rpy="0.0 0.0 0.0" />
+				<axis xyz="0.0 0.0 0.0" />
+			</joint>
+			<link name="tip_link" />
 			<!-- positions the camera inside the structure -->
 			<joint name="mount_to_cam" type="fixed">
@@ -49,5 +77,5 @@
 				<child link="camera_insert" />
 				<origin rpy="0.0 0.0 0.0" xyz="0.038 0.0 0.065" />
-				<axis xyz="0 0 0" />
+				<axis xyz="0.0 0.0 0.0" />
 			</joint>
 			<link name="camera_insert" />

File: igus_rebel_moveit_config/config/igus_rebel.srdf.xacro (robot description, xacro)
@@ -30,5 +30,5 @@
 		<disable_collisions link1="${link}" link2="camera_link" reason="Never" />
 		<disable_collisions link1="${link}" link2="camera_mount" reason="Never" />
-		<disable_collisions link1="${link}" link2="toucher" reason="Never" />
+		<disable_collisions link1="${link}" link2="toucher_cylinder" reason="Never" />
 		<disable_collisions link1="${link}" link2="camera_usb_plug_link" reason="Never" />
 	</xacro:macro>
@@ -72,5 +72,5 @@
 			</group_state>
 		</xacro:if>
-		<!-- if camera is placed => end effector on toucher link -->
+		<!-- if camera is placed => end effector on tip_link link -->
 		<xacro:if value="${gripper == 'camera'}">
 			<group name="camera">
@@ -78,10 +78,11 @@
 				<link name="camera_mount" />
 				<link name="camera_usb_plug_link" />
-				<link name="toucher" />
+				<link name="toucher_cylinder" />
+                <link name="tip_link" />
 			</group>
 			<group name="chain_arm_manipulator">
-				<chain base_link="igus_rebel_base_link" tip_link="toucher" />
+				<chain base_link="igus_rebel_base_link" tip_link="tip_link" />
 			</group>
-			<end_effector name="manipulator" parent_link="toucher" group="chain_arm_manipulator" parent_group="camera" />
+			<end_effector name="manipulator" parent_link="tip_link" group="chain_arm_manipulator" parent_group="camera" />
 			<group_state name="zero" group="chain_arm_manipulator">
 				<joint name="joint1" value="0" />
@@ -125,6 +126,7 @@
 			<disable_collisions link1="camera_link" link2="camera_usb_plug_link" reason="Adjacent" />
 			<disable_collisions link1="camera_mount" link2="camera_usb_plug_link" reason="Never" />
-			<disable_collisions link1="camera_link" link2="toucher" reason="Never" />
-			<disable_collisions link1="camera_mount" link2="toucher" reason="Never" />
+			<disable_collisions link1="camera_link" link2="toucher_cylinder" reason="Never" />
+			<disable_collisions link1="camera_mount" link2="toucher_cylinder" reason="Never" />
+            <disable_collisions link1="toucher_cylinder" link2="tip_link" reason="Adjacent" />
 			<xacro:no_collision_camera link="igus_rebel_base_link" />
 			<xacro:no_collision_camera link="link_1" />

Commit message: new toucher definition

File: igus_rebel_description_ros2/urdf/grippers/grippers.xacro (robot description, xacro)
@@ -44,22 +44,22 @@
 			</joint>
 			<!-- toucher is a cylindrical approximation of the pointer for touching objects -->
-			<!-- 22.5 cm = length of cylinder -->
+			<!-- 11 cm = length of cylinder -->
 			<link name="toucher_cylinder">
 				<inertial>
-					<origin xyz="0.1125 0.0 0.0" rpy="0.0 ${pi/2.0} 0.0" />
+					<origin xyz="0.055 0.0 0.0" rpy="0.0 ${pi/2.0} 0.0" />
 					<mass value="0.1" />
 					<inertia ixx="0.0001" iyy="0.0001" izz="0.0001" ixy="0" iyz="0" ixz="0" />
 				</inertial>
 				<visual>
-					<origin xyz="0.1125 0.0 0.0" rpy="0.0 ${pi/2.0} 0.0" />
+					<origin xyz="0.055 0.0 0.0" rpy="0.0 ${pi/2.0} 0.0" />
 					<geometry>
-						<cylinder length="0.225" radius="0.015" />
+						<cylinder length="0.11" radius="0.015" />
 					</geometry>
 					<material name="dark_green" />
 				</visual>
 				<collision>
-					<origin xyz="0.1125 0.0 0.0" rpy="0.0 ${pi/2.0} 0.0" />
+					<origin xyz="0.055 0.0 0.0" rpy="0.0 ${pi/2.0} 0.0" />
 					<geometry>
-						<cylinder length="0.225" radius="0.015" />
+						<cylinder length="0.11" radius="0.015" />
 					</geometry>
 				</collision>
@@ -68,5 +68,5 @@
 				<parent link="flange" />
 				<child link="tip_link" />
-				<origin xyz="0.225 0.0 0.0" rpy="0.0 0.0 0.0" />
+				<origin xyz="0.11 0.0 0.0" rpy="0.0 0.0 0.0" />
 				<axis xyz="0.0 0.0 0.0" />
 			</joint>

File: igus_rebel_description_ros2/urdf/robot.urdf.xacro (robot description, xacro)
@@ -34,5 +34,5 @@
 		<!-- load scout robot -->
 		<xacro:include
-			filename="$(find agilex_scout)/urdf/mobile_robot/scout_v2.xacro" />
+			filename="$(find agilex_scout)/urdf/mobile_robot/scout_v2.urdf.xacro" />
 		<xacro:scout_v2
 			load_gazebo="$(arg load_gazebo)" odometry_source="$(arg odometry_source)" />
