Commit message: added support for new mount and end effector

File: igus_rebel_description_ros2/urdf/end_effectors/soft_gripper.control.xacro (robot description, xacro)
@@ -2,9 +2,13 @@
 <robot xmlns:xacro="http://www.ros.org/wiki/xacro" name="igus_rebel">
 	<xacro:macro name="igus_rebel_gripper" params="use_dummy">
+		<!-- Set use_dummy to true to connect to a dummy driver for testing purposes. -->
+		<xacro:property name="baud_rate" value="115200"/>
+		<xacro:property name="serial_port" value="/dev/ttyUSB0"/>
 		<ros2_control name="igus_rebel_gripper_control" type="actuator">
 			<hardware>
-				<plugin>igus_rebel_gripper_controller/GripperController</plugin>
-				<!-- Set use_dummy to true to connect to a dummy driver for testing purposes. -->
+				<plugin>soft_gripper_controller/GripperController</plugin>
 				<param name="use_dummy">${use_dummy}</param>
+				<param name="baud_rate">${baud_rate}</param>
+				<param name="serial_port">${serial_port}</param>
 			</hardware>
 			<gpio name="soft_gripper_gpio">

File: igus_rebel_description_ros2/urdf/end_effectors/soft_gripper.description.xacro (robot description, xacro)
@@ -1,5 +1,4 @@
 <?xml version="1.0"?>
 <robot xmlns:xacro="http://www.ros.org/wiki/xacro" name="igus_rebel">
-	<xacro:arg name="use_dummy" default="false" />
 	<!-- TODO: add meshes, mount v2 and end effector tip link for the Soft gripper -->
 	<joint name="soft_gripper_joint" type="fixed">
@@ -29,7 +28,3 @@
 		</inertial>
 	</link>
-	<!-- Import gripper ros2_control description -->
-	<xacro:include
-		filename="$(find igus_rebel_description_ros2)/urdf/end_effectors/soft_gripper.control.xacro" />
-	<xacro:igus_rebel_control use_dummy="$(arg use_dummy)" />
 </robot>

File: igus_rebel_description_ros2/urdf/igus_rebel/igus_rebel.urdf.xacro (robot description, xacro)
@@ -12,10 +12,16 @@
 			filename="$(find igus_rebel_description_ros2)/urdf/igus_rebel/igus_rebel.control.xacro" />
 		<xacro:igus_rebel_control hardware_protocol="${hardware_protocol}" />
-		<!-- Mount macro -->
+		<!-- Mount macros -->
 		<xacro:if value="${mount == 'mount_v1'}">
 			<xacro:include filename="$(find igus_rebel_description_ros2)/urdf/mounts/mount_v1.xacro" />
-			<xacro:mount_v1 camera="$(arg camera)" end_effector="$(arg end_effector)"
-				load_gazebo="$(arg load_gazebo)" />
+			<xacro:mount_v1 end_effector="$(arg end_effector)" />
 		</xacro:if>
+		<xacro:if value="${mount == 'mount_v2'}">
+			<xacro:include filename="$(find igus_rebel_description_ros2)/urdf/mounts/mount_v2.xacro" />
+			<xacro:mount_v2 end_effector="$(arg end_effector)" />
+		</xacro:if>
+		<!-- Camera macro -->
+		<xacro:include filename="$(find igus_rebel_description_ros2)/urdf/cameras/cameras.urdf.xacro" />
+		<xacro:cameras camera="${camera}" load_gazebo="${load_gazebo}" />
 		<!-- Gazebo macro -->
 		<xacro:if value="${load_gazebo}">

File: igus_rebel_description_ros2/urdf/mounts/mount_v2.xacro (robot description, xacro)
@@ -1,8 +1,8 @@
 <?xml version="1.0"?>
-<robot xmlns:xacro="http://www.ros.org/wiki/xacro" name="mount_v1">
-	<material name="mount_dark_green">
-		<color rgba="${5/255.0} ${100/255.0} ${5/255.0} 1.000" />
+<robot xmlns:xacro="http://www.ros.org/wiki/xacro" name="mount_v2">
+	<material name="mount_dark_grey">
+		<color rgba="${12/255.0} ${12/255.0} ${12/255.0} 1.000" />
 	</material>
-	<xacro:macro name="mount_v1" params="end_effector">
+	<xacro:macro name="mount_v2" params="end_effector">
 		<!-- links the flange on the last joint to the mount_v1 -->
 		<joint name="flange_to_mount" type="fixed">
@@ -26,5 +26,5 @@
 				<geometry>
 					<mesh
-						filename="file://$(find igus_rebel_description_ros2)/meshes/mounts/mount_v1.stl"
+						filename="file://$(find igus_rebel_description_ros2)/meshes/mounts/mount_v2.stl"
 						scale="0.001 0.001 0.001" />
 				</geometry>
@@ -35,5 +35,5 @@
 				<geometry>
 					<mesh
-						filename="file://$(find igus_rebel_description_ros2)/meshes/mounts/mount_v1.stl"
+						filename="file://$(find igus_rebel_description_ros2)/meshes/mounts/mount_v2.stl"
 						scale="0.001 0.001 0.001" />
 				</geometry>
@@ -49,8 +49,12 @@
 		<link name="camera_insert" />
 		<!-- End effectors -->
-		<xacro:if value="${end_effector == 'toucher_v1'}">
+		<xacro:if value="${end_effector == 'soft_gripper'}">
+            <!-- description urdf of the soft gripper -->
 			<xacro:include
-				filename="$(find igus_rebel_description_ros2)/urdf/end_effectors/toucher_v1.xacro" />
-			<xacro:toucher_v1 parent="flange" />
+				filename="$(find igus_rebel_description_ros2)/urdf/end_effectors/soft_gripper.description.xacro" />
+            <!-- ros2 control of the soft gripper actuator -->
+            <xacro:include
+                filename="$(find igus_rebel_description_ros2)/urdf/end_effectors/soft_gripper.control.xacro" />
+            <xacro:igus_rebel_gripper use_dummy="false" />
 		</xacro:if>
 	</xacro:macro>

Commit message: working soft gripper hardware interface using ROS2-control

File: igus_rebel_description_ros2/urdf/end_effectors/soft_gripper.control.xacro (robot description, xacro)
@@ -4,8 +4,8 @@
 		<!-- Set use_dummy to true to connect to a dummy driver for testing purposes. -->
 		<xacro:property name="baud_rate" value="115200"/>
-		<xacro:property name="serial_port" value="/dev/ttyUSB0"/>
+		<xacro:property name="serial_port" value="/dev/ttyACM0"/>
 		<ros2_control name="igus_rebel_gripper_control" type="actuator">
 			<hardware>
-				<plugin>soft_gripper_controller/GripperController</plugin>
+				<plugin>igus_rebel_gripper_controller/GripperController</plugin>
 				<param name="use_dummy">${use_dummy}</param>
 				<param name="baud_rate">${baud_rate}</param>

File: igus_rebel_description_ros2/urdf/end_effectors/soft_gripper.description.xacro (robot description, xacro)
@@ -1,17 +1,24 @@
 <?xml version="1.0"?>
 <robot xmlns:xacro="http://www.ros.org/wiki/xacro" name="igus_rebel">
-	<!-- TODO: add meshes, mount v2 and end effector tip link for the Soft gripper -->
+	<material name="gripper_light_blue">
+		<color rgba="${0/255.0} ${127/255.0} ${255/255.0} 1.000" />
+	</material>
+	<material name="gripper_white">
+		<color rgba="${240/255.0} ${240/255.0} ${240/255.0} 1.000" />
+	</material>
 	<joint name="soft_gripper_joint" type="fixed">
-		<parent link="flange" />
-		<child link="soft_gripper_link" />
-		<origin xyz="0 0 0" rpy="0 0 0" />
+		<parent link="camera_mount" />
+		<child link="soft_gripper_mount" />
+		<origin xyz="0.0 0.0 0.0" rpy="0.0 0.0 ${pi/2.0}" />
 	</joint>
-	<link name="soft_gripper_link">
+	<link name="soft_gripper_mount">
 		<visual>
 			<origin xyz="0 0 0" rpy="0 0 0" />
 			<geometry>
 				<mesh
-					filename="package://igus_rebel_description_ros2/meshes/mounts/soft_gripper.stl" />
+					filename="package://igus_rebel_description_ros2/meshes/end_effectors/gripper_mount.stl"
+					scale="0.001 0.001 0.001" />
 			</geometry>
+			<material name="gripper_white" />
 		</visual>
 		<collision>
@@ -19,5 +26,6 @@
 			<geometry>
 				<mesh
-					filename="package://igus_rebel_description_ros2/meshes/mounts/soft_gripper.stl" />
+					filename="package://igus_rebel_description_ros2/meshes/end_effectors/gripper_mount.stl"
+					scale="0.001 0.001 0.001" />
 			</geometry>
 		</collision>
@@ -28,3 +36,38 @@
 		</inertial>
 	</link>
+	<joint name="soft_gripper_attachment" type="fixed">
+		<parent link="soft_gripper_mount" />
+		<child link="soft_gripper_link" />
+		<origin xyz="0.0 0 0" rpy="0 0 0" />
+	</joint>
+	<link name="soft_gripper_link">
+		<visual>
+			<origin xyz="0 0 0" rpy="0 0 0" />
+			<geometry>
+				<mesh
+					filename="package://igus_rebel_description_ros2/meshes/end_effectors/gripper.stl"
+					scale="0.001 0.001 0.001" />
+			</geometry>
+			<material name="gripper_light_blue" />
+		</visual>
+		<collision>
+			<origin xyz="0 0 0" rpy="0 0 0" />
+			<geometry>
+				<mesh
+					filename="package://igus_rebel_description_ros2/meshes/end_effectors/gripper.stl"
+					scale="0.001 0.001 0.001" />
+			</geometry>
+		</collision>
+		<inertial>
+			<origin xyz="0 0 0" rpy="0 0 0" />
+			<mass value="0.1" />
+			<inertia ixx="0.0001" ixy="0.0" ixz="0.0" iyy="0.0001" iyz="0.0" izz="0.0001" />
+		</inertial>
+	</link>
+	<joint name="soft_gripper_tip" type="fixed">
+		<parent link="soft_gripper_link" />
+		<child link="soft_gripper_tip_link" />
+		<origin xyz="0.0 0.0 0.1" rpy="${-pi/2.0} ${-pi/2.0} 0.0" />
+	</joint>
+	<link name="soft_gripper_tip_link" />
 </robot>

File: igus_rebel_description_ros2/urdf/igus_rebel/igus_rebel.description.xacro (robot description, xacro)
@@ -19,5 +19,6 @@
 				<geometry>
 					<mesh
-						filename="file://$(find igus_rebel_description_ros2)/meshes/igus_rebel_mod/Joint0.stl" />
+						filename="file://$(find igus_rebel_description_ros2)/meshes/igus_rebel_mod/Joint0.stl"
+						scale="0.0001 0.0001 0.0001" />
 				</geometry>
 			</collision>
@@ -47,5 +48,6 @@
 				<geometry>
 					<mesh
-						filename="file://$(find igus_rebel_description_ros2)/meshes/igus_rebel_mod/Joint1.stl" />
+						filename="file://$(find igus_rebel_description_ros2)/meshes/igus_rebel_mod/Joint1.stl"
+						scale="0.0001 0.0001 0.0001" />
 				</geometry>
 				<origin rpy="0 0 0" xyz="0 0 0" />
@@ -76,5 +78,6 @@
 				<geometry>
 					<mesh
-						filename="file://$(find igus_rebel_description_ros2)/meshes/igus_rebel_mod/Joint2.stl" />
+						filename="file://$(find igus_rebel_description_ros2)/meshes/igus_rebel_mod/Joint2.stl"
+						scale="0.0001 0.0001 0.0001" />
 				</geometry>
 				<origin rpy="0 0 0" xyz="0 0 0" />
@@ -105,5 +108,6 @@
 				<geometry>
 					<mesh
-						filename="file://$(find igus_rebel_description_ros2)/meshes/igus_rebel_mod/Joint3.stl" />
+						filename="file://$(find igus_rebel_description_ros2)/meshes/igus_rebel_mod/Joint3.stl"
+						scale="0.0001 0.0001 0.0001" />
 				</geometry>
 				<origin rpy="0 0 0" xyz="0 0 0" />
@@ -134,5 +138,6 @@
 				<geometry>
 					<mesh
-						filename="file://$(find igus_rebel_description_ros2)/meshes/igus_rebel_mod/Joint4.stl" />
+						filename="file://$(find igus_rebel_description_ros2)/meshes/igus_rebel_mod/Joint4.stl"
+						scale="0.0001 0.0001 0.0001" />
 				</geometry>
 				<origin rpy="0 0 0" xyz="0 0 0" />
@@ -163,5 +168,6 @@
 				<geometry>
 					<mesh
-						filename="file://$(find igus_rebel_description_ros2)/meshes/igus_rebel_mod/Joint5.stl" />
+						filename="file://$(find igus_rebel_description_ros2)/meshes/igus_rebel_mod/Joint5.stl"
+						scale="0.0001 0.0001 0.0001" />
 				</geometry>
 				<origin rpy="0 0 0" xyz="0 0 0" />
@@ -192,5 +198,6 @@
 				<geometry>
 					<mesh
-						filename="file://$(find igus_rebel_description_ros2)/meshes/igus_rebel_mod/Joint6.stl" />
+						filename="file://$(find igus_rebel_description_ros2)/meshes/igus_rebel_mod/Joint6.stl"
+						scale="0.0001 0.0001 0.0001" />
 				</geometry>
 				<origin rpy="0 0 0" xyz="0.0 0 0" />

File: igus_rebel_description_ros2/urdf/mounts/mount_v2.xacro (robot description, xacro)
@@ -9,19 +9,16 @@
 			<parent link="flange" />
 			<child link="camera_mount" />
-			<origin rpy="0.0 0.0 0.0" xyz="0.0 0.0 0.0" />
+			<origin rpy="0.0 ${pi/2.0} 0.0" xyz="0.0 0.0 0.0" />
 			<axis xyz="0 0 0" />
 		</joint>
-		<!-- camera mount urdf produced with fusion 360 urdf converter plugin-->
-		<!-- camera mount == mount_v1 link -->
+		<!-- camera mount == mount_v2 link -->
 		<link name="camera_mount">
 			<inertial>
-				<origin xyz="-0.01802331112330381 -0.0023580203613042293 0.03423412904225139"
-					rpy="0 0 0" />
+				<origin xyz="0.0 0.0 0.0" rpy="0.0 0.0 0.0" />
 				<mass value="1.0033" />
-				<inertia ixx="0.001725" iyy="0.00146" izz="0.000623" ixy="-2.3e-05" iyz="0.000102"
-					ixz="0.000224" />
+				<inertia ixx="0.001" iyy="0.001" izz="0.001" ixy="0.0" iyz="0.001" ixz="0.001" />
 			</inertial>
 			<visual>
-				<origin xyz="0.008 0 0" rpy="0 0 ${pi}" />
+				<origin xyz="0.0 0.0 0.0" rpy="0.0 0.0 ${pi/2.0}" />
 				<geometry>
 					<mesh
@@ -29,8 +26,8 @@
 						scale="0.001 0.001 0.001" />
 				</geometry>
-				<material name="mount_dark_green" />
+				<material name="mount_dark_grey" />
 			</visual>
 			<collision>
-				<origin xyz="0.008 0 0" rpy="0 0 ${pi}" />
+				<origin xyz="0.0 0.0 0.0" rpy="0.0 0.0 ${pi/2.0}" />
 				<geometry>
 					<mesh
@@ -44,5 +41,5 @@
 			<parent link="camera_mount" />
 			<child link="camera_insert" />
-			<origin rpy="0.0 0.0 0.0" xyz="0.038 0.0 0.065" />
+			<origin rpy="0.0 ${-pi/2.0} 0.0" xyz="-0.1 0.0 -0.035" />
 			<axis xyz="0 0 0" />
 		</joint>
@@ -50,11 +47,11 @@
 		<!-- End effectors -->
 		<xacro:if value="${end_effector == 'soft_gripper'}">
-            <!-- description urdf of the soft gripper -->
+			<!-- description urdf of the soft gripper -->
 			<xacro:include
 				filename="$(find igus_rebel_description_ros2)/urdf/end_effectors/soft_gripper.description.xacro" />
-            <!-- ros2 control of the soft gripper actuator -->
-            <xacro:include
-                filename="$(find igus_rebel_description_ros2)/urdf/end_effectors/soft_gripper.control.xacro" />
-            <xacro:igus_rebel_gripper use_dummy="false" />
+			<!-- ros2 control of the soft gripper actuator -->
+			<xacro:include
+				filename="$(find igus_rebel_description_ros2)/urdf/end_effectors/soft_gripper.control.xacro" />
+			<xacro:igus_rebel_gripper use_dummy="false" />
 		</xacro:if>
 	</xacro:macro>

File: igus_rebel_moveit_config/config/igus_rebel.srdf.xacro (robot description, xacro)
@@ -44,4 +44,17 @@
 					group="toucher_v1_group" parent_group="rebel_arm" />
 			</xacro:if>
+			<!-- If camera is realsense and toucher v1 is placed -->
+			<xacro:if value="${end_effector == 'soft_gripper'}">
+				<group name="rebel_arm">
+					<chain base_link="igus_rebel_base_link" tip_link="soft_gripper_tip_link" />
+				</group>
+				<group name="soft_gripper_group">
+					<link name="soft_gripper_mount" />
+					<link name="soft_gripper_link" />
+					<link name="soft_gripper_tip_link" />
+				</group>
+				<end_effector name="soft_gripper_EEF" parent_link="soft_gripper_tip_link"
+					group="soft_gripper_group" parent_group="rebel_arm" />
+			</xacro:if>
 		</xacro:if>
 		<!--############################################################################### -->
@@ -49,12 +62,4 @@
 		<!--############################################################################### -->
 		<!-- Positions common for every configuration -->
-		<group_state name="zero" group="rebel_arm">
-			<joint name="joint1" value="0" />
-			<joint name="joint2" value="0" />
-			<joint name="joint3" value="0" />
-			<joint name="joint4" value="0" />
-			<joint name="joint5" value="0" />
-			<joint name="joint6" value="0" />
-		</group_state>
 		<group_state name="home" group="rebel_arm">
 			<joint name="joint1" value="0" />
@@ -98,5 +103,5 @@
 		<disable_collisions link1="link_6" link2="link_7" reason="Adjacent" />
 		<disable_collisions link1="link_6" link2="link_8" reason="Never" />
-		<disable_collisions link1="link_7" link2="link_8" reason="Adjacent" /> <!-- 13 -->
+		<disable_collisions link1="link_7" link2="link_8" reason="Adjacent" />
 		<!-- Collisions checks due to the presence of the scout base -->
 		<xacro:if value="${load_base}">
@@ -154,5 +159,5 @@
 		</xacro:if>
 		<!-- Collision checks due to the presence of the mount -->
-		<xacro:if value="${mount == 'mount_v1'}">
+		<xacro:if value="${mount == 'mount_v1' or mount == 'mount_v2'}">
 			<disable_collisions link1="link_5" link2="camera_mount" reason="Never" />
 			<disable_collisions link1="link_6" link2="camera_mount" reason="Never" />
@@ -225,4 +230,29 @@
 					reason="Never" />
 			</xacro:if>
+			<xacro:if value="${camera == 'realsense' and end_effector == 'soft_gripper'}">
+				<disable_collisions link1="camera_mount" link2="camera_link" reason="Adjacent" />
+				<disable_collisions link1="link_7" link2="camera_link" reason="Never" />
+				<disable_collisions link1="link_8" link2="camera_link" reason="Never" />
+				<disable_collisions link1="camera_link" link2="camera_usb_plug_link"
+					reason="Adjacent" />
+				<disable_collisions link1="camera_mount" link2="camera_usb_plug_link" reason="Never" />
+				<disable_collisions link1="link_7" link2="camera_usb_plug_link" reason="Never" />
+				<disable_collisions link1="link_8" link2="camera_usb_plug_link" reason="Never" />
+				<disable_collisions link1="camera_mount" link2="soft_gripper_link" reason="Adjacent" />
+				<disable_collisions link1="camera_mount" link2="soft_gripper_mount"
+					reason="Adjacent" />
+				<disable_collisions link1="camera_link" link2="soft_gripper_mount" reason="Never" />
+				<disable_collisions link1="camera_link" link2="soft_gripper_link" reason="Never" />
+				<disable_collisions link1="soft_gripper_mount" link2="camera_usb_plug_link"
+					reason="Never" />
+				<disable_collisions link1="soft_gripper_link" link2="camera_usb_plug_link"
+					reason="Never" />
+				<disable_collisions link1="link_7" link2="soft_gripper_link" reason="Never" />
+				<disable_collisions link1="link_8" link2="soft_gripper_link" reason="Never" />
+				<disable_collisions link1="link_7" link2="soft_gripper_mount" reason="Never" />
+				<disable_collisions link1="link_8" link2="soft_gripper_mount" reason="Never" />
+				<disable_collisions link1="soft_gripper_mount" link2="soft_gripper_link"
+					reason="Adjacent" />
+			</xacro:if>
 		</xacro:if>
 	</xacro:macro>
