Commit message: added simplified collision meshes for soft gripper, new setup on robot

File: igus_rebel_description_ros2/urdf/end_effectors/soft_gripper.description.xacro (robot description, xacro)
@@ -10,9 +10,9 @@
 		<parent link="camera_mount" />
 		<child link="soft_gripper_mount" />
-		<origin xyz="0.0 0.0 -0.02" rpy="0.0 0.0 ${pi/2.0}" />
+		<origin xyz="0.0 0.0 0.0" rpy="0.0 0.0 0.0" />
 	</joint>
 	<link name="soft_gripper_mount">
 		<visual>
-			<origin xyz="0 0 0" rpy="0 0 0" />
+			<origin xyz="0.0 0.0 0.02" rpy="0.0 ${pi} 0.0" />
 			<geometry>
 				<mesh
@@ -23,13 +23,13 @@
 		</visual>
 		<collision>
-			<origin xyz="0 0 0" rpy="0 0 0" />
+			<origin xyz="0.0 0.0 0.02" rpy="0.0 ${pi} 0.0" />
 			<geometry>
 				<mesh
-					filename="package://igus_rebel_description_ros2/meshes/end_effectors/gripper_mount.stl"
+					filename="package://igus_rebel_description_ros2/meshes/end_effectors/gripper_mount_collision_mesh.stl"
 					scale="0.001 0.001 0.001" />
 			</geometry>
 		</collision>
 		<inertial>
-			<origin xyz="0 0 0" rpy="0 0 0" />
+			<origin xyz="0.0 0.0 0.02" rpy="0.0 ${pi} 0.0" />
 			<mass value="0.1" />
 			<inertia ixx="0.0001" ixy="0.0" ixz="0.0" iyy="0.0001" iyz="0.0" izz="0.0001" />
@@ -39,9 +39,9 @@
 		<parent link="soft_gripper_mount" />
 		<child link="soft_gripper_link" />
-		<origin xyz="0.0 0.0 0.0" rpy="0 0 0" />
+		<origin xyz="0.0 0.0 0.0" rpy="0.0 0.0 0.0" />
 	</joint>
 	<link name="soft_gripper_link">
 		<visual>
-			<origin xyz="0 0 0" rpy="0 0 0" />
+			<origin xyz="0.0 0.0 0.0" rpy="0.0 0.0 0.5" />
 			<geometry>
 				<mesh
@@ -52,13 +52,13 @@
 		</visual>
 		<collision>
-			<origin xyz="0 0 0" rpy="0 0 0" />
+			<origin xyz="0.0 0.0 0.02" rpy="0.0 0.0 0.5" />
 			<geometry>
 				<mesh
-					filename="package://igus_rebel_description_ros2/meshes/end_effectors/gripper.stl"
-					scale="0.001 0.001 0.001" />
-			</geometry>
-		</collision>
+				filename="package://igus_rebel_description_ros2/meshes/end_effectors/gripper_collision_mesh.stl"
+				scale="0.001 0.001 0.001" />
+		</geometry>
+	</collision>
 		<inertial>
-			<origin xyz="0 0 0" rpy="0 0 0" />
+			<origin xyz="0.0 0.0 0.0" rpy="0.0 0.0 0.5" />
 			<mass value="0.1" />
 			<inertia ixx="0.0001" ixy="0.0" ixz="0.0" iyy="0.0001" iyz="0.0" izz="0.0001" />
@@ -68,5 +68,5 @@
 		<parent link="soft_gripper_link" />
 		<child link="soft_gripper_tip_link" />
-		<origin xyz="0.0 0.0 0.095" rpy="${-pi/2.0} ${-pi/2.0} 0.0" />
+		<origin xyz="0.0 0.0 0.075" rpy="0.0 ${-pi/2.0} 0.0" />
 	</joint>
 	<link name="soft_gripper_tip_link" />

File: igus_rebel_description_ros2/urdf/mobile_robot/castle.urdf (robot description, URDF)
Before this commit: robot scout_v2, 1 links, 1 joints
Links:
- link tower_link: geometry collision box size=0.18 0.32 0.24; collision box size=0.38 0.32 0.69

File: igus_rebel_description_ros2/urdf/mounts/mount_v2.xacro (robot description, xacro)
@@ -32,7 +32,8 @@
 				<geometry>
 					<mesh
-						filename="file://$(find igus_rebel_description_ros2)/meshes/mounts/mount_v2.stl"
+						filename="file://$(find igus_rebel_description_ros2)/meshes/mounts/mount_v2_collision_mesh.stl"
 						scale="0.001 0.001 0.001" />
 				</geometry>
+				<material name="mount_dark_grey" />
 			</collision>
 		</link>

File: igus_rebel_moveit_config/config/igus_rebel.srdf.xacro (robot description, xacro)
@@ -11,5 +11,5 @@
 		<!-- 				Planning Groups Definitions and End Effectors					-->
 		<!--############################################################################### -->
-		<!-- If mount is not placed -->
+		<!-- If mount is not placed, naked robot -->
 		<xacro:if value="${mount == 'none'}">
 			<group name="rebel_arm">
@@ -24,5 +24,5 @@
 		<!-- If mount is placed -->
 		<xacro:if value="${mount != 'none'}">
-			<!-- If camera is oakd and no end effector-->
+			<!-- If camera is relasense or oakd and no end effector placed -->
 			<xacro:if value="${end_effector == 'none'}">
 				<group name="rebel_arm">
@@ -32,5 +32,5 @@
 					group="rebel_arm" />
 			</xacro:if>
-			<!-- If camera is realsense and toucher v1 is placed -->
+			<!-- If camera is realsense or oakd and toucher v1 is placed -->
 			<xacro:if value="${end_effector == 'toucher_v1'}">
 				<group name="rebel_arm">
@@ -44,5 +44,5 @@
 					group="toucher_v1_group" parent_group="rebel_arm" />
 			</xacro:if>
-			<!-- If camera is realsense and toucher v1 is placed -->
+			<!-- If camera is realsense and soft gripper is placed -->
 			<xacro:if value="${end_effector == 'soft_gripper'}">
 				<group name="rebel_arm">
@@ -218,4 +218,6 @@
 				<disable_collisions link1="link_7" link2="camera_link" reason="Never" />
 				<disable_collisions link1="link_8" link2="camera_link" reason="Never" />
+				<disable_collisions link1="link_7" link2="camera_mount" reason="Adjacent" />
+				<disable_collisions link1="link_8" link2="camera_mount" reason="Adjacent" />
 				<disable_collisions link1="camera_mount" link2="soft_gripper_link" reason="Adjacent" />
 				<disable_collisions link1="camera_mount" link2="soft_gripper_mount"

Commit message: new IK solver, better params for sensor3d, fixed pump control software

File: igus_rebel_description_ros2/urdf/end_effectors/soft_gripper.description.xacro (robot description, xacro)
@@ -70,5 +70,5 @@
 		<!-- suction cup mounted: 7.5cm offset -->
 		<!-- M5 screw 50mm mounted: 8.5mm offset -->
-		<origin xyz="0.0 0.0 0.075" rpy="0.0 ${-pi/2.0} 0.0" />
+		<origin xyz="0.0 0.0 0.045" rpy="0.0 ${-pi/2.0} 0.0" />
 	</joint>
 	<link name="soft_gripper_tip_link" />
