Commit message: bux fixes and new sensors parameters

File: igus_rebel_description_ros2/urdf/igus_rebel/igus_rebel.gazebo.xacro (robot description, xacro)
@@ -135,6 +135,6 @@
 					<horizontal_fov>1.05</horizontal_fov>
 					<image>
-						<width>1280</width>
-						<height>720</height>
+						<width>640</width>
+						<height>480</height>
 					</image>
 					<clip>
@@ -152,12 +152,9 @@
 			<sensor type="rgbd_camera" name="depth_camera">
 				<update_rate>10</update_rate>
-				<depth_camera>
+				<camera>
 					<horizontal_fov>1.05</horizontal_fov>
 					<image>
-						<width>320</width>
-						<height>240</height>
-						<!-- <width>1280</width>
-						<height>720</height> -->
-						<format>R8G8B8</format>
+						<width>640</width>
+						<height>480</height>
 					</image>
 					<clip>
@@ -165,5 +162,13 @@
 						<far>10.0</far>
 					</clip>
-				</depth_camera>
+					<lens>
+						<projection>
+							<p_fx>554</p_fx>
+							<p_fy>554</p_fy>
+							<p_cx>320</p_cx>
+							<p_cy>240</p_cy>
+						</projection>
+					</lens>
+				</camera>
 			</sensor>
 		</gazebo>
@@ -174,6 +179,6 @@
 					<horizontal_fov>1.05</horizontal_fov>
 					<image>
-						<width>320</width>
-						<height>240</height>
+						<width>640</width>
+						<height>480</height>
 						<format>R8G8B8</format>
 					</image>

File: igus_rebel_description_ros2/urdf/robot.urdf.xacro (robot description, xacro)
@@ -21,5 +21,5 @@
 	<xacro:property name="friction" value="0.0" />
 	<!-- Add world link, necessary only when igus rebel is loaded on gazebo without the scout -->
-	<xacro:if value="$(arg load_gazebo)">
+	<!-- <xacro:if value="$(arg load_gazebo)">
 		<xacro:unless value="$(arg load_base)">
 			<link name="world" />
@@ -29,7 +29,14 @@
 			</joint>
 		</xacro:unless>
-	</xacro:if>
+	</xacro:if> -->
 	<!-- Load mobile robot base, load_base must be true -->
 	<xacro:if value="$(arg load_base)">
+		<!-- <xacro:if value="$(arg load_gazebo)">
+			<link name="world" />
+			<joint name="world_joint" type="fixed">
+				<parent link="world" />
+				<child link="base_footprint" />
+			</joint>
+		</xacro:if> -->
 		<!-- add virtual joints and links to create a complete TF tree supporting both igus rebel
 		and mobile robot -->

File: igus_rebel_moveit_config/config/igus_rebel.srdf.xacro (robot description, xacro)
@@ -42,5 +42,5 @@
 				</group>
 				<end_effector name="toucher_v1_EEF" parent_link="toucher_endpoint"
-					group="rebel_arm" parent_group="toucher_v1_group" />
+					group="toucher_v1_group" parent_group="rebel_arm" />
 			</xacro:if>
 		</xacro:if>
