Commit message: new URDF structure with support for new cameras, mounts, end effectors

File: igus_rebel_description_ros2/urdf/igus_rebel/igus_rebel.control.xacro (robot description, xacro)
@@ -14,17 +14,19 @@
 				<xacro:if value="${hardware_protocol == 'cri'}">
 					<plugin>igus_rebel_hw_controller/RebelController</plugin>
-					<!--<param
-					name="ip">192.168.3.11</param>-->
-					<!--<param
-					name="port">3920</param>-->
+					<!--<param name="ip">192.168.1.102</param>-->
+					<!--<param name="port">3920</param>-->
+				</xacro:if>
+				<xacro:if value="${hardware_protocol == 'ignition'}">
+					<plugin>ign_ros2_control/IgnitionSystem</plugin>
 				</xacro:if>
 			</hardware>
-			<xacro:macro name="rebel_joint" params="name position_min=0 position_max=0 cri_joint_offset=0">
+			<xacro:macro name="rebel_joint"
+				params="name position_min=0 position_max=0 cri_joint_offset=0">
 				<joint name="${name}">
+					<!-- Position control can be optionally deployed -->
 					<!--<command_interface name="position">
 						<param name="min">${position_min}</param>
 						<param name="max">${position_max}</param>
 					</command_interface>-->
-					<!-- If you want to increase the velocity and/or speed limit please consult the readme of this package first -->
 					<command_interface name="velocity">
 						<param name="min">${-pi/4}</param>
@@ -34,5 +36,4 @@
 						<param name="initial_value">0.0</param>
 					</state_interface>
-					<!-- Velocity is required for moveit+mock_components -->
 					<state_interface name="velocity">
 						<param name="initial_value">0.0</param>
@@ -42,31 +43,17 @@
 				</joint>
 			</xacro:macro>
-			<!-- Position limit difference with iRC files due to 30 degree offset in joint 2 and 3 -->
-			<xacro:rebel_joint name="joint1" position_min="${-pi*179/180}" position_max="${pi*179/180}" />
-			<xacro:rebel_joint name="joint2" position_min="${-pi*2/3}" position_max="${pi*2/3}" cri_joint_offset="${-pi/6.0}" />
-			<xacro:rebel_joint name="joint3" position_min="${-pi*2/3}" position_max="${pi*2/3}" cri_joint_offset="${-pi/6.0}" />
-			<xacro:rebel_joint name="joint4" position_min="${-pi*179/180}" position_max="${pi*179/180}" />
-			<xacro:rebel_joint name="joint5" position_min="${-pi*19/36}" position_max="${pi*19/36}" cri_joint_offset="${pi/24.0}" />
-			<xacro:rebel_joint name="joint6" position_min="${-pi*179/180}" position_max="${pi*179/180}" />
-			<!--
-			<xacro:macro name="arm_control" params="transmission joint motor">
-				<transmission name="${transmission}">
-					<plugin>transmission_interface/SimpleTransmission</plugin>
-					<joint name="${joint}">
-						<hardwareInterface>hardware_interface/EffortJointInterface</hardwareInterface>
-					</joint>
-					<actuator name="${motor}" role="actuator_${motor}">
-						<hardwareInterface>hardware_interface/EffortJointInterface</hardwareInterface>
-						<mechanicalReduction>1</mechanicalReduction>
-					</actuator>
-				</transmission>
-			</xacro:macro>
-			<xacro:arm_control transmission="rebel_tran_1" joint="joint1" motor="rebel_motor_1" />
-			<xacro:arm_control transmission="rebel_tran_2" joint="joint2" motor="rebel_motor_2" />
-			<xacro:arm_control transmission="rebel_tran_3" joint="joint3" motor="rebel_motor_3" />
-			<xacro:arm_control transmission="rebel_tran_4" joint="joint4" motor="rebel_motor_4" />
-			<xacro:arm_control transmission="rebel_tran_5" joint="joint5" motor="rebel_motor_5" />
-			<xacro:arm_control transmission="rebel_tran_6" joint="joint6" motor="rebel_motor_6" />
-		-->
+			<!-- CRI joints offset for virtual zero definition -->
+			<xacro:rebel_joint name="joint1" position_min="${-pi*179/180}"
+				position_max="${pi*179/180}" />
+			<xacro:rebel_joint name="joint2" position_min="${-pi*2/3}" position_max="${pi*2/3}"
+				cri_joint_offset="${-pi/6.0}" />
+			<xacro:rebel_joint name="joint3" position_min="${-pi*2/3}" position_max="${pi*2/3}"
+				cri_joint_offset="${-pi/6.0}" />
+			<xacro:rebel_joint name="joint4" position_min="${-pi*179/180}"
+				position_max="${pi*179/180}" />
+			<xacro:rebel_joint name="joint5" position_min="${-pi*19/36}" position_max="${pi*19/36}"
+				cri_joint_offset="${pi/24.0}" />
+			<xacro:rebel_joint name="joint6" position_min="${-pi*179/180}"
+				position_max="${pi*179/180}" />
 		</ros2_control>
 	</xacro:macro>

File: igus_rebel_description_ros2/urdf/igus_rebel/igus_rebel.description.xacro (robot description, xacro)
@@ -1,16 +1,23 @@
 <?xml version="1.0"?>
 <robot xmlns:xacro="http://www.ros.org/wiki/xacro" name="igus_rebel">
+	<material name="dark_grey">
+		<color rgba="${5/255.0} ${5/255.0} ${5/255.0} 1.000" />
+	</material>
 	<xacro:macro name="igus_rebel_description">
+		<!-- Set both at 0.0 if collapsing is not interesting in gazebo -->
+		<xacro:property name="damping" value="0.0" />
+		<xacro:property name="friction" value="0.0" />
 		<link name="igus_rebel_base_link">
 			<visual>
 				<geometry>
 					<mesh
-						filename="file://$(find igus_rebel_description_ros2)/meshes/new/Joint0.dae" />
-				</geometry>
-			</visual>
-			<collision>
-				<geometry>
-					<mesh
-						filename="file://$(find igus_rebel_description_ros2)/meshes/new/Joint0.dae" />
+						filename="file://$(find igus_rebel_description_ros2)/meshes/igus_rebel/Joint0.dae" />
+				</geometry>
+				<material name="dark_grey" />
+			</visual>
+			<collision>
+				<geometry>
+					<mesh
+						filename="file://$(find igus_rebel_description_ros2)/meshes/igus_rebel/Joint0.dae" />
 				</geometry>
 			</collision>
@@ -27,4 +34,5 @@
 			<limit effort="330.0" lower="${-pi*179/180}" upper="${pi*179/180}"
 				velocity="${pi*45/180}" />
+			<dynamics damping="${damping}" friction="${friction}" />
 		</joint>
 		<link name="link_1">
@@ -32,12 +40,13 @@
 				<geometry>
 					<mesh
-						filename="file://$(find igus_rebel_description_ros2)/meshes/new/Joint1.dae" />
-				</geometry>
-				<origin rpy="0 0 0" xyz="0 0 0" />
-			</visual>
-			<collision>
-				<geometry>
-					<mesh
-						filename="file://$(find igus_rebel_description_ros2)/meshes/new/Joint1.dae" />
+						filename="file://$(find igus_rebel_description_ros2)/meshes/igus_rebel/Joint1.dae" />
+				</geometry>
+				<origin rpy="0 0 0" xyz="0 0 0" />
+				<material name="dark_grey" />
+			</visual>
+			<collision>
+				<geometry>
+					<mesh
+						filename="file://$(find igus_rebel_description_ros2)/meshes/igus_rebel/Joint1.dae" />
 				</geometry>
 				<origin rpy="0 0 0" xyz="0 0 0" />
@@ -56,4 +65,5 @@
 			limits lower -->
 			<limit effort="330.0" lower="${-pi*11/18}" upper="${pi*11/18}" velocity="${pi*45/180}" />
+			<dynamics damping="${damping}" friction="${friction}" />
 		</joint>
 		<link name="link_2">
@@ -61,12 +71,13 @@
 				<geometry>
 					<mesh
-						filename="file://$(find igus_rebel_description_ros2)/meshes/new/Joint2.dae" />
-				</geometry>
-				<origin rpy="0 0 0" xyz="0 0 0" />
-			</visual>
-			<collision>
-				<geometry>
-					<mesh
-						filename="file://$(find igus_rebel_description_ros2)/meshes/new/Joint2.dae" />
+						filename="file://$(find igus_rebel_description_ros2)/meshes/igus_rebel/Joint2.dae" />
+				</geometry>
+				<origin rpy="0 0 0" xyz="0 0 0" />
+				<material name="dark_grey" />
+			</visual>
+			<collision>
+				<geometry>
+					<mesh
+						filename="file://$(find igus_rebel_description_ros2)/meshes/igus_rebel/Joint2.dae" />
 				</geometry>
 				<origin rpy="0 0 0" xyz="0 0 0" />
@@ -85,4 +96,5 @@
 			limits lower -->
 			<limit effort="330.0" lower="${-pi*11/18}" upper="${pi*11/18}" velocity="${pi*45/180}" />
+			<dynamics damping="${damping}" friction="${friction}" />
 		</joint>
 		<link name="link_5">
@@ -90,12 +102,13 @@
 				<geometry>
 					<mesh
-						filename="file://$(find igus_rebel_description_ros2)/meshes/new/Joint3.dae" />
-				</geometry>
-				<origin rpy="0 0 0" xyz="0 0 0" />
-			</visual>
-			<collision>
-				<geometry>
-					<mesh
-						filename="file://$(find igus_rebel_description_ros2)/meshes/new/Joint3.dae" />
+						filename="file://$(find igus_rebel_description_ros2)/meshes/igus_rebel/Joint3.dae" />
+				</geometry>
+				<origin rpy="0 0 0" xyz="0 0 0" />
+				<material name="dark_grey" />
+			</visual>
+			<collision>
+				<geometry>
+					<mesh
+						filename="file://$(find igus_rebel_description_ros2)/meshes/igus_rebel/Joint3.dae" />
 				</geometry>
 				<origin rpy="0 0 0" xyz="0 0 0" />
@@ -109,9 +122,9 @@
 			<parent link="link_5" />
 			<child link="link_6" />
-			<!-- TODO The 0.03m offset are most likely caused by the mesh file (Issue 15)-->
 			<origin rpy="0.0 0.0 0.0" xyz="0.0 0 ${0.149 - 0.03}" />
 			<axis xyz="0 0 1" />
 			<limit effort="330.0" lower="${-pi*179/180}" upper="${pi*179/180}"
 				velocity="${pi*45/180}" />
+			<dynamics damping="${damping}" friction="${friction}" />
 		</joint>
 		<link name="link_6">
@@ -119,12 +132,13 @@
 				<geometry>
 					<mesh
-						filename="file://$(find igus_rebel_description_ros2)/meshes/new/Joint4.dae" />
-				</geometry>
-				<origin rpy="0 0 0" xyz="0 0 0" />
-			</visual>
-			<collision>
-				<geometry>
-					<mesh
-						filename="file://$(find igus_rebel_description_ros2)/meshes/new/Joint4.dae" />
+						filename="file://$(find igus_rebel_description_ros2)/meshes/igus_rebel/Joint4.dae" />
+				</geometry>
+				<origin rpy="0 0 0" xyz="0 0 0" />
+				<material name="dark_grey" />
+			</visual>
+			<collision>
+				<geometry>
+					<mesh
+						filename="file://$(find igus_rebel_description_ros2)/meshes/igus_rebel/Joint4.dae" />
 				</geometry>
 				<origin rpy="0 0 0" xyz="0 0 0" />
@@ -138,9 +152,9 @@
 			<parent link="link_6" />
 			<child link="link_7" />
-			<!-- TODO The 0.03m offset are most likely caused by the mesh file (Issue 15) -->
 			<origin rpy="0.0 ${-pi/24} 0.0" xyz="0.0 0 ${0.14 + 0.03}" />
 			<axis xyz="0 1 0" />
 			<limit effort="330.0" lower="${-pi*19/36 + pi/24}" upper="${pi*19/36 + pi/24}"
 				velocity="${pi*45/180}" />
+			<dynamics damping="${damping}" friction="${friction}" />
 		</joint>
 		<link name="link_7">
@@ -148,12 +162,13 @@
 				<geometry>
 					<mesh
-						filename="file://$(find igus_rebel_description_ros2)/meshes/new/Joint5.dae" />
-				</geometry>
-				<origin rpy="0 0 0" xyz="0 0 0" />
-			</visual>
-			<collision>
-				<geometry>
-					<mesh
-						filename="file://$(find igus_rebel_description_ros2)/meshes/new/Joint5.dae" />
+						filename="file://$(find igus_rebel_description_ros2)/meshes/igus_rebel/Joint5.dae" />
+				</geometry>
+				<origin rpy="0 0 0" xyz="0 0 0" />
+				<material name="dark_grey" />
+			</visual>
+			<collision>
+				<geometry>
+					<mesh
+						filename="file://$(find igus_rebel_description_ros2)/meshes/igus_rebel/Joint5.dae" />
 				</geometry>
 				<origin rpy="0 0 0" xyz="0 0 0" />
@@ -171,4 +186,5 @@
 			<limit effort="330.0" lower="${-pi*179/180}" upper="${pi*179/180}"
 				velocity="${pi*45/180}" />
+			<dynamics damping="${damping}" friction="${friction}" />
 		</joint>
 		<link name="link_8">
@@ -176,12 +192,13 @@
 				<geometry>
 					<mesh
-						filename="file://$(find igus_rebel_description_ros2)/meshes/new/Joint6.dae" />
+						filename="file://$(find igus_rebel_description_ros2)/meshes/igus_rebel/Joint6.dae" />
 				</geometry>
 				<origin rpy="0 0 0" xyz="0.0 0 0" />
-			</visual>
-			<collision>
-				<geometry>
-					<mesh
-						filename="file://$(find igus_rebel_description_ros2)/meshes/new/Joint6.dae" />
+				<material name="dark_grey" />
+			</visual>
+			<collision>
+				<geometry>
+					<mesh
+						filename="file://$(find igus_rebel_description_ros2)/meshes/igus_rebel/Joint6.dae" />
 				</geometry>
 				<origin rpy="0 0 0" xyz="0.0 0 0" />
@@ -197,7 +214,7 @@
 			<origin rpy="0.0 ${-pi/2} 0.0" xyz="0.0 0 0.0012" />
 			<axis xyz="0 0 0" />
-		</joint>
-		<link name="flange">
-		</link>
+			<dynamics damping="${damping}" friction="${friction}" />
+		</joint>
+		<link name="flange" />
 	</xacro:macro>
 </robot>

File: igus_rebel_description_ros2/urdf/igus_rebel/igus_rebel.urdf.xacro (robot description, xacro)
@@ -2,5 +2,6 @@
 <robot xmlns:xacro="http://www.ros.org/wiki/xacro" name="igus_rebel">
 	<!-- macro definition for the robot -->
-	<xacro:macro name="igus_rebel" params="hardware_protocol gripper load_base">
+	<xacro:macro name="igus_rebel"
+		params="load_base mount camera end_effector hardware_protocol load_gazebo moveit">
 		<!-- Include and call rebel macro -->
 		<xacro:include
@@ -8,9 +9,39 @@
 		<xacro:igus_rebel_description />
 		<!-- controller macro -->
-		<xacro:include filename="$(find igus_rebel_description_ros2)/urdf/igus_rebel/igus_rebel.control.xacro" />
+		<xacro:include
+			filename="$(find igus_rebel_description_ros2)/urdf/igus_rebel/igus_rebel.control.xacro" />
 		<xacro:igus_rebel_control hardware_protocol="${hardware_protocol}" />
-		<!-- Grippers -->
-		<xacro:include filename="$(find igus_rebel_description_ros2)/urdf/grippers/grippers.xacro" />
-		<xacro:gripper gripper_type="${gripper}" />
+		<!-- Mount macro -->
+		<xacro:if value="${mount == 'mount_v1'}">
+			<xacro:include filename="$(find igus_rebel_description_ros2)/urdf/mounts/mount_v1.xacro" />
+			<xacro:mount_v1 camera="$(arg camera)" end_effector="$(arg end_effector)"
+				load_gazebo="$(arg load_gazebo)" />
+		</xacro:if>
+		<!-- Gazebo macro -->
+		<xacro:if value="${load_gazebo}">
+			<xacro:include
+				filename="$(find igus_rebel_description_ros2)/urdf/igus_rebel/igus_rebel.gazebo.xacro" />
+			<!-- The plugin that control the robot in Ignition is loaded if Moveit2 will be used.
+			The Moveit2 controller configuration file is directly passed as a parameter to this plugin -->
+			<xacro:if value="${moveit}">
+				<xacro:ign_ros2_control
+					controller_parameters="$(find igus_rebel_moveit_config)/config/ros2_controllers.yaml" />
+			</xacro:if>
+			<!-- The joint state publisher and the joint position controller are loaded if Moveit2
+			is not used	because the robot is controllable directly from Ignition if some movement are needed -->
+			<xacro:unless value="${moveit}">
+				<xacro:ign_joint_state_publisher />
+				<xacro:ign_joint_position_controller />
+			</xacro:unless>
+			<!-- The sensors used in Ignition are loaded only if a camera is attached -->
+			<xacro:unless value="${camera == 'none' or mount == 'none'}">
+				<xacro:virtual_sensors />
+				<!-- Since there is already a a sensor plugin in the scout, if the scout is loaded
+				the sensor plugin of the igus rebel is not loaded (temporary solution) -->
+				<xacro:unless value="${load_base}">
+					<xacro:ign_sensor_plugin />
+				</xacro:unless>
+			</xacro:unless>
+		</xacro:if>
 	</xacro:macro>
 </robot>

File: igus_rebel_description_ros2/urdf/robot.urdf.xacro (robot description, xacro)
@@ -1,14 +1,33 @@
 <?xml version="1.0"?>
 <robot xmlns:xacro="http://www.ros.org/wiki/xacro" name="igus_rebel">
+	<!-- Scout base selection -->
+	<xacro:arg name="load_base" default="true" />
+	<!-- Mount selection -->
+	<xacro:arg name="mount" default="none" />
+	<!-- Camera type selection -->
+	<xacro:arg name="camera" default="none" />
+	<!-- End effector type selection -->
+	<xacro:arg name="end_effector" default="none" />
+	<!-- Gazebo version -->
+	<xacro:arg name="load_gazebo" default="false" />
 	<!-- Controller settings, only enable a single one in the launch file -->
 	<xacro:arg name="hardware_protocol" default="simulation" />
-	<!-- Gripper selection -->
-	<xacro:arg name="gripper" default="camera" />
-	<!-- Load base -->
-	<xacro:arg name="load_base" default="false" />
-	<!-- load gazebo xacro -->
-	<xacro:arg name="load_gazebo" default="false" />
+	<!-- Argument that tells if Moveit2 is used or not -->
+	<xacro:arg name="moveit" default="false" />
 	<!-- odometry source: world ground truth or wheels encoders -->
 	<xacro:arg name="odometry_source" default="ground_truth" />
+	<!-- Set both at 0.0 if collapsing is not interesting in gazebo -->
+	<xacro:property name="damping" value="0.0" />
+	<xacro:property name="friction" value="0.0" />
+	<!-- Add world link, necessary only when igus rebel is loaded on gazebo without the scout -->
+	<xacro:if value="$(arg load_gazebo)">
+		<xacro:unless value="$(arg load_base)">
+			<link name="world" />
+			<joint name="world_joint" type="fixed">
+				<parent link="world" />
+				<child link="base_link" />
+			</joint>
+		</xacro:unless>
+	</xacro:if>
 	<!-- Load mobile robot base, load_base must be true -->
 	<xacro:if value="$(arg load_base)">
@@ -51,5 +70,6 @@
 		filename="$(find igus_rebel_description_ros2)/urdf/igus_rebel/igus_rebel.urdf.xacro" />
 	<xacro:igus_rebel
-		gripper="$(arg gripper)" hardware_protocol="$(arg hardware_protocol)"
-		load_base="$(arg load_base)" />
+		load_base="$(arg load_base)" mount="$(arg mount)" camera="$(arg camera)"
+		end_effector="$(arg end_effector)" hardware_protocol="$(arg hardware_protocol)"
+		load_gazebo="$(arg load_gazebo)" moveit="$(arg moveit)" />
 </robot>

Commit message: corrected wrong link positions and wrong length of the arm

File: igus_rebel_description_ros2/urdf/igus_rebel/igus_rebel.control.xacro (robot description, xacro)
@@ -49,5 +49,5 @@
 				cri_joint_offset="${-pi/6.0}" />
 			<xacro:rebel_joint name="joint3" position_min="${-pi*2/3}" position_max="${pi*2/3}"
-				cri_joint_offset="${-pi/6.0}" />
+				cri_joint_offset="${-pi*34.0/180.0}" />
 			<xacro:rebel_joint name="joint4" position_min="${-pi*179/180}"
 				position_max="${pi*179/180}" />

File: igus_rebel_description_ros2/urdf/igus_rebel/igus_rebel.description.xacro (robot description, xacro)
@@ -30,8 +30,7 @@
 			<parent link="igus_rebel_base_link" />
 			<child link="link_1" />
-			<origin rpy="0.0 0.0 0.0" xyz="0.0 0 0.100" />
+			<origin rpy="0.0 0.0 0.0" xyz="0.0 0 0.103" />
 			<axis xyz="0 0 1" />
-			<limit effort="330.0" lower="${-pi*179/180}" upper="${pi*179/180}"
-				velocity="${pi*45/180}" />
+			<limit effort="330.0" lower="${-pi*179/180}" upper="${pi*179/180}" velocity="${pi/4.0}" />
 			<dynamics damping="${damping}" friction="${friction}" />
 		</joint>
@@ -60,9 +59,9 @@
 			<parent link="link_1" />
 			<child link="link_2" />
-			<origin rpy="0.0 ${pi/6} 0.0" xyz="0.0 0 0.149" />
+			<origin rpy="0.0 ${pi/6} 0.0" xyz="0.0 0.0 0.149" />
 			<axis xyz="0 1 0" />
 			<!-- pi*2/3 are the physical limits, but to avoid any collisions we set the actual
 			limits lower -->
-			<limit effort="330.0" lower="${-pi*11/18}" upper="${pi*11/18}" velocity="${pi*45/180}" />
+			<limit effort="330.0" lower="${-pi*11/18}" upper="${pi*11/18}" velocity="${pi/4.0}" />
 			<dynamics damping="${damping}" friction="${friction}" />
 		</joint>
@@ -91,9 +90,7 @@
 			<parent link="link_2" />
 			<child link="link_5" />
-			<origin rpy="0.0 ${pi/6} 0.0" xyz="0.0 0.0 0.2384" />
+			<origin rpy="0.0 ${pi/6} 0.0" xyz="0.0 0.0 0.237" />
 			<axis xyz="0 1 0" />
-			<!-- pi*2/3 are the physical limits, but to avoid any collisions we set the actual
-			limits lower -->
-			<limit effort="330.0" lower="${-pi*11/18}" upper="${pi*11/18}" velocity="${pi*45/180}" />
+			<limit effort="330.0" lower="${-pi*11/18}" upper="${pi*11/18}" velocity="${pi/4.0}" />
 			<dynamics damping="${damping}" friction="${friction}" />
 		</joint>
@@ -122,8 +119,7 @@
 			<parent link="link_5" />
 			<child link="link_6" />
-			<origin rpy="0.0 0.0 0.0" xyz="0.0 0 ${0.149 - 0.03}" />
+			<origin rpy="0.0 0.0 0.0" xyz="0.0 0.0 0.127" />
 			<axis xyz="0 0 1" />
-			<limit effort="330.0" lower="${-pi*179/180}" upper="${pi*179/180}"
-				velocity="${pi*45/180}" />
+			<limit effort="330.0" lower="${-pi*179/180}" upper="${pi*179/180}" velocity="${pi/4.0}" />
 			<dynamics damping="${damping}" friction="${friction}" />
 		</joint>
@@ -152,8 +148,8 @@
 			<parent link="link_6" />
 			<child link="link_7" />
-			<origin rpy="0.0 ${-pi/24} 0.0" xyz="0.0 0 ${0.14 + 0.03}" />
+			<origin rpy="0.0 ${-pi/24} 0.0" xyz="0.0 0.0 0.170" />
 			<axis xyz="0 1 0" />
 			<limit effort="330.0" lower="${-pi*19/36 + pi/24}" upper="${pi*19/36 + pi/24}"
-				velocity="${pi*45/180}" />
+				velocity="${pi/4.0}" />
 			<dynamics damping="${damping}" friction="${friction}" />
 		</joint>
@@ -184,6 +180,5 @@
 			<origin rpy="0.0 0.0 0.0" xyz="0.0 0 0.1208" />
 			<axis xyz="0 0 1" />
-			<limit effort="330.0" lower="${-pi*179/180}" upper="${pi*179/180}"
-				velocity="${pi*45/180}" />
+			<limit effort="330.0" lower="${-pi*179/180}" upper="${pi*179/180}" velocity="${pi/4.0}" />
 			<dynamics damping="${damping}" friction="${friction}" />
 		</joint>
@@ -212,5 +207,5 @@
 			<parent link="link_8" />
 			<child link="flange" />
-			<origin rpy="0.0 ${-pi/2} 0.0" xyz="0.0 0 0.0012" />
+			<origin rpy="0.0 ${-pi/2} 0.0" xyz="0.0 0 0.0052" />
 			<axis xyz="0 0 0" />
 			<dynamics damping="${damping}" friction="${friction}" />

File: igus_rebel_description_ros2/urdf/robot.urdf.xacro (robot description, xacro)
@@ -20,32 +20,11 @@
 	<xacro:property name="damping" value="0.0" />
 	<xacro:property name="friction" value="0.0" />
-	<!-- Add world link, necessary only when igus rebel is loaded on gazebo without the scout -->
-	<!-- <xacro:if value="$(arg load_gazebo)">
-		<xacro:unless value="$(arg load_base)">
-			<link name="world" />
-			<joint name="world_joint" type="fixed">
-				<parent link="world" />
-				<child link="base_link" />
-			</joint>
-		</xacro:unless>
-	</xacro:if> -->
 	<!-- Load mobile robot base, load_base must be true -->
 	<xacro:if value="$(arg load_base)">
-		<!-- <xacro:if value="$(arg load_gazebo)">
-			<link name="world" />
-			<joint name="world_joint" type="fixed">
-				<parent link="world" />
-				<child link="base_footprint" />
-			</joint>
-		</xacro:if> -->
-		<!-- add virtual joints and links to create a complete TF tree supporting both igus rebel
-		and mobile robot -->
-		<!-- base_footprint -> base_link -> { mobile_robot_base_link, rebel_support ->
-		igus_rebel_base_link } -> other links -->
 		<!-- virtual joints acting as a link between base_link and igus_rebel_base_link -->
 		<joint name="base_link_to_rebel_support" type="fixed">
 			<parent link="base_link" />
 			<child link="rebel_support" />
-			<origin xyz="-0.28 0.0 0.135" rpy="0 0 ${pi}" />
+			<origin xyz="-0.28 0.0 0.125" rpy="0 0 ${pi}" />
 		</joint>
 		<link name="rebel_support" />
