Commit message: removed static offsets due to rotations in the joints urdf

File: igus_rebel_description_ros2/urdf/igus_rebel/igus_rebel.control.xacro (robot description, xacro)
@@ -47,11 +47,10 @@
 				position_max="${pi*179/180}" />
 			<xacro:rebel_joint name="joint2" position_min="${-pi*2/3}" position_max="${pi*2/3}"
-				cri_joint_offset="${-pi/6.0}" />
+				cri_joint_offset="${-pi*0.8/180.0}" />
 			<xacro:rebel_joint name="joint3" position_min="${-pi*2/3}" position_max="${pi*2/3}"
-				cri_joint_offset="${-pi*34.0/180.0}" />
+				cri_joint_offset="${-pi*0.5/180.0}" />
 			<xacro:rebel_joint name="joint4" position_min="${-pi*179/180}"
 				position_max="${pi*179/180}" />
-			<xacro:rebel_joint name="joint5" position_min="${-pi*19/36}" position_max="${pi*19/36}"
-				cri_joint_offset="${pi/24.0}" />
+			<xacro:rebel_joint name="joint5" position_min="${-pi*19/36}" position_max="${pi*19/36}" />
 			<xacro:rebel_joint name="joint6" position_min="${-pi*179/180}"
 				position_max="${pi*179/180}" />

File: igus_rebel_description_ros2/urdf/igus_rebel/igus_rebel.description.xacro (robot description, xacro)
@@ -59,9 +59,9 @@
 			<parent link="link_1" />
 			<child link="link_2" />
-			<origin rpy="0.0 ${pi/6} 0.0" xyz="0.0 0.0 0.149" />
+			<origin rpy="0.0 0.0 0.0" xyz="0.0 0.0 0.149" />
 			<axis xyz="0 1 0" />
 			<!-- pi*2/3 are the physical limits, but to avoid any collisions we set the actual
 			limits lower -->
-			<limit effort="330.0" lower="${-pi*11/18}" upper="${pi*11/18}" velocity="${pi/4.0}" />
+			<limit effort="330.0" lower="${-pi*80/180}" upper="${pi*140/180}" velocity="${pi/4.0}" />
 			<dynamics damping="${damping}" friction="${friction}" />
 		</joint>
@@ -90,7 +90,7 @@
 			<parent link="link_2" />
 			<child link="link_5" />
-			<origin rpy="0.0 ${pi/6} 0.0" xyz="0.0 0.0 0.237" />
+			<origin rpy="0.0 0.0 0.0" xyz="0.0 0.0 0.237" />
 			<axis xyz="0 1 0" />
-			<limit effort="330.0" lower="${-pi*11/18}" upper="${pi*11/18}" velocity="${pi/4.0}" />
+			<limit effort="330.0" lower="${-pi*80/180}" upper="${pi*140/180}" velocity="${pi/4.0}" />
 			<dynamics damping="${damping}" friction="${friction}" />
 		</joint>
@@ -148,8 +148,7 @@
 			<parent link="link_6" />
 			<child link="link_7" />
-			<origin rpy="0.0 ${-pi/24} 0.0" xyz="0.0 0.0 0.170" />
+			<origin rpy="0.0 0.0 0.0" xyz="0.0 0.0 0.170" />
 			<axis xyz="0 1 0" />
-			<limit effort="330.0" lower="${-pi*19/36 + pi/24}" upper="${pi*19/36 + pi/24}"
-				velocity="${pi/4.0}" />
+			<limit effort="330.0" lower="${-pi/2.0}" upper="${pi/2.0}" velocity="${pi/4.0}" />
 			<dynamics damping="${damping}" friction="${friction}" />
 		</joint>

File: igus_rebel_moveit_config/config/igus_rebel.srdf.xacro (robot description, xacro)
@@ -59,24 +59,24 @@
 		<group_state name="home" group="rebel_arm">
 			<joint name="joint1" value="0" />
-			<joint name="joint2" value="${-pi/6.0}" />
-			<joint name="joint3" value="${-pi/6.0}" />
+			<joint name="joint2" value="0" />
+			<joint name="joint3" value="0" />
 			<joint name="joint4" value="0" />
-			<joint name="joint5" value="${pi/24.0}" />
+			<joint name="joint5" value="0" />
 			<joint name="joint6" value="0" />
 		</group_state>
 		<group_state name="parked" group="rebel_arm">
 			<joint name="joint1" value="${-42.0 * pi / 180.0}" />
-			<joint name="joint2" value="${40.0 * pi / 180.0}" />
-			<joint name="joint3" value="${73.0 * pi / 180.0}" />
+			<joint name="joint2" value="${70.0 * pi / 180.0}" />
+			<joint name="joint3" value="${103.0 * pi / 180.0}" />
 			<joint name="joint4" value="${82.0 * pi / 180.0}" />
-			<joint name="joint5" value="${-78.0 * pi / 180.0}" />
+			<joint name="joint5" value="${-86.0 * pi / 180.0}" />
 			<joint name="joint6" value="${-95.0 * pi / 180.0}" />
 		</group_state>
 		<group_state name="stand" group="rebel_arm">
 			<joint name="joint1" value="${61.0 * pi / 180.0}" />
-			<joint name="joint2" value="${-90.0 * pi / 180.0}" />
-			<joint name="joint3" value="${36.0 * pi / 180.0}" />
+			<joint name="joint2" value="${-60.0 * pi / 180.0}" />
+			<joint name="joint3" value="${66.0 * pi / 180.0}" />
 			<joint name="joint4" value="0" />
-			<joint name="joint5" value="${95.0 * pi / 180.0}" />
+			<joint name="joint5" value="${87.0 * pi / 180.0}" />
 			<joint name="joint6" value="${5.0 * pi / 180.0}" />
 		</group_state>
