Commit message: Minimal features to work with the arm. Changes for Humble support

File: igus_rebel_description_ros2/urdf/igus_rebel/igus_rebel.urdf.xacro (robot description, xacro)
@@ -2,6 +2,32 @@
 <robot xmlns:xacro="http://www.ros.org/wiki/xacro" name="igus_rebel">
 	<!-- macro definition for the robot -->
-	<xacro:macro name="igus_rebel"
-		params="load_base mount camera end_effector hardware_protocol load_gazebo moveit">
+	<xacro:macro name="igus_rebel" params="hardware_protocol load_gazebo moveit">
+<!--		params="load_base mount camera end_effector hardware_protocol load_gazebo moveit">-->
+		<!-- Gazebo macro -->
+		<xacro:if value="${load_gazebo}">
+			<xacro:include
+					filename="$(find igus_rebel_description_ros2)/urdf/igus_rebel/igus_rebel.gazebo.xacro" />
+			<!-- The plugin that control the robot in Ignition is loaded if Moveit2 will be used.
+			The Moveit2 controller configuration file is directly passed as a parameter to this plugin -->
+			<xacro:if value="${moveit}">
+				<xacro:ign_ros2_control
+						controller_parameters="$(find igus_rebel_moveit_config)/config/gazebo_controllers.yaml" />
+			</xacro:if>
+			<!-- The joint state publisher and the joint position controller are loaded if Moveit2
+			is not used	because the robot is controllable directly from Ignition if some movement are needed -->
+			<xacro:unless value="${moveit}">
+				<xacro:ign_joint_state_publisher />
+				<xacro:ign_joint_position_controller />
+			</xacro:unless>
+			<!--			&lt;!&ndash; The sensors used in Ignition are loaded only if a camera is attached &ndash;&gt;-->
+			<!--			<xacro:unless value="${camera == 'none' or mount == 'none'}">-->
+			<!--				<xacro:virtual_sensors />-->
+			<!--				&lt;!&ndash; Since there is already a sensor plugin in the scout, if the scout is loaded-->
+			<!--				the sensor plugin of the igus rebel is not loaded (temporary solution) &ndash;&gt;-->
+			<!--				<xacro:unless value="${load_base}">-->
+			<!--					<xacro:ign_sensor_plugin />-->
+			<!--				</xacro:unless>-->
+			<!--			</xacro:unless>-->
+		</xacro:if>
 		<!-- Include and call rebel macro -->
 		<xacro:include
@@ -12,42 +38,16 @@
 			filename="$(find igus_rebel_description_ros2)/urdf/igus_rebel/igus_rebel.control.xacro" />
 		<xacro:igus_rebel_control hardware_protocol="${hardware_protocol}" />
-		<!-- Mount macros -->
-		<xacro:if value="${mount == 'mount_v1'}">
-			<xacro:include filename="$(find igus_rebel_description_ros2)/urdf/mounts/mount_v1.xacro" />
-			<xacro:mount_v1 end_effector="$(arg end_effector)" />
-		</xacro:if>
-		<xacro:if value="${mount == 'mount_v2'}">
-			<xacro:include filename="$(find igus_rebel_description_ros2)/urdf/mounts/mount_v2.xacro" />
-			<xacro:mount_v2 end_effector="$(arg end_effector)" />
-		</xacro:if>
-		<!-- Camera macro -->
-		<xacro:include filename="$(find igus_rebel_description_ros2)/urdf/cameras/cameras.urdf.xacro" />
-		<xacro:cameras camera="${camera}" load_gazebo="${load_gazebo}" />
-		<!-- Gazebo macro -->
-		<xacro:if value="${load_gazebo}">
-			<xacro:include
-				filename="$(find igus_rebel_description_ros2)/urdf/igus_rebel/igus_rebel.gazebo.xacro" />
-			<!-- The plugin that control the robot in Ignition is loaded if Moveit2 will be used.
-			The Moveit2 controller configuration file is directly passed as a parameter to this plugin -->
-			<xacro:if value="${moveit}">
-				<xacro:ign_ros2_control
-					controller_parameters="$(find igus_rebel_moveit_config)/config/ros2_controllers.yaml" />
-			</xacro:if>
-			<!-- The joint state publisher and the joint position controller are loaded if Moveit2
-			is not used	because the robot is controllable directly from Ignition if some movement are needed -->
-			<xacro:unless value="${moveit}">
-				<xacro:ign_joint_state_publisher />
-				<xacro:ign_joint_position_controller />
-			</xacro:unless>
-			<!-- The sensors used in Ignition are loaded only if a camera is attached -->
-			<xacro:unless value="${camera == 'none' or mount == 'none'}">
-				<xacro:virtual_sensors />
-				<!-- Since there is already a a sensor plugin in the scout, if the scout is loaded
-				the sensor plugin of the igus rebel is not loaded (temporary solution) -->
-				<xacro:unless value="${load_base}">
-					<xacro:ign_sensor_plugin />
-				</xacro:unless>
-			</xacro:unless>
-		</xacro:if>
+<!--		&lt;!&ndash; Mount macros &ndash;&gt;-->
+<!--		<xacro:if value="${mount == 'mount_v1'}">-->
+<!--			<xacro:include filename="$(find igus_rebel_description_ros2)/urdf/mounts/mount_v1.xacro" />-->
+<!--			<xacro:mount_v1 end_effector="$(arg end_effector)" />-->
+<!--		</xacro:if>-->
+<!--		<xacro:if value="${mount == 'mount_v2'}">-->
+<!--			<xacro:include filename="$(find igus_rebel_description_ros2)/urdf/mounts/mount_v2.xacro" />-->
+<!--			<xacro:mount_v2 end_effector="$(arg end_effector)" />-->
+<!--		</xacro:if>-->
+<!--		&lt;!&ndash; Camera macro &ndash;&gt;-->
+<!--		<xacro:include filename="$(find igus_rebel_description_ros2)/urdf/cameras/cameras.urdf.xacro" />-->
+<!--		<xacro:cameras camera="${camera}" load_gazebo="${load_gazebo}" />-->
 	</xacro:macro>
 </robot>

File: igus_rebel_description_ros2/urdf/robot.urdf.xacro (robot description, xacro)
@@ -1,12 +1,4 @@
 <?xml version="1.0"?>
 <robot xmlns:xacro="http://www.ros.org/wiki/xacro" name="igus_rebel">
-	<!-- Scout base selection -->
-	<xacro:arg name="load_base" default="true" />
-	<!-- Mount selection -->
-	<xacro:arg name="mount" default="none" />
-	<!-- Camera type selection -->
-	<xacro:arg name="camera" default="none" />
-	<!-- End effector type selection -->
-	<xacro:arg name="end_effector" default="none" />
 	<!-- Gazebo version -->
 	<xacro:arg name="load_gazebo" default="false" />
@@ -15,50 +7,25 @@
 	<!-- Argument that tells if Moveit2 is used or not -->
 	<xacro:arg name="moveit" default="false" />
-	<!-- odometry source: world ground truth or wheels encoders -->
-	<xacro:arg name="odometry_source" default="ground_truth" />
-	<!-- Set both at 0.0 if collapsing is not interesting in gazebo -->
+	<!-- Set both at 0.0 if collapsing is not interested in gazebo -->
 	<xacro:property name="damping" value="0.0" />
 	<xacro:property name="friction" value="0.0" />
-	<!-- Load mobile robot base, load_base must be true -->
-	<xacro:if value="$(arg load_base)">
-		<!-- virtual joints acting as a link between base_link and igus_rebel_base_link -->
-		<joint name="base_link_to_rebel_support" type="fixed">
-			<parent link="base_link" />
-			<child link="rebel_support" />
-			<origin xyz="-0.28 0.0 0.125" rpy="0 0 ${pi}" />
-		</joint>
-		<link name="rebel_support" />
-		<joint name="rebel_support_to_igus_rebel" type="fixed">
-			<parent link="rebel_support" />
-			<child link="igus_rebel_base_link" />
-			<origin xyz="0.0 0.0 0.0" rpy="0 0 ${-pi/3}" />
-		</joint>
-		<!-- castle with tower mounting sensors, batteries, computer and everyhting else,
-		attached to mobile_robot_base_link
-		set with_basket to false to remove the extra box on the tower
-		-->
-		<xacro:include filename="$(find igus_rebel_description_ros2)/urdf/mobile_robot/castle.urdf" />
-		<xacro:castle with_basket="true" />
-		<!-- load scout robot -->
-		<xacro:include
-			filename="$(find agilex_scout)/urdf/mobile_robot/scout_v2.urdf.xacro" />
-		<xacro:scout_v2
-			load_gazebo="$(arg load_gazebo)" odometry_source="$(arg odometry_source)" />
-	</xacro:if>
-	<!-- Add base_link attachment when no mobile robot is loaded -->
-	<xacro:unless value="$(arg load_base)">
-		<link name="base_link" />
-		<joint name="base_link_to_igus_rebel" type="fixed">
-			<parent link="base_link" />
-			<child link="igus_rebel_base_link" />
-			<origin xyz="0.0 0.0 0.0" rpy="0.0 0.0 0.0" />
-		</joint>
-	</xacro:unless>
+    <xacro:if value="$(arg load_gazebo)">
+        <link name="world" />
+        <joint name="world_joint" type="fixed">
+            <parent link="world" />
+            <child link="base_link" />
+        </joint>
+    </xacro:if>
+	<link name="base_link" />
+	<joint name="base_link_to_igus_rebel" type="fixed">
+		<parent link="base_link" />
+		<child link="igus_rebel_base_link" />
+		<origin xyz="0.0 0.0 0.0" rpy="0.0 0.0 0.0" />
+	</joint>
 	<!-- load igus rebel with camera gripper and castle -->
 	<xacro:include
 		filename="$(find igus_rebel_description_ros2)/urdf/igus_rebel/igus_rebel.urdf.xacro" />
 	<xacro:igus_rebel
-		load_base="$(arg load_base)" mount="$(arg mount)" camera="$(arg camera)"
-		end_effector="$(arg end_effector)" hardware_protocol="$(arg hardware_protocol)"
+		hardware_protocol="$(arg hardware_protocol)"
 		load_gazebo="$(arg load_gazebo)" moveit="$(arg moveit)" />
 </robot>

File: igus_rebel_moveit_config/config/igus_rebel.srdf.xacro (robot description, xacro)
@@ -1,61 +1,18 @@
 <?xml version="1.0"?>
 <robot xmlns:xacro="http://wiki.ros.org/xacro" name="igus_rebel">
-	<!-- Arguments -->
-	<xacro:arg name="load_base" default="false" />
-	<xacro:arg name="mount" default="none" />
-	<xacro:arg name="camera" default="none" />
-	<xacro:arg name="end_effector" default="none" />
 	<!-- macro xacro definition to load mount and mobile robot base -->
-	<xacro:macro name="srdf" params="mount camera end_effector load_base">
+	<xacro:macro name="srdf">
 		<!--############################################################################### -->
 		<!-- 				Planning Groups Definitions and End Effectors					-->
 		<!--############################################################################### -->
 		<!-- If mount is not placed, naked robot -->
-		<xacro:if value="${mount == 'none'}">
-			<group name="rebel_arm">
-				<chain base_link="igus_rebel_base_link" tip_link="link_8" />
-			</group>
-			<group name="flange_group">
-				<link name="flange" />
-			</group>
-			<end_effector name="flange_EEF" parent_link="link_8" group="flange_group"
-				parent_group="rebel_arm" />
-		</xacro:if>
-		<!-- If mount is placed -->
-		<xacro:if value="${mount != 'none'}">
-			<!-- If camera is relasense or oakd and no end effector placed -->
-			<xacro:if value="${end_effector == 'none'}">
-				<group name="rebel_arm">
-					<chain base_link="igus_rebel_base_link" tip_link="flange" />
-				</group>
-				<end_effector name="flange_EEF" parent_link="flange"
-					group="rebel_arm" />
-			</xacro:if>
-			<!-- If camera is realsense or oakd and toucher v1 is placed -->
-			<xacro:if value="${end_effector == 'toucher_v1'}">
-				<group name="rebel_arm">
-					<chain base_link="igus_rebel_base_link" tip_link="toucher_endpoint" />
-				</group>
-				<group name="toucher_v1_group">
-					<link name="toucher_v1" />
-					<link name="toucher_endpoint" />
-				</group>
-				<end_effector name="toucher_v1_EEF" parent_link="toucher_endpoint"
-					group="toucher_v1_group" parent_group="rebel_arm" />
-			</xacro:if>
-			<!-- If camera is realsense and soft gripper is placed -->
-			<xacro:if value="${end_effector == 'soft_gripper'}">
-				<group name="rebel_arm">
-					<chain base_link="igus_rebel_base_link" tip_link="soft_gripper_tip_link" />
-				</group>
-				<group name="soft_gripper_group">
-					<link name="soft_gripper_mount" />
-					<link name="soft_gripper_link" />
-					<link name="soft_gripper_tip_link" />
-				</group>
-				<end_effector name="soft_gripper_EEF" parent_link="soft_gripper_tip_link"
-					group="soft_gripper_group" parent_group="rebel_arm" />
-			</xacro:if>
-		</xacro:if>
+		<group name="rebel_arm">
+			<chain base_link="igus_rebel_base_link" tip_link="link_8" />
+		</group>
+		<group name="flange_group">
+			<link name="flange" />
+		</group>
+		<end_effector name="flange_EEF" parent_link="link_8" group="flange_group"
+			parent_group="rebel_arm" />
 		<!--############################################################################### -->
 		<!-- 				Planning Groups states 											-->
@@ -104,136 +61,6 @@
 		<disable_collisions link1="link_6" link2="link_8" reason="Never" />
 		<disable_collisions link1="link_7" link2="link_8" reason="Adjacent" />
-		<!-- Collisions checks due to the presence of the scout base -->
-		<xacro:if value="${load_base}">
-			<!-- Default collision checks for base robot and scout. The collision between the scout
-			and the mount are all enabled-->
-			<disable_collisions link1="front_left_wheel_link" link2="front_right_wheel_link"
-				reason="Never" />
-			<disable_collisions link1="front_left_wheel_link" link2="igus_rebel_base_link"
-				reason="Never" />
-			<disable_collisions link1="front_left_wheel_link" link2="link_1" reason="Never" />
-			<disable_collisions link1="front_left_wheel_link" link2="link_2" reason="Never" />
-			<disable_collisions link1="front_left_wheel_link" link2="link_5" reason="Never" />
-			<disable_collisions link1="front_left_wheel_link" link2="mobile_robot_base_link"
-				reason="Adjacent" />
-			<disable_collisions link1="front_left_wheel_link" link2="rear_left_wheel_link"
-				reason="Never" />
-			<disable_collisions link1="front_left_wheel_link" link2="rear_right_wheel_link"
-				reason="Never" />
-			<disable_collisions link1="front_left_wheel_link" link2="tower_link" reason="Never" />
-			<disable_collisions link1="front_right_wheel_link" link2="igus_rebel_base_link"
-				reason="Never" />
-			<disable_collisions link1="front_right_wheel_link" link2="link_1" reason="Never" />
-			<disable_collisions link1="front_right_wheel_link" link2="link_2" reason="Never" />
-			<disable_collisions link1="front_right_wheel_link" link2="link_5" reason="Never" />
-			<disable_collisions link1="front_right_wheel_link" link2="mobile_robot_base_link"
-				reason="Adjacent" />
-			<disable_collisions link1="front_right_wheel_link" link2="rear_left_wheel_link"
-				reason="Never" />
-			<disable_collisions link1="front_right_wheel_link" link2="rear_right_wheel_link"
-				reason="Never" />
-			<disable_collisions link1="front_right_wheel_link" link2="tower_link" reason="Never" />
-			<disable_collisions link1="igus_rebel_base_link" link2="mobile_robot_base_link"
-				reason="Adjacent" />
-			<disable_collisions link1="igus_rebel_base_link" link2="rear_left_wheel_link"
-				reason="Never" />
-			<disable_collisions link1="igus_rebel_base_link" link2="rear_right_wheel_link"
-				reason="Never" />
-			<disable_collisions link1="igus_rebel_base_link" link2="tower_link" reason="Never" />
-			<disable_collisions link1="link_1" link2="mobile_robot_base_link" reason="Never" />
-			<disable_collisions link1="link_1" link2="rear_left_wheel_link" reason="Never" />
-			<disable_collisions link1="link_1" link2="rear_right_wheel_link" reason="Never" />
-			<disable_collisions link1="link_1" link2="tower_link" reason="Never" />
-			<disable_collisions link1="link_2" link2="mobile_robot_base_link" reason="Never" />
-			<disable_collisions link1="link_2" link2="rear_left_wheel_link" reason="Never" />
-			<disable_collisions link1="link_2" link2="rear_right_wheel_link" reason="Never" />
-			<disable_collisions link1="mobile_robot_base_link" link2="rear_left_wheel_link"
-				reason="Adjacent" />
-			<disable_collisions link1="mobile_robot_base_link" link2="rear_right_wheel_link"
-				reason="Adjacent" />
-			<disable_collisions link1="mobile_robot_base_link" link2="tower_link" reason="Adjacent" />
-			<disable_collisions link1="rear_left_wheel_link" link2="rear_right_wheel_link"
-				reason="Never" />
-			<disable_collisions link1="rear_left_wheel_link" link2="tower_link" reason="Never" />
-			<disable_collisions link1="rear_right_wheel_link" link2="tower_link" reason="Never" />
-		</xacro:if>
-		<!-- Collision checks due to the presence of the mount -->
-		<xacro:if value="${mount == 'mount_v1' or mount == 'mount_v2'}">
-			<disable_collisions link1="link_5" link2="camera_mount" reason="Never" />
-			<disable_collisions link1="link_6" link2="camera_mount" reason="Never" />
-			<disable_collisions link1="link_7" link2="camera_mount" reason="Never" />
-			<disable_collisions link1="link_8" link2="camera_mount" reason="Adjacent" />
-			<xacro:if value="${camera == 'oakd' and end_effector == 'none'}">
-				<disable_collisions link1="camera_mount" link2="camera_link" reason="Adjacent" />
-				<disable_collisions link1="link_5" link2="camera_link" reason="Never" />
-				<disable_collisions link1="link_6" link2="camera_link" reason="Never" />
-				<disable_collisions link1="link_7" link2="camera_link" reason="Never" />
-				<disable_collisions link1="link_8" link2="camera_link" reason="Never" />
-			</xacro:if>
-			<xacro:if value="${camera == 'realsense' and end_effector == 'none'}">
-				<disable_collisions link1="camera_mount" link2="camera_link" reason="Adjacent" />
-				<disable_collisions link1="link_5" link2="camera_link" reason="Never" />
-				<disable_collisions link1="link_6" link2="camera_link" reason="Never" />
-				<disable_collisions link1="link_7" link2="camera_link" reason="Never" />
-				<disable_collisions link1="link_8" link2="camera_link" reason="Never" />
-			</xacro:if>
-			<xacro:if value="${camera == 'none' and end_effector == 'toucher_v1'}">
-				<disable_collisions link1="camera_mount" link2="toucher_v1" reason="Adjacent" />
-				<disable_collisions link1="link_2" link2="toucher_v1" reason="Never" />
-				<disable_collisions link1="link_5" link2="toucher_v1" reason="Never" />
-				<disable_collisions link1="link_6" link2="toucher_v1" reason="Never" />
-				<disable_collisions link1="link_7" link2="toucher_v1" reason="Never" />
-				<disable_collisions link1="link_8" link2="toucher_v1" reason="Default" />
-			</xacro:if>
-			<xacro:if value="${camera == 'oakd' and end_effector == 'toucher_v1'}">
-				<disable_collisions link1="camera_mount" link2="camera_link" reason="Adjacent" />
-				<disable_collisions link1="link_5" link2="camera_link" reason="Never" />
-				<disable_collisions link1="link_6" link2="camera_link" reason="Never" />
-				<disable_collisions link1="link_7" link2="camera_link" reason="Never" />
-				<disable_collisions link1="link_8" link2="camera_link" reason="Never" />
-				<disable_collisions link1="camera_mount" link2="toucher_v1" reason="Adjacent" />
-				<disable_collisions link1="link_2" link2="toucher_v1" reason="Never" />
-				<disable_collisions link1="link_5" link2="toucher_v1" reason="Never" />
-				<disable_collisions link1="link_6" link2="toucher_v1" reason="Never" />
-				<disable_collisions link1="link_7" link2="toucher_v1" reason="Never" />
-				<disable_collisions link1="link_8" link2="toucher_v1" reason="Default" />
-				<disable_collisions link1="camera_link" link2="toucher_v1" reason="Never" />
-			</xacro:if>
-			<xacro:if value="${camera == 'realsense' and end_effector == 'toucher_v1'}">
-				<disable_collisions link1="camera_mount" link2="camera_link" reason="Adjacent" />
-				<disable_collisions link1="link_5" link2="camera_link" reason="Never" />
-				<disable_collisions link1="link_6" link2="camera_link" reason="Never" />
-				<disable_collisions link1="link_7" link2="camera_link" reason="Never" />
-				<disable_collisions link1="link_8" link2="camera_link" reason="Never" />
-				<disable_collisions link1="camera_mount" link2="toucher_v1" reason="Adjacent" />
-				<disable_collisions link1="link_2" link2="toucher_v1" reason="Never" />
-				<disable_collisions link1="link_5" link2="toucher_v1" reason="Never" />
-				<disable_collisions link1="link_6" link2="toucher_v1" reason="Never" />
-				<disable_collisions link1="link_7" link2="toucher_v1" reason="Never" />
-				<disable_collisions link1="link_8" link2="toucher_v1" reason="Default" />
-				<disable_collisions link1="camera_link" link2="toucher_v1" reason="Never" />
-			</xacro:if>
-			<xacro:if value="${camera == 'realsense' and end_effector == 'soft_gripper'}">
-				<disable_collisions link1="camera_mount" link2="camera_link" reason="Adjacent" />
-				<disable_collisions link1="link_7" link2="camera_link" reason="Never" />
-				<disable_collisions link1="link_8" link2="camera_link" reason="Never" />
-				<disable_collisions link1="link_7" link2="camera_mount" reason="Adjacent" />
-				<disable_collisions link1="link_8" link2="camera_mount" reason="Adjacent" />
-				<disable_collisions link1="camera_mount" link2="soft_gripper_link" reason="Adjacent" />
-				<disable_collisions link1="camera_mount" link2="soft_gripper_mount"
-					reason="Adjacent" />
-				<disable_collisions link1="camera_link" link2="soft_gripper_mount" reason="Never" />
-				<disable_collisions link1="camera_link" link2="soft_gripper_link" reason="Never" />
-				<disable_collisions link1="link_7" link2="soft_gripper_link" reason="Never" />
-				<disable_collisions link1="link_8" link2="soft_gripper_link" reason="Never" />
-				<disable_collisions link1="link_7" link2="soft_gripper_mount" reason="Never" />
-				<disable_collisions link1="link_8" link2="soft_gripper_mount" reason="Never" />
-				<disable_collisions link1="soft_gripper_mount" link2="soft_gripper_link"
-					reason="Adjacent" />
-			</xacro:if>
-		</xacro:if>
 	</xacro:macro>
 	<!-- Call the macro and define the arguments -->
-	<xacro:srdf mount="$(arg mount)" camera="$(arg camera)" end_effector="$(arg end_effector)"
-		load_base="$(arg load_base)" />
+	<xacro:srdf />
 </robot>
