Commit message: modified URDF and XACROs definitions for mobile robot unified TF tree

File: igus_rebel_description_ros2/urdf/igus_rebel/igus_rebel.description.xacro (robot description, xacro)
@@ -2,13 +2,15 @@
 <robot xmlns:xacro="http://www.ros.org/wiki/xacro" name="igus_rebel">
 	<xacro:macro name="igus_rebel_description">
-		<link name="base_link">
-			<visual>
-				<geometry>
-					<mesh filename="file://$(find igus_rebel_description_ros2)/meshes/new/Joint0.dae" />
-				</geometry>
-			</visual>
-			<collision>
-				<geometry>
-					<mesh filename="file://$(find igus_rebel_description_ros2)/meshes/new/Joint0.dae" />
+		<link name="igus_rebel_base_link">
+			<visual>
+				<geometry>
+					<mesh
+						filename="file://$(find igus_rebel_description_ros2)/meshes/new/Joint0.dae" />
+				</geometry>
+			</visual>
+			<collision>
+				<geometry>
+					<mesh
+						filename="file://$(find igus_rebel_description_ros2)/meshes/new/Joint0.dae" />
 				</geometry>
 			</collision>
@@ -19,20 +21,23 @@
 		</link>
 		<joint name="joint1" type="revolute">
-			<parent link="base_link" />
+			<parent link="igus_rebel_base_link" />
 			<child link="link_1" />
 			<origin rpy="0.0 0.0 0.0" xyz="0.0 0 0.100" />
 			<axis xyz="0 0 1" />
-			<limit effort="330.0" lower="${-pi*179/180}" upper="${pi*179/180}" velocity="${pi*45/180}" />
+			<limit effort="330.0" lower="${-pi*179/180}" upper="${pi*179/180}"
+				velocity="${pi*45/180}" />
 		</joint>
 		<link name="link_1">
 			<visual>
 				<geometry>
-					<mesh filename="file://$(find igus_rebel_description_ros2)/meshes/new/Joint1.dae" />
-				</geometry>
-				<origin rpy="0 0 0" xyz="0 0 0" />
-			</visual>
-			<collision>
-				<geometry>
-					<mesh filename="file://$(find igus_rebel_description_ros2)/meshes/new/Joint1.dae" />
+					<mesh
+						filename="file://$(find igus_rebel_description_ros2)/meshes/new/Joint1.dae" />
+				</geometry>
+				<origin rpy="0 0 0" xyz="0 0 0" />
+			</visual>
+			<collision>
+				<geometry>
+					<mesh
+						filename="file://$(find igus_rebel_description_ros2)/meshes/new/Joint1.dae" />
 				</geometry>
 				<origin rpy="0 0 0" xyz="0 0 0" />
@@ -48,5 +53,6 @@
 			<origin rpy="0.0 ${pi/6} 0.0" xyz="0.0 0 0.149" />
 			<axis xyz="0 1 0" />
-			<!-- pi*2/3 are the physical limits, but to avoid any collisions we set the actual limits lower -->
+			<!-- pi*2/3 are the physical limits, but to avoid any collisions we set the actual
+			limits lower -->
 			<limit effort="330.0" lower="${-pi*11/18}" upper="${pi*11/18}" velocity="${pi*45/180}" />
 		</joint>
@@ -54,11 +60,13 @@
 			<visual>
 				<geometry>
-					<mesh filename="file://$(find igus_rebel_description_ros2)/meshes/new/Joint2.dae" />
-				</geometry>
-				<origin rpy="0 0 0" xyz="0 0 0" />
-			</visual>
-			<collision>
-				<geometry>
-					<mesh filename="file://$(find igus_rebel_description_ros2)/meshes/new/Joint2.dae" />
+					<mesh
+						filename="file://$(find igus_rebel_description_ros2)/meshes/new/Joint2.dae" />
+				</geometry>
+				<origin rpy="0 0 0" xyz="0 0 0" />
+			</visual>
+			<collision>
+				<geometry>
+					<mesh
+						filename="file://$(find igus_rebel_description_ros2)/meshes/new/Joint2.dae" />
 				</geometry>
 				<origin rpy="0 0 0" xyz="0 0 0" />
@@ -74,5 +82,6 @@
 			<origin rpy="0.0 ${pi/6} 0.0" xyz="0.0 0.0 0.2384" />
 			<axis xyz="0 1 0" />
-			<!-- pi*2/3 are the physical limits, but to avoid any collisions we set the actual limits lower -->
+			<!-- pi*2/3 are the physical limits, but to avoid any collisions we set the actual
+			limits lower -->
 			<limit effort="330.0" lower="${-pi*11/18}" upper="${pi*11/18}" velocity="${pi*45/180}" />
 		</joint>
@@ -80,11 +89,13 @@
 			<visual>
 				<geometry>
-					<mesh filename="file://$(find igus_rebel_description_ros2)/meshes/new/Joint3.dae" />
-				</geometry>
-				<origin rpy="0 0 0" xyz="0 0 0" />
-			</visual>
-			<collision>
-				<geometry>
-					<mesh filename="file://$(find igus_rebel_description_ros2)/meshes/new/Joint3.dae" />
+					<mesh
+						filename="file://$(find igus_rebel_description_ros2)/meshes/new/Joint3.dae" />
+				</geometry>
+				<origin rpy="0 0 0" xyz="0 0 0" />
+			</visual>
+			<collision>
+				<geometry>
+					<mesh
+						filename="file://$(find igus_rebel_description_ros2)/meshes/new/Joint3.dae" />
 				</geometry>
 				<origin rpy="0 0 0" xyz="0 0 0" />
@@ -101,16 +112,19 @@
 			<origin rpy="0.0 0.0 0.0" xyz="0.0 0 ${0.149 - 0.03}" />
 			<axis xyz="0 0 1" />
-			<limit effort="330.0" lower="${-pi*179/180}" upper="${pi*179/180}" velocity="${pi*45/180}" />
+			<limit effort="330.0" lower="${-pi*179/180}" upper="${pi*179/180}"
+				velocity="${pi*45/180}" />
 		</joint>
 		<link name="link_6">
 			<visual>
 				<geometry>
-					<mesh filename="file://$(find igus_rebel_description_ros2)/meshes/new/Joint4.dae" />
-				</geometry>
-				<origin rpy="0 0 0" xyz="0 0 0" />
-			</visual>
-			<collision>
-				<geometry>
-					<mesh filename="file://$(find igus_rebel_description_ros2)/meshes/new/Joint4.dae" />
+					<mesh
+						filename="file://$(find igus_rebel_description_ros2)/meshes/new/Joint4.dae" />
+				</geometry>
+				<origin rpy="0 0 0" xyz="0 0 0" />
+			</visual>
+			<collision>
+				<geometry>
+					<mesh
+						filename="file://$(find igus_rebel_description_ros2)/meshes/new/Joint4.dae" />
 				</geometry>
 				<origin rpy="0 0 0" xyz="0 0 0" />
@@ -127,16 +141,19 @@
 			<origin rpy="0.0 ${-pi/24} 0.0" xyz="0.0 0 ${0.14 + 0.03}" />
 			<axis xyz="0 1 0" />
-			<limit effort="330.0" lower="${-pi*19/36 + pi/24}" upper="${pi*19/36 + pi/24}" velocity="${pi*45/180}" />
+			<limit effort="330.0" lower="${-pi*19/36 + pi/24}" upper="${pi*19/36 + pi/24}"
+				velocity="${pi*45/180}" />
 		</joint>
 		<link name="link_7">
 			<visual>
 				<geometry>
-					<mesh filename="file://$(find igus_rebel_description_ros2)/meshes/new/Joint5.dae" />
-				</geometry>
-				<origin rpy="0 0 0" xyz="0 0 0" />
-			</visual>
-			<collision>
-				<geometry>
-					<mesh filename="file://$(find igus_rebel_description_ros2)/meshes/new/Joint5.dae" />
+					<mesh
+						filename="file://$(find igus_rebel_description_ros2)/meshes/new/Joint5.dae" />
+				</geometry>
+				<origin rpy="0 0 0" xyz="0 0 0" />
+			</visual>
+			<collision>
+				<geometry>
+					<mesh
+						filename="file://$(find igus_rebel_description_ros2)/meshes/new/Joint5.dae" />
 				</geometry>
 				<origin rpy="0 0 0" xyz="0 0 0" />
@@ -152,10 +169,12 @@
 			<origin rpy="0.0 0.0 0.0" xyz="0.0 0 0.1208" />
 			<axis xyz="0 0 1" />
-			<limit effort="330.0" lower="${-pi*179/180}" upper="${pi*179/180}" velocity="${pi*45/180}" />
+			<limit effort="330.0" lower="${-pi*179/180}" upper="${pi*179/180}"
+				velocity="${pi*45/180}" />
 		</joint>
 		<link name="link_8">
 			<visual>
 				<geometry>
-					<mesh filename="file://$(find igus_rebel_description_ros2)/meshes/new/Joint6.dae" />
+					<mesh
+						filename="file://$(find igus_rebel_description_ros2)/meshes/new/Joint6.dae" />
 				</geometry>
 				<origin rpy="0 0 0" xyz="0.0 0 0" />
@@ -163,5 +182,6 @@
 			<collision>
 				<geometry>
-					<mesh filename="file://$(find igus_rebel_description_ros2)/meshes/new/Joint6.dae" />
+					<mesh
+						filename="file://$(find igus_rebel_description_ros2)/meshes/new/Joint6.dae" />
 				</geometry>
 				<origin rpy="0 0 0" xyz="0.0 0 0" />

File: igus_rebel_description_ros2/urdf/igus_rebel/igus_rebel_mod.description.xacro (robot description, xacro)
@@ -2,5 +2,5 @@
 <robot xmlns:xacro="http://www.ros.org/wiki/xacro" name="igus_rebel_mod">
 	<xacro:macro name="igus_rebel_mod_description" params="hardware_protocol">
-		<link name="base_link">
+		<link name="igus_rebel_base_link">
 			<visual>
 				<geometry>
@@ -19,5 +19,5 @@
 		</link>
 		<joint name="joint1" type="revolute">
-			<parent link="base_link" />
+			<parent link="igus_rebel_base_link" />
 			<child link="link_1" />
 			<origin rpy="0.0 0.0 ${pi}" xyz="0.0 0.0 0.126" />

File: igus_rebel_description_ros2/urdf/igus_rebel/igus_rebel_mod.urdf.xacro (robot description, xacro)
@@ -2,18 +2,16 @@
 <robot xmlns:xacro="http://www.ros.org/wiki/xacro" name="igus_rebel_mod">
 	<!-- Controller settings, only enable a single one in the launch file -->
-	<xacro:arg name="hardware_protocol" default="cri" />
+	<xacro:arg name="hardware_protocol" default="simulation" />
 	<!-- Gripper selection -->
 	<xacro:arg name="gripper" default="none" />
 	<!-- Include and call rebel macro -->
-	<xacro:include filename="$(find igus_rebel_description_ros2)/urdf/igus_rebel_mod.description.xacro" />
+	<xacro:include filename="$(find igus_rebel_description_ros2)/urdf/igus_rebel/igus_rebel_mod.description.xacro" />
 	<xacro:igus_rebel_mod_description hardware_protocol="$(arg hardware_protocol)" />
 	<!-- controller macro -->
-	<xacro:include filename="$(find igus_rebel_description_ros2)/urdf/igus_rebel.control.xacro" />
+	<xacro:include filename="$(find igus_rebel_description_ros2)/urdf/igus_rebel/igus_rebel.control.xacro" />
 	<xacro:igus_rebel_control hardware_protocol="$(arg hardware_protocol)"/>
-	<!-- Add world link -->
-	<link name="world" />
-	<joint name="world_to_base" type="fixed">
-		<parent link="world" />
-		<child link="base_link" />
+	<joint name="base_link_to_igus_rebel" type="fixed">
+		<parent link="base_link" />
+		<child link="igus_rebel_base_link" />
 		<origin xyz="0.0 0.0 0.0" rpy="0.0 0.0 0.0" />
 	</joint>

File: igus_rebel_moveit_config/config/igus_rebel.srdf.xacro (robot description, xacro)
@@ -1,4 +1,20 @@
 <?xml version="1.0"?>
 <robot xmlns:xacro="http://wiki.ros.org/xacro" name="igus_rebel">
+	<!--GROUPS:
+	Representation of a set of joints and links. This can be useful for specifying DOF to plan for,
+	defining arms, end effectors, etc-->
+	<!--LINKS:
+	When a link is specified, the parent joint of that link (if it exists) is automatically
+	included-->
+	<!--JOINTS:
+	When a joint is specified, the child link of that joint (which will always exist) is
+	automatically included-->
+	<!--CHAINS:
+	When a chain is specified, all the links along the chain (including endpoints) are included in
+	the group. Additionally, all the joints that are parents to included links are also included.
+	This means that joints along the chain and the parent joint of the base link are included in the
+	group-->
+	<!--SUBGROUPS:
+	Groups can also be formed by referencing to already defined group names-->
 	<!-- disable collisions between a link and the robot scout and tower -->
 	<xacro:macro name="no_collision_scout" params="link">
@@ -23,5 +39,5 @@
 		<!-- common definitions -->
 		<group name="rebel_arm">
-			<link name="base_link" />
+			<link name="igus_rebel_base_link" />
 			<link name="link_1" />
 			<link name="link_2" />
@@ -31,67 +47,66 @@
 			<link name="link_8" />
 		</group>
+		<group name="chain_arm">
+			<chain base_link="igus_rebel_base_link" tip_link="link_8" />
+		</group>
 		<!-- no grippers installed => end effector placed on link_8 -->
 		<xacro:if value="${gripper == 'none'}">
-			<group name="chain_arm">
-				<chain base_link="base_link" tip_link="link_8" />
-			</group>
-			<end_effector name="manipulator" parent_link="link_8" group="rebel_arm" parent_group="chain_arm" />
+			<end_effector name="manipulator" parent_link="link_8" group="rebel_arm"
+				parent_group="chain_arm" />
+			<!-- default positions common for every configuration -->
+			<group_state name="zero" group="chain_arm">
+				<joint name="joint1" value="0" />
+				<joint name="joint2" value="0" />
+				<joint name="joint3" value="0" />
+				<joint name="joint4" value="0" />
+				<joint name="joint5" value="0" />
+				<joint name="joint6" value="0" />
+			</group_state>
+			<group_state name="home" group="chain_arm">
+				<joint name="joint1" value="0" />
+				<joint name="joint2" value="${-pi/6.0}" />
+				<joint name="joint3" value="${-pi/6.0}" />
+				<joint name="joint4" value="0" />
+				<joint name="joint5" value="${pi/24.0}" />
+				<joint name="joint6" value="0" />
+			</group_state>
 		</xacro:if>
 		<!-- if camera is placed => end effector on toucher link -->
 		<xacro:if value="${gripper == 'camera'}">
 			<group name="camera">
-				<link name="flange" />
-				<joint name="flange_to_mount" />
+				<link name="camera_link" />
 				<link name="camera_mount" />
-				<joint name="mount_to_cam" />
-				<link name="camera_insert" />
+				<link name="camera_usb_plug_link" />
 				<link name="toucher" />
-				<joint name="flange_to_toucher" />
 			</group>
 			<group name="chain_arm_manipulator">
-				<chain base_link="base_link" tip_link="toucher" />
+				<chain base_link="igus_rebel_base_link" tip_link="toucher" />
 			</group>
-			<end_effector name="manipulator" parent_link="toucher" group="chain_arm_manipulator"
-				parent_group="camera" />
-		</xacro:if>
-		<!-- default positions common for every configuration -->
-		<group_state name="zero" group="rebel_arm">
-			<joint name="joint1" value="0" />
-			<joint name="joint2" value="0" />
-			<joint name="joint3" value="0" />
-			<joint name="joint4" value="0" />
-			<joint name="joint5" value="0" />
-			<joint name="joint6" value="0" />
-		</group_state>
-		<group_state name="home" group="rebel_arm">
-			<joint name="joint1" value="0" />
-			<joint name="joint2" value="${-pi/6.0}" />
-			<joint name="joint3" value="${-pi/6.0}" />
-			<joint name="joint4" value="0" />
-			<joint name="joint5" value="${pi/24.0}" />
-			<joint name="joint6" value="0" />
-		</group_state>
-		<group_state name="zero" group="chain_arm_manipulator">
-			<joint name="joint1" value="0" />
-			<joint name="joint2" value="0" />
-			<joint name="joint3" value="0" />
-			<joint name="joint4" value="0" />
-			<joint name="joint5" value="0" />
-			<joint name="joint6" value="0" />
-		</group_state>
-		<group_state name="home" group="chain_arm_manipulator">
-			<joint name="joint1" value="0" />
-			<joint name="joint2" value="${-pi/6.0}" />
-			<joint name="joint3" value="${-pi/6.0}" />
-			<joint name="joint4" value="0" />
-			<joint name="joint5" value="${pi/24.0}" />
-			<joint name="joint6" value="0" />
-		</group_state>
+			<end_effector name="manipulator" parent_link="toucher" group="chain_arm_manipulator" parent_group="camera" />
+			<group_state name="zero" group="chain_arm_manipulator">
+				<joint name="joint1" value="0" />
+				<joint name="joint2" value="0" />
+				<joint name="joint3" value="0" />
+				<joint name="joint4" value="0" />
+				<joint name="joint5" value="0" />
+				<joint name="joint6" value="0" />
+			</group_state>
+			<group_state name="home" group="chain_arm_manipulator">
+				<joint name="joint1" value="0" />
+				<joint name="joint2" value="${-pi/6.0}" />
+				<joint name="joint3" value="${-pi/6.0}" />
+				<joint name="joint4" value="0" />
+				<joint name="joint5" value="${pi/24.0}" />
+				<joint name="joint6" value="0" />
+			</group_state>
+		</xacro:if>
 		<!--TODO:
 		add parking position -->
-		<virtual_joint name="world_to_base" type="fixed" parent_frame="world" child_link="base_link" />
+		<!--<virtual_joint
+		name="world_to_base" type="fixed" parent_frame="world" child_link="base_link" />-->
 		<!-- default collision checks for base robot -->
-		<disable_collisions link1="base_link" link2="link_1" reason="Adjacent" />
-		<disable_collisions link1="base_link" link2="link_2" reason="Never" />
+		<disable_collisions link1="base_link" link2="igus_rebel_base_link" reason="Adjacent" />
+		<disable_collisions link1="igus_rebel_base_link" link2="link_1" reason="Adjacent" />
+		<disable_collisions link1="igus_rebel_base_link" link2="link_2" reason="Never" />
 		<disable_collisions link1="link_1" link2="link_2" reason="Adjacent" />
 		<disable_collisions link1="link_2" link2="link_5" reason="Adjacent" />
@@ -112,5 +127,5 @@
 			<disable_collisions link1="camera_link" link2="toucher" reason="Never" />
 			<disable_collisions link1="camera_mount" link2="toucher" reason="Never" />
-			<xacro:no_collision_camera link="base_link" />
+			<xacro:no_collision_camera link="igus_rebel_base_link" />
 			<xacro:no_collision_camera link="link_1" />
 			<xacro:no_collision_camera link="link_2" />
@@ -134,24 +149,36 @@
 				<link name="tower_link" />
 			</group>
-			<disable_collisions link1="base_link" link2="front_left_wheel_link" reason="Never" />
-			<disable_collisions link1="base_link" link2="front_right_wheel_link" reason="Never" />
-			<disable_collisions link1="base_link" link2="mobile_robot_base_link" reason="Adjacent" />
-			<disable_collisions link1="base_link" link2="rear_left_wheel_link" reason="Never" />
-			<disable_collisions link1="base_link" link2="rear_right_wheel_link" reason="Never" />
-			<disable_collisions link1="base_link" link2="tower_link" reason="Never" />
-			<disable_collisions link1="front_left_wheel_link" link2="front_right_wheel_link" reason="Never" />
+			<disable_collisions link1="igus_rebel_base_link" link2="front_left_wheel_link"
+				reason="Never" />
+			<disable_collisions link1="igus_rebel_base_link" link2="front_right_wheel_link"
+				reason="Never" />
+			<disable_collisions link1="igus_rebel_base_link" link2="mobile_robot_base_link"
+				reason="Adjacent" />
+			<disable_collisions link1="igus_rebel_base_link" link2="rear_left_wheel_link"
+				reason="Never" />
+			<disable_collisions link1="igus_rebel_base_link" link2="rear_right_wheel_link"
+				reason="Never" />
+			<disable_collisions link1="igus_rebel_base_link" link2="tower_link" reason="Never" />
+			<disable_collisions link1="front_left_wheel_link" link2="front_right_wheel_link"
+				reason="Never" />
 			<disable_collisions link1="front_left_wheel_link" link2="link_1" reason="Never" />
 			<disable_collisions link1="front_left_wheel_link" link2="link_2" reason="Never" />
 			<disable_collisions link1="front_left_wheel_link" link2="link_5" reason="Never" />
-			<disable_collisions link1="front_left_wheel_link" link2="mobile_robot_base_link" reason="Adjacent" />
-			<disable_collisions link1="front_left_wheel_link" link2="rear_left_wheel_link" reason="Never" />
-			<disable_collisions link1="front_left_wheel_link" link2="rear_right_wheel_link" reason="Never" />
+			<disable_collisions link1="front_left_wheel_link" link2="mobile_robot_base_link"
+				reason="Adjacent" />
+			<disable_collisions link1="front_left_wheel_link" link2="rear_left_wheel_link"
+				reason="Never" />
+			<disable_collisions link1="front_left_wheel_link" link2="rear_right_wheel_link"
+				reason="Never" />
 			<disable_collisions link1="front_left_wheel_link" link2="tower_link" reason="Never" />
 			<disable_collisions link1="front_right_wheel_link" link2="link_1" reason="Never" />
 			<disable_collisions link1="front_right_wheel_link" link2="link_2" reason="Never" />
 			<disable_collisions link1="front_right_wheel_link" link2="link_5" reason="Never" />
-			<disable_collisions link1="front_right_wheel_link" link2="mobile_robot_base_link" reason="Adjacent" />
-			<disable_collisions link1="front_right_wheel_link" link2="rear_left_wheel_link" reason="Never" />
-			<disable_collisions link1="front_right_wheel_link" link2="rear_right_wheel_link" reason="Never" />
+			<disable_collisions link1="front_right_wheel_link" link2="mobile_robot_base_link"
+				reason="Adjacent" />
+			<disable_collisions link1="front_right_wheel_link" link2="rear_left_wheel_link"
+				reason="Never" />
+			<disable_collisions link1="front_right_wheel_link" link2="rear_right_wheel_link"
+				reason="Never" />
 			<disable_collisions link1="front_right_wheel_link" link2="tower_link" reason="Never" />
 			<disable_collisions link1="link_1" link2="mobile_robot_base_link" reason="Never" />
@@ -162,8 +189,11 @@
 			<disable_collisions link1="link_2" link2="rear_left_wheel_link" reason="Never" />
 			<disable_collisions link1="link_2" link2="rear_right_wheel_link" reason="Never" />
-			<disable_collisions link1="mobile_robot_base_link" link2="rear_left_wheel_link" reason="Adjacent" />
-			<disable_collisions link1="mobile_robot_base_link" link2="rear_right_wheel_link" reason="Adjacent" />
+			<disable_collisions link1="mobile_robot_base_link" link2="rear_left_wheel_link"
+				reason="Adjacent" />
+			<disable_collisions link1="mobile_robot_base_link" link2="rear_right_wheel_link"
+				reason="Adjacent" />
 			<disable_collisions link1="mobile_robot_base_link" link2="tower_link" reason="Adjacent" />
-			<disable_collisions link1="rear_left_wheel_link" link2="rear_right_wheel_link" reason="Never" />
+			<disable_collisions link1="rear_left_wheel_link" link2="rear_right_wheel_link"
+				reason="Never" />
 			<disable_collisions link1="rear_left_wheel_link" link2="tower_link" reason="Never" />
 			<disable_collisions link1="rear_right_wheel_link" link2="tower_link" reason="Never" />

Commit message: stand position changed

File: igus_rebel_description_ros2/urdf/igus_rebel/igus_rebel.description.xacro (robot description, xacro)
@@ -61,5 +61,5 @@
 			<parent link="link_1" />
 			<child link="link_2" />
-			<origin rpy="0.0 0.0 0.0" xyz="0.0 0.0 0.149" />
+			<origin rpy="0.0 ${pi/6} 0.0" xyz="0.0 0 0.149" />
 			<axis xyz="0 1 0" />
 			<limit effort="330.0" lower="${-pi*80/180}" upper="${pi*140/180}" velocity="${pi/4.0}" />
@@ -91,5 +91,5 @@
 			<parent link="link_2" />
 			<child link="link_5" />
-			<origin rpy="0.0 0.0 0.0" xyz="0.0 0.0 0.237" />
+			<origin rpy="0.0 ${pi/6} 0.0" xyz="0.0 0.0 0.2384" />
 			<axis xyz="0 1 0" />
 			<limit effort="330.0" lower="${-pi*80/180}" upper="${pi*140/180}" velocity="${pi/4.0}" />
@@ -151,5 +151,5 @@
 			<parent link="link_6" />
 			<child link="link_7" />
-			<origin rpy="0.0 0.0 0.0" xyz="0.0 0.0 0.170" />
+			<origin rpy="0.0 ${-pi/24} 0.0" xyz="0.0 0 ${0.14 + 0.03}" />
 			<axis xyz="0 1 0" />
 			<limit effort="330.0" lower="${-pi/2.0}" upper="${pi/2.0}" velocity="${pi/4.0}" />
