Commit message: adjustments: - world frame is added (between base_link and basefootprint) only regarding the base (true or false) - igus rebel is parallel to the base - the initial position of igus rebel is standing - enable collisions between wheels and the other part of the system

File: igus_rebel_description_ros2/urdf/igus_rebel/igus_rebel.description.xacro (robot description, xacro)
@@ -61,5 +61,5 @@
 			<parent link="link_1" />
 			<child link="link_2" />
-			<origin rpy="0.0 ${pi/6} 0.0" xyz="0.0 0 0.149" />
+			<origin rpy="0.0 0.0 0.0" xyz="0.0 0 0.149" />
 			<axis xyz="0 1 0" />
 			<limit effort="330.0" lower="${-pi*80/180}" upper="${pi*140/180}" velocity="${pi/4.0}" />
@@ -91,5 +91,5 @@
 			<parent link="link_2" />
 			<child link="link_5" />
-			<origin rpy="0.0 ${pi/6} 0.0" xyz="0.0 0.0 0.2384" />
+			<origin rpy="0.0 0.0 0.0" xyz="0.0 0.0 0.2384" />
 			<axis xyz="0 1 0" />
 			<limit effort="330.0" lower="${-pi*80/180}" upper="${pi*140/180}" velocity="${pi/4.0}" />
@@ -151,5 +151,5 @@
 			<parent link="link_6" />
 			<child link="link_7" />
-			<origin rpy="0.0 ${-pi/24} 0.0" xyz="0.0 0 ${0.14 + 0.03}" />
+			<origin rpy="0.0 0.0 0.0" xyz="0.0 0 ${0.14 + 0.03}" />
 			<axis xyz="0 1 0" />
 			<limit effort="330.0" lower="${-pi/2.0}" upper="${pi/2.0}" velocity="${pi/4.0}" />

File: igus_rebel_description_ros2/urdf/robot.urdf.xacro (robot description, xacro)
@@ -20,23 +20,20 @@
 	<xacro:property name="damping" value="0.0" />
 	<xacro:property name="friction" value="0.0" />
-	<!-- Add world link, necessary only when igus rebel is loaded on gazebo without the scout -->
-	<xacro:if value="$(arg load_gazebo)">
-		<xacro:unless value="$(arg load_base)">
-			<link name="world" />
-			<joint name="world_joint" type="fixed">
-				<parent link="world" />
-				<child link="base_link" />
-			</joint>
-		</xacro:unless>
-	</xacro:if>
+	<!-- Add world link -->
+	<xacro:unless value="$(arg load_base)">
+		<link name="world" />
+		<joint name="world_joint" type="fixed">
+			<parent link="world" />
+			<child link="base_link" />
+		</joint>
+	</xacro:unless>
 	<!-- Load mobile robot base, load_base must be true -->
 	<xacro:if value="$(arg load_base)">
-		<xacro:if value="$(arg load_gazebo)">
-			<link name="world" />
-			<joint name="world_joint" type="fixed">
-				<parent link="world" />
-				<child link="base_footprint" />
-			</joint>
-		</xacro:if>
+		<link name="world" />
+		<joint name="world_joint" type="fixed">
+			<origin rpy="0 0 ${pi}" />
+			<parent link="world" />
+			<child link="base_footprint" />
+		</joint>
 		<!-- add virtual joints and links to create a complete TF tree supporting both igus rebel
 		and mobile robot -->
@@ -53,5 +50,5 @@
 			<parent link="rebel_support" />
 			<child link="igus_rebel_base_link" />
-			<origin xyz="0.0 0.0 0.0" rpy="0 0 ${-pi/3}" />
+			<origin xyz="0.0 0.0 0.0" rpy="0 0 0" />
 		</joint>
 		<!-- castle with tower mounting sensors, batteries, computer and everyhting else, attached

File: igus_rebel_moveit_config/config/igus_rebel.srdf.xacro (robot description, xacro)
@@ -119,5 +119,5 @@
 			<!-- Default collision checks for base robot and scout. The collision between the scout
 			and the mount are all enabled-->
-			<disable_collisions link1="front_left_wheel_link" link2="front_right_wheel_link"
+			<!-- <disable_collisions link1="front_left_wheel_link" link2="front_right_wheel_link"
 				reason="Never" />
 			<disable_collisions link1="front_left_wheel_link" link2="igus_rebel_base_link"
@@ -144,28 +144,28 @@
 			<disable_collisions link1="front_right_wheel_link" link2="rear_right_wheel_link"
 				reason="Never" />
-			<disable_collisions link1="front_right_wheel_link" link2="tower_link" reason="Never" />
+			<disable_collisions link1="front_right_wheel_link" link2="tower_link" reason="Never" /> -->
 			<disable_collisions link1="igus_rebel_base_link" link2="mobile_robot_base_link"
 				reason="Adjacent" />
-			<disable_collisions link1="igus_rebel_base_link" link2="rear_left_wheel_link"
+			<!-- <disable_collisions link1="igus_rebel_base_link" link2="rear_left_wheel_link"
 				reason="Never" />
 			<disable_collisions link1="igus_rebel_base_link" link2="rear_right_wheel_link"
-				reason="Never" />
+				reason="Never" /> -->
 			<disable_collisions link1="igus_rebel_base_link" link2="tower_link" reason="Never" />
 			<disable_collisions link1="link_1" link2="mobile_robot_base_link" reason="Never" />
-			<disable_collisions link1="link_1" link2="rear_left_wheel_link" reason="Never" />
-			<disable_collisions link1="link_1" link2="rear_right_wheel_link" reason="Never" />
+			<!-- <disable_collisions link1="link_1" link2="rear_left_wheel_link" reason="Never" /> -->
+			<!-- <disable_collisions link1="link_1" link2="rear_right_wheel_link" reason="Never" /> -->
 			<disable_collisions link1="link_1" link2="tower_link" reason="Never" />
 			<disable_collisions link1="link_2" link2="mobile_robot_base_link" reason="Never" />
-			<disable_collisions link1="link_2" link2="rear_left_wheel_link" reason="Never" />
-			<disable_collisions link1="link_2" link2="rear_right_wheel_link" reason="Never" />
-			<disable_collisions link1="mobile_robot_base_link" link2="rear_left_wheel_link"
+			<!-- <disable_collisions link1="link_2" link2="rear_left_wheel_link" reason="Never" /> -->
+			<!-- <disable_collisions link1="link_2" link2="rear_right_wheel_link" reason="Never" /> -->
+			<!-- <disable_collisions link1="mobile_robot_base_link" link2="rear_left_wheel_link"
 				reason="Adjacent" />
 			<disable_collisions link1="mobile_robot_base_link" link2="rear_right_wheel_link"
-				reason="Adjacent" />
+				reason="Adjacent" /> -->
 			<disable_collisions link1="mobile_robot_base_link" link2="tower_link" reason="Adjacent" />
-			<disable_collisions link1="rear_left_wheel_link" link2="rear_right_wheel_link"
+			<!-- <disable_collisions link1="rear_left_wheel_link" link2="rear_right_wheel_link"
 				reason="Never" />
 			<disable_collisions link1="rear_left_wheel_link" link2="tower_link" reason="Never" />
-			<disable_collisions link1="rear_right_wheel_link" link2="tower_link" reason="Never" />
+			<disable_collisions link1="rear_right_wheel_link" link2="tower_link" reason="Never" /> -->
 		</xacro:if>
 		<!-- Collision checks due to the presence of the mount -->
