Commit message: SRDF modular and comprehensive collisions

File: igus_rebel_moveit_config/config/igus_rebel.srdf.xacro (robot description, xacro)
@@ -1,111 +1,128 @@
 <?xml version="1.0"?>
 <robot xmlns:xacro="http://wiki.ros.org/xacro" name="igus_rebel">
-	<!--GROUPS:
-	Representation of a set of joints and links. This can be useful for specifying DOF to plan for,
-	defining arms, end effectors, etc-->
-	<!--LINKS:
-	When a link is specified, the parent joint of that link (if it exists) is automatically
-	included-->
-	<!--JOINTS:
-	When a joint is specified, the child link of that joint (which will always exist) is
-	automatically included-->
-	<!--CHAINS:
-	When a chain is specified, all the links along the chain (including endpoints) are included in
-	the group. Additionally, all the joints that are parents to included links are also included.
-	This means that joints along the chain and the parent joint of the base link are included in the
-	group-->
-	<!--SUBGROUPS:
-	Groups can also be formed by referencing to already defined group names-->
-	<!-- disable collisions between a link and the robot scout and tower -->
-	<xacro:macro name="no_collision_scout" params="link">
-		<disable_collisions link1="${link}" link2="mobile_robot_base_link" reason="Never" />
-		<disable_collisions link1="${link}" link2="tower_link" reason="Never" />
-		<disable_collisions link1="${link}" link2="front_right_wheel_link" reason="Never" />
-		<disable_collisions link1="${link}" link2="front_left_wheel_link" reason="Never" />
-		<disable_collisions link1="${link}" link2="rear_right_wheel_link" reason="Never" />
-		<disable_collisions link1="${link}" link2="rear_left_wheel_link" reason="Never" />
-	</xacro:macro>
-	<!-- disable collision between a link and the camera links-->
-	<xacro:macro name="no_collision_camera" params="link">
-		<disable_collisions link1="${link}" link2="camera_link" reason="Never" />
-		<disable_collisions link1="${link}" link2="camera_mount" reason="Never" />
-		<disable_collisions link1="${link}" link2="toucher_cylinder" reason="Never" />
-		<disable_collisions link1="${link}" link2="camera_usb_plug_link" reason="Never" />
-	</xacro:macro>
-	<xacro:arg name="gripper" default="none" />
+	<!-- Arguments -->
 	<xacro:arg name="load_base" default="false" />
-	<!-- macro xacro definition to load gripper and mobile robot base -->
-	<xacro:macro name="srdf" params="gripper load_base">
-		<!-- common definitions -->
-		<group name="rebel_arm">
-			<link name="igus_rebel_base_link" />
-			<link name="link_1" />
-			<link name="link_2" />
-			<link name="link_5" />
-			<link name="link_6" />
-			<link name="link_7" />
-			<link name="link_8" />
-		</group>
-		<group name="chain_arm">
-			<chain base_link="igus_rebel_base_link" tip_link="link_8" />
-		</group>
-		<!-- no grippers installed => end effector placed on link_8 -->
-		<xacro:if value="${gripper == 'none'}">
-			<end_effector name="manipulator" parent_link="link_8" group="rebel_arm"
-				parent_group="chain_arm" />
-			<!-- default positions common for every configuration -->
-			<group_state name="zero" group="chain_arm">
-				<joint name="joint1" value="0" />
-				<joint name="joint2" value="0" />
-				<joint name="joint3" value="0" />
-				<joint name="joint4" value="0" />
-				<joint name="joint5" value="0" />
-				<joint name="joint6" value="0" />
-			</group_state>
-			<group_state name="home" group="chain_arm">
-				<joint name="joint1" value="0" />
-				<joint name="joint2" value="${-pi/6.0}" />
-				<joint name="joint3" value="${-pi/6.0}" />
-				<joint name="joint4" value="0" />
-				<joint name="joint5" value="${pi/24.0}" />
-				<joint name="joint6" value="0" />
-			</group_state>
-		</xacro:if>
-		<!-- if camera is placed => end effector on tip_link link -->
-		<xacro:if value="${gripper == 'camera'}">
-			<group name="camera">
-				<link name="camera_link" />
-				<link name="camera_mount" />
-				<link name="camera_usb_plug_link" />
-				<link name="toucher_cylinder" />
-                <link name="tip_link" />
+	<xacro:arg name="mount" default="none" />
+	<xacro:arg name="camera" default="none" />
+	<xacro:arg name="end_effector" default="none" />
+	<!-- macro xacro definition to load mount and mobile robot base -->
+	<xacro:macro name="srdf" params="mount camera end_effector load_base">
+		<!-- Groups -->
+		<!-- If mount is not placed -->
+		<xacro:if value="${mount == 'none'}">
+			<group name="rebel_arm">
+				<chain base_link="igus_rebel_base_link" tip_link="link_8" />
 			</group>
-			<group name="chain_arm_manipulator">
-				<chain base_link="igus_rebel_base_link" tip_link="tip_link" />
+			<group name="flange_group">
+				<link name="flange" />
 			</group>
-			<end_effector name="manipulator" parent_link="tip_link" group="chain_arm_manipulator" parent_group="camera" />
-			<group_state name="zero" group="chain_arm_manipulator">
-				<joint name="joint1" value="0" />
-				<joint name="joint2" value="0" />
-				<joint name="joint3" value="0" />
-				<joint name="joint4" value="0" />
-				<joint name="joint5" value="0" />
-				<joint name="joint6" value="0" />
-			</group_state>
-			<group_state name="home" group="chain_arm_manipulator">
-				<joint name="joint1" value="0" />
-				<joint name="joint2" value="${-pi/6.0}" />
-				<joint name="joint3" value="${-pi/6.0}" />
-				<joint name="joint4" value="0" />
-				<joint name="joint5" value="${pi/24.0}" />
-				<joint name="joint6" value="0" />
-			</group_state>
-		</xacro:if>
+			<end_effector name="flange_EEF" parent_link="link_8" group="flange_group"
+				parent_group="rebel_arm" />
+		</xacro:if>
+		<!-- If mount is placed -->
+		<xacro:if value="${mount == 'mount_v1'}">
+			<!-- If camera is none and no end effector -->
+			<xacro:if value="${camera == 'none' and end_effector == 'none'}">
+				<group name="rebel_arm">
+					<chain base_link="igus_rebel_base_link" tip_link="flange" />
+				</group>
+				<group name="camera_mount_group">
+					<link name="camera_mount" />
+				</group>
+				<end_effector name="camera_mount_EEF" parent_link="flange"
+					group="camera_mount_group" parent_group="rebel_arm" />
+			</xacro:if>
+			<!-- If camera is realsense and no end effector-->
+			<xacro:if value="${camera == 'realsense' and end_effector == 'none'}">
+				<group name="rebel_arm">
+					<chain base_link="igus_rebel_base_link" tip_link="camera_mount" />
+				</group>
+				<group name="camera_link_group">
+					<link name="camera_insert" />
+					<link name="camera_bottom_screw_frame" />
+					<link name="camera_link" />
+					<link name="camera_usb_plug_link" />
+				</group>
+				<end_effector name="camera_link_EEF" parent_link="camera_mount"
+					group="camera_link_group" parent_group="rebel_arm" />
+			</xacro:if>
+			<!-- If camera is oakd and no end effector-->
+			<xacro:if value="${camera == 'oakd' and end_effector == 'none'}">
+				<group name="rebel_arm">
+					<chain base_link="igus_rebel_base_link" tip_link="camera_mount" />
+				</group>
+				<group name="camera_link_group">
+					<link name="camera_insert" />
+					<link name="camera_link" />
+				</group>
+				<end_effector name="camera_link_EEF" parent_link="camera_mount"
+					group="camera_link_group" parent_group="rebel_arm" />
+			</xacro:if>
+			<!-- If camera is none and toucher v1 is placed -->
+			<xacro:if value="${camera == 'none' and end_effector == 'toucher_v1'}">
+				<group name="rebel_arm">
+					<chain base_link="igus_rebel_base_link" tip_link="camera_mount" />
+				</group>
+				<group name="toucher_v1_group">
+					<link name="toucher_v1" />
+				</group>
+				<end_effector name="toucher_v1_EEF" parent_link="camera_mount"
+					group="toucher_v1_group" parent_group="rebel_arm" />
+			</xacro:if>
+			<!-- If camera is realsense and toucher v1 is placed -->
+			<xacro:if value="${camera == 'realsense' and end_effector == 'toucher_v1'}">
+				<group name="rebel_arm">
+					<chain base_link="igus_rebel_base_link" tip_link="camera_mount" />
+				</group>
+				<group name="camera_link_group">
+					<link name="camera_insert" />
+					<link name="camera_bottom_screw_frame" />
+					<link name="camera_link" />
+					<link name="camera_usb_plug_link" />
+				</group>
+				<group name="toucher_v1_group">
+					<link name="toucher_v1" />
+				</group>
+				<end_effector name="toucher_v1_EEF" parent_link="camera_mount"
+					group="toucher_v1_group" parent_group="rebel_arm" />
+			</xacro:if>
+			<!-- If camera is oakd and toucher v1 is placed -->
+			<xacro:if value="${camera == 'oakd' and end_effector == 'toucher_v1'}">
+				<group name="rebel_arm">
+					<chain base_link="igus_rebel_base_link" tip_link="camera_mount" />
+				</group>
+				<group name="camera_link_group">
+					<link name="camera_insert" />
+					<link name="camera_link" />
+				</group>
+				<group name="toucher_v1_group">
+					<link name="toucher_v1" />
+				</group>
+				<end_effector name="toucher_v1_EEF" parent_link="camera_mount"
+					group="toucher_v1_group" parent_group="rebel_arm" />
+			</xacro:if>
+		</xacro:if>
+		<!-- Positions common for every configuration -->
+		<group_state name="zero" group="rebel_arm">
+			<joint name="joint1" value="0" />
+			<joint name="joint2" value="0" />
+			<joint name="joint3" value="0" />
+			<joint name="joint4" value="0" />
+			<joint name="joint5" value="0" />
+			<joint name="joint6" value="0" />
+		</group_state>
+		<group_state name="home" group="rebel_arm">
+			<joint name="joint1" value="0" />
+			<joint name="joint2" value="${-pi/6.0}" />
+			<joint name="joint3" value="${-pi/6.0}" />
+			<joint name="joint4" value="0" />
+			<joint name="joint5" value="${pi/24.0}" />
+			<joint name="joint6" value="0" />
+		</group_state>
 		<!--TODO:
 		add parking position -->
-		<!--<virtual_joint
-		name="world_to_base" type="fixed" parent_frame="world" child_link="base_link" />-->
-		<!-- default collision checks for base robot -->
-		<disable_collisions link1="base_link" link2="igus_rebel_base_link" reason="Adjacent" />
+		<!-- Collisions -->
+		<!-- Default collision checks for base robot. This is the simplest configuration, that is
+		always present. -->
 		<disable_collisions link1="igus_rebel_base_link" link2="link_1" reason="Adjacent" />
 		<disable_collisions link1="igus_rebel_base_link" link2="link_2" reason="Never" />
@@ -120,22 +137,6 @@
 		<disable_collisions link1="link_6" link2="link_7" reason="Adjacent" />
 		<disable_collisions link1="link_6" link2="link_8" reason="Never" />
-		<disable_collisions link1="link_7" link2="link_8" reason="Adjacent" />
-		<!-- additional collision checks due to the presence of the camera mount -->
-		<xacro:if value="${gripper == 'camera'}">
-			<disable_collisions link1="camera_link" link2="camera_mount" reason="Adjacent" />
-			<disable_collisions link1="camera_link" link2="camera_usb_plug_link" reason="Adjacent" />
-			<disable_collisions link1="camera_mount" link2="camera_usb_plug_link" reason="Never" />
-			<disable_collisions link1="camera_link" link2="toucher_cylinder" reason="Never" />
-			<disable_collisions link1="camera_mount" link2="toucher_cylinder" reason="Never" />
-            <disable_collisions link1="toucher_cylinder" link2="tip_link" reason="Adjacent" />
-			<xacro:no_collision_camera link="igus_rebel_base_link" />
-			<xacro:no_collision_camera link="link_1" />
-			<xacro:no_collision_camera link="link_2" />
-			<xacro:no_collision_camera link="link_5" />
-			<xacro:no_collision_camera link="link_6" />
-			<xacro:no_collision_camera link="link_7" />
-			<xacro:no_collision_camera link="link_8" />
-		</xacro:if>
-		<!-- when the robot scout is loaded define the collision checks -->
+		<disable_collisions link1="link_7" link2="link_8" reason="Adjacent" /> <!-- 13 -->
+		<!-- Collisions checks due to the presence of the scout base -->
 		<xacro:if value="${load_base}">
 			<group name="mobile_robot">
@@ -151,16 +152,9 @@
 				<link name="tower_link" />
 			</group>
-			<disable_collisions link1="igus_rebel_base_link" link2="front_left_wheel_link"
-				reason="Never" />
-			<disable_collisions link1="igus_rebel_base_link" link2="front_right_wheel_link"
-				reason="Never" />
-			<disable_collisions link1="igus_rebel_base_link" link2="mobile_robot_base_link"
-				reason="Adjacent" />
-			<disable_collisions link1="igus_rebel_base_link" link2="rear_left_wheel_link"
-				reason="Never" />
-			<disable_collisions link1="igus_rebel_base_link" link2="rear_right_wheel_link"
-				reason="Never" />
-			<disable_collisions link1="igus_rebel_base_link" link2="tower_link" reason="Never" />
+			<!-- Default collision checks for base robot and scout. The collision between the scout
+			and the mount are all enabled-->
 			<disable_collisions link1="front_left_wheel_link" link2="front_right_wheel_link"
+				reason="Never" />
+			<disable_collisions link1="front_left_wheel_link" link2="igus_rebel_base_link"
 				reason="Never" />
 			<disable_collisions link1="front_left_wheel_link" link2="link_1" reason="Never" />
@@ -174,4 +168,6 @@
 				reason="Never" />
 			<disable_collisions link1="front_left_wheel_link" link2="tower_link" reason="Never" />
+			<disable_collisions link1="front_right_wheel_link" link2="igus_rebel_base_link"
+				reason="Never" />
 			<disable_collisions link1="front_right_wheel_link" link2="link_1" reason="Never" />
 			<disable_collisions link1="front_right_wheel_link" link2="link_2" reason="Never" />
@@ -184,4 +180,11 @@
 				reason="Never" />
 			<disable_collisions link1="front_right_wheel_link" link2="tower_link" reason="Never" />
+			<disable_collisions link1="igus_rebel_base_link" link2="mobile_robot_base_link"
+				reason="Adjacent" />
+			<disable_collisions link1="igus_rebel_base_link" link2="rear_left_wheel_link"
+				reason="Never" />
+			<disable_collisions link1="igus_rebel_base_link" link2="rear_right_wheel_link"
+				reason="Never" />
+			<disable_collisions link1="igus_rebel_base_link" link2="tower_link" reason="Never" />
 			<disable_collisions link1="link_1" link2="mobile_robot_base_link" reason="Never" />
 			<disable_collisions link1="link_1" link2="rear_left_wheel_link" reason="Never" />
@@ -201,6 +204,83 @@
 			<disable_collisions link1="rear_right_wheel_link" link2="tower_link" reason="Never" />
 		</xacro:if>
+		<!-- Collision checks due to the presence of the mount -->
+		<xacro:if value="${mount == 'mount_v1'}">
+			<disable_collisions link1="link_5" link2="camera_mount" reason="Never" />
+			<disable_collisions link1="link_6" link2="camera_mount" reason="Never" />
+			<disable_collisions link1="link_7" link2="camera_mount" reason="Never" />
+			<disable_collisions link1="link_8" link2="camera_mount" reason="Adjacent" />
+			<!-- <xacro:if value="${camera == 'none' and end_effector == 'none}">
+				nothing
+			</xacro:if> -->
+			<xacro:if value="${camera == 'oakd' and end_effector == 'none'}">
+				<disable_collisions link1="camera_mount" link2="camera_link" reason="Adjacent" />
+				<disable_collisions link1="link_5" link2="camera_link" reason="Never" />
+				<disable_collisions link1="link_6" link2="camera_link" reason="Never" />
+				<disable_collisions link1="link_7" link2="camera_link" reason="Never" />
+				<disable_collisions link1="link_8" link2="camera_link" reason="Never" />
+			</xacro:if>
+			<xacro:if value="${camera == 'realsense' and end_effector == 'none'}">
+				<disable_collisions link1="camera_mount" link2="camera_link" reason="Adjacent" />
+				<disable_collisions link1="camera_link" link2="camera_usb_plug_link"
+					reason="Adjacent" />
+				<disable_collisions link1="camera_mount" link2="camera_usb_plug_link" reason="Never" />
+				<disable_collisions link1="link_5" link2="camera_link" reason="Never" />
+				<disable_collisions link1="link_5" link2="camera_usb_plug_link" reason="Never" />
+				<disable_collisions link1="link_6" link2="camera_link" reason="Never" />
+				<disable_collisions link1="link_6" link2="camera_usb_plug_link" reason="Never" />
+				<disable_collisions link1="link_7" link2="camera_link" reason="Never" />
+				<disable_collisions link1="link_7" link2="camera_usb_plug_link" reason="Never" />
+				<disable_collisions link1="link_8" link2="camera_link" reason="Never" />
+				<disable_collisions link1="link_8" link2="camera_usb_plug_link" reason="Never" />
+			</xacro:if>
+			<xacro:if value="${camera == 'none' and end_effector == 'toucher_v1'}">
+				<disable_collisions link1="camera_mount" link2="toucher_v1" reason="Adjacent" />
+				<disable_collisions link1="link_2" link2="toucher_v1" reason="Never" />
+				<disable_collisions link1="link_5" link2="toucher_v1" reason="Never" />
+				<disable_collisions link1="link_6" link2="toucher_v1" reason="Never" />
+				<disable_collisions link1="link_7" link2="toucher_v1" reason="Never" />
+				<disable_collisions link1="link_8" link2="toucher_v1" reason="Default" />
+			</xacro:if>
+			<xacro:if value="${camera == 'oakd' and end_effector == 'toucher_v1'}">
+				<disable_collisions link1="camera_mount" link2="camera_link" reason="Adjacent" />
+				<disable_collisions link1="link_5" link2="camera_link" reason="Never" />
+				<disable_collisions link1="link_6" link2="camera_link" reason="Never" />
+				<disable_collisions link1="link_7" link2="camera_link" reason="Never" />
+				<disable_collisions link1="link_8" link2="camera_link" reason="Never" />
+				<disable_collisions link1="camera_mount" link2="toucher_v1" reason="Adjacent" />
+				<disable_collisions link1="link_2" link2="toucher_v1" reason="Never" />
+				<disable_collisions link1="link_5" link2="toucher_v1" reason="Never" />
+				<disable_collisions link1="link_6" link2="toucher_v1" reason="Never" />
+				<disable_collisions link1="link_7" link2="toucher_v1" reason="Never" />
+				<disable_collisions link1="link_8" link2="toucher_v1" reason="Default" />
+				<disable_collisions link1="camera_link" link2="toucher_v1" reason="Never" />
+			</xacro:if>
+			<xacro:if value="${camera == 'realsense' and end_effector == 'toucher_v1'}">
+				<disable_collisions link1="camera_mount" link2="camera_link" reason="Adjacent" />
+				<disable_collisions link1="link_5" link2="camera_link" reason="Never" />
+				<disable_collisions link1="link_6" link2="camera_link" reason="Never" />
+				<disable_collisions link1="link_7" link2="camera_link" reason="Never" />
+				<disable_collisions link1="link_8" link2="camera_link" reason="Never" />
+				<disable_collisions link1="camera_mount" link2="toucher_v1" reason="Adjacent" />
+				<disable_collisions link1="link_2" link2="toucher_v1" reason="Never" />
+				<disable_collisions link1="link_5" link2="toucher_v1" reason="Never" />
+				<disable_collisions link1="link_6" link2="toucher_v1" reason="Never" />
+				<disable_collisions link1="link_7" link2="toucher_v1" reason="Never" />
+				<disable_collisions link1="link_8" link2="toucher_v1" reason="Default" />
+				<disable_collisions link1="camera_link" link2="toucher_v1" reason="Never" />
+				<disable_collisions link1="camera_link" link2="camera_usb_plug_link"
+					reason="Adjacent" />
+				<disable_collisions link1="camera_mount" link2="camera_usb_plug_link" reason="Never" />
+				<disable_collisions link1="link_5" link2="camera_usb_plug_link" reason="Never" />
+				<disable_collisions link1="link_6" link2="camera_usb_plug_link" reason="Never" />
+				<disable_collisions link1="link_7" link2="camera_usb_plug_link" reason="Never" />
+				<disable_collisions link1="link_8" link2="camera_usb_plug_link" reason="Never" />
+				<disable_collisions link1="toucher_v1" link2="camera_usb_plug_link"
+					reason="Never" />
+			</xacro:if>
+		</xacro:if>
 	</xacro:macro>
-	<!-- call the macro and define everything -->
-	<xacro:srdf gripper="$(arg gripper)" load_base="$(arg load_base)" />
+	<!-- Call the macro and define the arguments -->
+	<xacro:srdf mount="$(arg mount)" camera="$(arg camera)" end_effector="$(arg end_effector)"
+		load_base="$(arg load_base)" />
 </robot>

Commit message: updated readme with new documentation

File: igus_rebel_moveit_config/config/igus_rebel.srdf.xacro (robot description, xacro)
@@ -66,10 +66,10 @@
 		</group_state>
 		<group_state name="parked" group="rebel_arm">
-			<joint name="joint1" value="0" />
-			<joint name="joint2" value="${36.0 * pi / 180.0}" />
-			<joint name="joint3" value="${76.0 * pi / 180.0}" />
-			<joint name="joint4" value="${124.0 * pi / 180.0}" />
-			<joint name="joint5" value="${-81.0 * pi / 180.0}" />
-			<joint name="joint6" value="0" />
+			<joint name="joint1" value="${-42.0 * pi / 180.0}" />
+			<joint name="joint2" value="${40.0 * pi / 180.0}" />
+			<joint name="joint3" value="${73.0 * pi / 180.0}" />
+			<joint name="joint4" value="${82.0 * pi / 180.0}" />
+			<joint name="joint5" value="${-78.0 * pi / 180.0}" />
+			<joint name="joint6" value="${-95.0 * pi / 180.0}" />
 		</group_state>
 		<!--############################################################################### -->

Commit message: add manipulator action server

File: igus_rebel_moveit_config/config/igus_rebel.srdf.xacro (robot description, xacro)
@@ -72,4 +72,12 @@
 			<joint name="joint5" value="${-78.0 * pi / 180.0}" />
 			<joint name="joint6" value="${-95.0 * pi / 180.0}" />
+		</group_state>
+		<group_state name="stand" group="rebel_arm">
+			<joint name="joint1" value="${11.0 * pi / 180.0}" />
+			<joint name="joint2" value="${-40.0 * pi / 180.0}" />
+			<joint name="joint3" value="${-18.0 * pi / 180.0}" />
+			<joint name="joint4" value="0" />
+			<joint name="joint5" value="${85.0 * pi / 180.0}" />
+			<joint name="joint6" value="0" />
 		</group_state>
 		<!--############################################################################### -->

Commit message: major fix

File: igus_rebel_moveit_config/config/igus_rebel.srdf.xacro (robot description, xacro)
@@ -74,10 +74,10 @@
 		</group_state>
 		<group_state name="stand" group="rebel_arm">
-			<joint name="joint1" value="${11.0 * pi / 180.0}" />
-			<joint name="joint2" value="${-40.0 * pi / 180.0}" />
-			<joint name="joint3" value="${-18.0 * pi / 180.0}" />
+			<joint name="joint1" value="${61.0 * pi / 180.0}" />
+			<joint name="joint2" value="${-90.0 * pi / 180.0}" />
+			<joint name="joint3" value="${36.0 * pi / 180.0}" />
 			<joint name="joint4" value="0" />
-			<joint name="joint5" value="${85.0 * pi / 180.0}" />
-			<joint name="joint6" value="0" />
+			<joint name="joint5" value="${95.0 * pi / 180.0}" />
+			<joint name="joint6" value="${5.0 * pi / 180.0}" />
 		</group_state>
 		<!--############################################################################### -->
