Commit message: updated mounts with new improved design

File: igus_rebel_description_ros2/urdf/cameras/cameras.urdf.xacro (robot description, xacro)
@@ -4,5 +4,6 @@
         <!-- virtual frames for gazebo -->
         <xacro:if value="${load_gazebo}">
-            <xacro:include filename="$(find igus_rebel_description_ros2)/urdf/cameras/virtual_camera_frames.xacro" />
+            <xacro:include
+                filename="$(find igus_rebel_description_ros2)/urdf/cameras/virtual_camera_frames.xacro" />
             <xacro:virtual_camera_frames />
         </xacro:if>
@@ -11,8 +12,10 @@
             <!-- includes the realsense D435 ros2 description file and its collision box-->
             <xacro:arg name="use_nominal_extrinsics" default="false" />
-            <xacro:arg name="add_plug" default="true" />
+            <xacro:arg name="add_plug" default="false" />
             <xacro:arg name="use_mesh" default="true" />
             <xacro:include filename="$(find realsense2_description)/urdf/_d435.urdf.xacro" />
-            <xacro:sensor_d435 parent="camera_insert" use_nominal_extrinsics="$(arg use_nominal_extrinsics)" add_plug="$(arg add_plug)" use_mesh="$(arg use_mesh)">
+            <xacro:sensor_d435 parent="camera_insert"
+                use_nominal_extrinsics="$(arg use_nominal_extrinsics)" add_plug="$(arg add_plug)"
+                use_mesh="$(arg use_mesh)">
                 <origin xyz="0.0 0 0" rpy="0 0 0" />
             </xacro:sensor_d435>
@@ -24,5 +27,7 @@
                     <xacro:insert_block name="origin" />
                     <mass value="${mass}" />
-                    <inertia ixx="${(1/12) * mass * (y*y+z*z)}" ixy="0.0" ixz="0.0" iyy="${(1/12) * mass * (x*x+z*z)}" iyz="0.0" izz="${(1/12) * mass * (x*x+y*y)}" />
+                    <inertia ixx="${(1/12) * mass * (y*y+z*z)}" ixy="0.0" ixz="0.0"
+                        iyy="${(1/12) * mass * (x*x+z*z)}" iyz="0.0"
+                        izz="${(1/12) * mass * (x*x+y*y)}" />
                 </inertial>
             </xacro:macro>
@@ -39,5 +44,6 @@
                 <visual>
                     <geometry>
-                        <mesh filename="file://$(find igus_rebel_description_ros2)/meshes/cameras/oak_d_pro_camera.dae" />
+                        <mesh
+                            filename="file://$(find igus_rebel_description_ros2)/meshes/cameras/oak_d_pro_camera.dae" />
                     </geometry>
                 </visual>
@@ -48,5 +54,6 @@
                     </geometry>
                 </collision>
-                <xacro:inertial_box mass="${oakd_mass}" x="${oakd_length}" y="${oakd_width}" z="${oakd_depth}">
+                <xacro:inertial_box mass="${oakd_mass}" x="${oakd_length}" y="${oakd_width}"
+                    z="${oakd_depth}">
                     <origin xyz="0.0 0 0.0" rpy="0 0 0" />
                 </xacro:inertial_box>

File: igus_rebel_description_ros2/urdf/end_effectors/soft_gripper.description.xacro (robot description, xacro)
@@ -10,5 +10,5 @@
 		<parent link="camera_mount" />
 		<child link="soft_gripper_mount" />
-		<origin xyz="0.0 0.0 0.0" rpy="0.0 0.0 ${pi/2.0}" />
+		<origin xyz="0.0 0.0 -0.02" rpy="0.0 0.0 ${pi/2.0}" />
 	</joint>
 	<link name="soft_gripper_mount">
@@ -39,5 +39,5 @@
 		<parent link="soft_gripper_mount" />
 		<child link="soft_gripper_link" />
-		<origin xyz="0.0 0 0" rpy="0 0 0" />
+		<origin xyz="0.0 0.0 0.0" rpy="0 0 0" />
 	</joint>
 	<link name="soft_gripper_link">
@@ -68,5 +68,5 @@
 		<parent link="soft_gripper_link" />
 		<child link="soft_gripper_tip_link" />
-		<origin xyz="0.0 0.0 0.1" rpy="${-pi/2.0} ${-pi/2.0} 0.0" />
+		<origin xyz="0.0 0.0 0.095" rpy="${-pi/2.0} ${-pi/2.0} 0.0" />
 	</joint>
 	<link name="soft_gripper_tip_link" />

File: igus_rebel_description_ros2/urdf/igus_rebel/igus_rebel.description.xacro (robot description, xacro)
@@ -181,5 +181,5 @@
 			<parent link="link_7" />
 			<child link="link_8" />
-			<origin rpy="0.0 0.0 0.0" xyz="0.0 0 0.1208" />
+			<origin rpy="0.0 0.0 0.0" xyz="0.0 0 0.126" />
 			<axis xyz="0 0 1" />
 			<limit effort="330.0" lower="${-pi*179/180}" upper="${pi*179/180}" velocity="${pi/4.0}" />
@@ -211,5 +211,5 @@
 			<parent link="link_8" />
 			<child link="flange" />
-			<origin rpy="0.0 ${-pi/2} 0.0" xyz="0.0 0 0.0052" />
+			<origin rpy="0.0 ${-pi/2} 0.0" xyz="0.0 0.0 0.0" />
 			<axis xyz="0 0 0" />
 			<dynamics damping="${damping}" friction="${friction}" />

File: igus_rebel_description_ros2/urdf/mounts/mount_v2.xacro (robot description, xacro)
@@ -9,5 +9,5 @@
 			<parent link="flange" />
 			<child link="camera_mount" />
-			<origin rpy="0.0 ${pi/2.0} 0.0" xyz="0.0 0.0 0.0" />
+			<origin rpy="0.0 ${pi/2.0} 0.0" xyz="0.02 0.0 0.0" />
 			<axis xyz="0 0 0" />
 		</joint>
@@ -41,5 +41,5 @@
 			<parent link="camera_mount" />
 			<child link="camera_insert" />
-			<origin rpy="0.0 ${-pi/2.0} 0.0" xyz="-0.1 0.0 -0.035" />
+			<origin rpy="0.0 ${-pi/2.0} 0.0" xyz="-0.1 0.0 -0.068" />
 			<axis xyz="0 0 0" />
 		</joint>

File: igus_rebel_moveit_config/config/igus_rebel.srdf.xacro (robot description, xacro)
@@ -173,15 +173,8 @@
 			<xacro:if value="${camera == 'realsense' and end_effector == 'none'}">
 				<disable_collisions link1="camera_mount" link2="camera_link" reason="Adjacent" />
-				<disable_collisions link1="camera_link" link2="camera_usb_plug_link"
-					reason="Adjacent" />
-				<disable_collisions link1="camera_mount" link2="camera_usb_plug_link" reason="Never" />
-				<disable_collisions link1="link_5" link2="camera_link" reason="Never" />
-				<disable_collisions link1="link_5" link2="camera_usb_plug_link" reason="Never" />
-				<disable_collisions link1="link_6" link2="camera_link" reason="Never" />
-				<disable_collisions link1="link_6" link2="camera_usb_plug_link" reason="Never" />
-				<disable_collisions link1="link_7" link2="camera_link" reason="Never" />
-				<disable_collisions link1="link_7" link2="camera_usb_plug_link" reason="Never" />
-				<disable_collisions link1="link_8" link2="camera_link" reason="Never" />
-				<disable_collisions link1="link_8" link2="camera_usb_plug_link" reason="Never" />
+				<disable_collisions link1="link_5" link2="camera_link" reason="Never" />
+				<disable_collisions link1="link_6" link2="camera_link" reason="Never" />
+				<disable_collisions link1="link_7" link2="camera_link" reason="Never" />
+				<disable_collisions link1="link_8" link2="camera_link" reason="Never" />
 			</xacro:if>
 			<xacro:if value="${camera == 'none' and end_effector == 'toucher_v1'}">
@@ -220,13 +213,4 @@
 				<disable_collisions link1="link_8" link2="toucher_v1" reason="Default" />
 				<disable_collisions link1="camera_link" link2="toucher_v1" reason="Never" />
-				<disable_collisions link1="camera_link" link2="camera_usb_plug_link"
-					reason="Adjacent" />
-				<disable_collisions link1="camera_mount" link2="camera_usb_plug_link" reason="Never" />
-				<disable_collisions link1="link_5" link2="camera_usb_plug_link" reason="Never" />
-				<disable_collisions link1="link_6" link2="camera_usb_plug_link" reason="Never" />
-				<disable_collisions link1="link_7" link2="camera_usb_plug_link" reason="Never" />
-				<disable_collisions link1="link_8" link2="camera_usb_plug_link" reason="Never" />
-				<disable_collisions link1="toucher_v1" link2="camera_usb_plug_link"
-					reason="Never" />
 			</xacro:if>
 			<xacro:if value="${camera == 'realsense' and end_effector == 'soft_gripper'}">
@@ -234,9 +218,4 @@
 				<disable_collisions link1="link_7" link2="camera_link" reason="Never" />
 				<disable_collisions link1="link_8" link2="camera_link" reason="Never" />
-				<disable_collisions link1="camera_link" link2="camera_usb_plug_link"
-					reason="Adjacent" />
-				<disable_collisions link1="camera_mount" link2="camera_usb_plug_link" reason="Never" />
-				<disable_collisions link1="link_7" link2="camera_usb_plug_link" reason="Never" />
-				<disable_collisions link1="link_8" link2="camera_usb_plug_link" reason="Never" />
 				<disable_collisions link1="camera_mount" link2="soft_gripper_link" reason="Adjacent" />
 				<disable_collisions link1="camera_mount" link2="soft_gripper_mount"
@@ -244,8 +223,4 @@
 				<disable_collisions link1="camera_link" link2="soft_gripper_mount" reason="Never" />
 				<disable_collisions link1="camera_link" link2="soft_gripper_link" reason="Never" />
-				<disable_collisions link1="soft_gripper_mount" link2="camera_usb_plug_link"
-					reason="Never" />
-				<disable_collisions link1="soft_gripper_link" link2="camera_usb_plug_link"
-					reason="Never" />
 				<disable_collisions link1="link_7" link2="soft_gripper_link" reason="Never" />
 				<disable_collisions link1="link_8" link2="soft_gripper_link" reason="Never" />

Commit message: active vision modifications: - world link on robot xacro - camera check xacro - realsense xacro for physic camera - mesh mod for gazebo (soft gripper) - removed rgb and pointcould virtual frames - adjusted srdf - not add camera if mount is none - removed stomp - default moveit rviz config is default of arg - new moveit arg

File: igus_rebel_description_ros2/urdf/cameras/cameras.urdf.xacro (robot description, xacro)
@@ -3,9 +3,11 @@
     <xacro:macro name="cameras" params="camera load_gazebo">
         <!-- virtual frames for gazebo -->
-        <xacro:if value="${load_gazebo}">
-            <xacro:include
-                filename="$(find igus_rebel_description_ros2)/urdf/cameras/virtual_camera_frames.xacro" />
-            <xacro:virtual_camera_frames />
-        </xacro:if>
+        <xacro:unless value="${camera == 'none'}">
+            <xacro:if value="${load_gazebo}">
+                <xacro:include
+                    filename="$(find igus_rebel_description_ros2)/urdf/cameras/virtual_camera_frames.xacro" />
+                <xacro:virtual_camera_frames />
+            </xacro:if>
+        </xacro:unless>
         <!-- Cameras -->
         <xacro:if value="${camera == 'realsense'}">

File: igus_rebel_description_ros2/urdf/end_effectors/soft_gripper.description.xacro (robot description, xacro)
@@ -17,5 +17,5 @@
 			<geometry>
 				<mesh
-					filename="package://igus_rebel_description_ros2/meshes/end_effectors/gripper_mount.stl"
+					filename="file://$(find igus_rebel_description_ros2)/meshes/end_effectors/gripper_mount.stl"
 					scale="0.001 0.001 0.001" />
 			</geometry>
@@ -26,5 +26,5 @@
 			<geometry>
 				<mesh
-					filename="package://igus_rebel_description_ros2/meshes/end_effectors/gripper_mount_collision_mesh.stl"
+					filename="file://$(find igus_rebel_description_ros2)/meshes/end_effectors/gripper_mount_collision_mesh.stl"
 					scale="0.001 0.001 0.001" />
 			</geometry>
@@ -46,5 +46,5 @@
 			<geometry>
 				<mesh
-					filename="package://igus_rebel_description_ros2/meshes/end_effectors/gripper.stl"
+					filename="file://$(find igus_rebel_description_ros2)/meshes/end_effectors/gripper.stl"
 					scale="0.001 0.001 0.001" />
 			</geometry>
@@ -55,8 +55,8 @@
 			<geometry>
 				<mesh
-				filename="package://igus_rebel_description_ros2/meshes/end_effectors/gripper_collision_mesh.stl"
-				scale="0.001 0.001 0.001" />
-		</geometry>
-	</collision>
+					filename="file://$(find igus_rebel_description_ros2)/meshes/end_effectors/gripper_collision_mesh.stl"
+					scale="0.001 0.001 0.001" />
+			</geometry>
+		</collision>
 		<inertial>
 			<origin xyz="0.0 0.0 0.0" rpy="0.0 0.0 0.5" />

File: igus_rebel_description_ros2/urdf/igus_rebel/igus_rebel.gazebo.xacro (robot description, xacro)
@@ -121,32 +121,5 @@
 		</joint>
 		<link name="igus_rebel/link_8/depth_camera" />
-		<!-- Optical frame id for pointcloud sensor -->
-		<joint name="camera_link_to_pointcloud" type="fixed">
-			<parent link="camera_link" />
-			<child link="igus_rebel/link_8/pointcloud" />
-			<origin rpy="0.0 0.0 0.0" xyz="0.0 0.0 0.0" />
-			<axis xyz="0 0 0" />
-		</joint>
-		<link name="igus_rebel/link_8/pointcloud" />
-		<!-- Sensor for RGB, depth and pointcloud data -->
-		<gazebo reference="virtual_rgb_camera_frame">
-			<sensor type="camera" name="rgb_camera">
-				<camera>
-					<horizontal_fov>1.05</horizontal_fov>
-					<image>
-						<width>640</width>
-						<height>480</height>
-					</image>
-					<clip>
-						<near>0.3</near>
-						<far>100</far>
-					</clip>
-					<optical_frame_id>virtual_rgb_camera_frame</optical_frame_id>
-				</camera>
-				<always_on>1</always_on>
-				<update_rate>30</update_rate>
-				<visualize>true</visualize>
-			</sensor>
-		</gazebo>
+		<!-- Sensor for RGB and depth image data -->
 		<gazebo reference="virtual_depth_camera_frame">
 			<sensor type="rgbd_camera" name="depth_camera">
@@ -173,21 +146,4 @@
 			</sensor>
 		</gazebo>
-		<gazebo reference="virtual_depth_camera_frame">
-			<sensor type="rgbd_camera" name="pointcloud">
-				<update_rate>10</update_rate>
-				<camera>
-					<horizontal_fov>1.05</horizontal_fov>
-					<image>
-						<width>640</width>
-						<height>480</height>
-						<format>R8G8B8</format>
-					</image>
-					<clip>
-						<near>0.1</near>
-						<far>10.0</far>
-					</clip>
-				</camera>
-			</sensor>
-		</gazebo>
 	</xacro:macro>
 </robot>

File: igus_rebel_description_ros2/urdf/igus_rebel/igus_rebel.urdf.xacro (robot description, xacro)
@@ -22,6 +22,8 @@
 		</xacro:if>
 		<!-- Camera macro -->
-		<xacro:include filename="$(find igus_rebel_description_ros2)/urdf/cameras/cameras.urdf.xacro" />
-		<xacro:cameras camera="${camera}" load_gazebo="${load_gazebo}" />
+		<xacro:unless value="${mount == 'none'}"> <!-- Do not add cameras if no mount is present -->
+			<xacro:include filename="$(find igus_rebel_description_ros2)/urdf/cameras/cameras.urdf.xacro" />
+			<xacro:cameras camera="${camera}" load_gazebo="${load_gazebo}" />
+		</xacro:unless>
 		<!-- Gazebo macro -->
 		<xacro:if value="${load_gazebo}">

File: igus_rebel_description_ros2/urdf/robot.urdf.xacro (robot description, xacro)
@@ -20,6 +20,27 @@
 	<xacro:property name="damping" value="0.0" />
 	<xacro:property name="friction" value="0.0" />
+	<!-- Add world link, necessary only when igus rebel is loaded on gazebo without the scout -->
+	<xacro:if value="$(arg load_gazebo)">
+		<xacro:unless value="$(arg load_base)">
+			<link name="world" />
+			<joint name="world_joint" type="fixed">
+				<parent link="world" />
+				<child link="base_link" />
+			</joint>
+		</xacro:unless>
+	</xacro:if>
 	<!-- Load mobile robot base, load_base must be true -->
 	<xacro:if value="$(arg load_base)">
+		<xacro:if value="$(arg load_gazebo)">
+			<link name="world" />
+			<joint name="world_joint" type="fixed">
+				<parent link="world" />
+				<child link="base_footprint" />
+			</joint>
+		</xacro:if>
+		<!-- add virtual joints and links to create a complete TF tree supporting both igus rebel
+		and mobile robot -->
+		<!-- base_footprint -> base_link -> { mobile_robot_base_link, rebel_support ->
+		igus_rebel_base_link } -> other links -->
 		<!-- virtual joints acting as a link between base_link and igus_rebel_base_link -->
 		<joint name="base_link_to_rebel_support" type="fixed">

File: igus_rebel_moveit_config/config/igus_rebel.srdf.xacro (robot description, xacro)
@@ -22,8 +22,8 @@
 				parent_group="rebel_arm" />
 		</xacro:if>
-		<!-- If mount is placed -->
-		<xacro:if value="${mount != 'none'}">
+		<!-- If mount v1 is placed -->
+		<xacro:if value="${mount == 'mount_v1'}">
 			<!-- If camera is relasense or oakd and no end effector placed -->
-			<xacro:if value="${end_effector == 'none'}">
+			<xacro:unless value="${end_effector == 'toucher_v1'}">
 				<group name="rebel_arm">
 					<chain base_link="igus_rebel_base_link" tip_link="flange" />
@@ -31,5 +31,5 @@
 				<end_effector name="flange_EEF" parent_link="flange"
 					group="rebel_arm" />
-			</xacro:if>
+			</xacro:unless>
 			<!-- If camera is realsense or oakd and toucher v1 is placed -->
 			<xacro:if value="${end_effector == 'toucher_v1'}">
@@ -44,4 +44,15 @@
 					group="toucher_v1_group" parent_group="rebel_arm" />
 			</xacro:if>
+		</xacro:if>
+		<!-- If mount v2 is placed -->
+		<xacro:if value="${mount == 'mount_v2'}">
+			<!-- If camera is relasense or oakd and no end effector placed -->
+			<xacro:unless value="${end_effector == 'soft_gripper'}">
+				<group name="rebel_arm">
+					<chain base_link="igus_rebel_base_link" tip_link="flange" />
+				</group>
+				<end_effector name="flange_EEF" parent_link="flange"
+					group="rebel_arm" />
+			</xacro:unless>
 			<!-- If camera is realsense and soft gripper is placed -->
 			<xacro:if value="${end_effector == 'soft_gripper'}">
@@ -159,9 +170,10 @@
 		</xacro:if>
 		<!-- Collision checks due to the presence of the mount -->
-		<xacro:if value="${mount == 'mount_v1' or mount == 'mount_v2'}">
+		<xacro:if value="${mount == 'mount_v1'}">
 			<disable_collisions link1="link_5" link2="camera_mount" reason="Never" />
 			<disable_collisions link1="link_6" link2="camera_mount" reason="Never" />
 			<disable_collisions link1="link_7" link2="camera_mount" reason="Never" />
 			<disable_collisions link1="link_8" link2="camera_mount" reason="Adjacent" />
+			<!-- TODO: need to handle case when gripper is not none or toucher with a camera -->
 			<xacro:if value="${camera == 'oakd' and end_effector == 'none'}">
 				<disable_collisions link1="camera_mount" link2="camera_link" reason="Adjacent" />
@@ -213,4 +225,71 @@
 				<disable_collisions link1="link_8" link2="toucher_v1" reason="Default" />
 				<disable_collisions link1="camera_link" link2="toucher_v1" reason="Never" />
+			</xacro:if>
+		</xacro:if>
+		<xacro:if value="${mount == 'mount_v2'}">
+			<disable_collisions link1="link_5" link2="camera_mount" reason="Never" />
+			<disable_collisions link1="link_6" link2="camera_mount" reason="Never" />
+			<disable_collisions link1="link_7" link2="camera_mount" reason="Never" />
+			<disable_collisions link1="link_8" link2="camera_mount" reason="Adjacent" />
+			<!-- TODO: need to handle case when gripper is not none or soft gripper with a camera -->
+			<xacro:if value="${camera == 'oakd' and end_effector == 'none'}">
+				<disable_collisions link1="camera_mount" link2="camera_link" reason="Adjacent" />
+				<disable_collisions link1="link_5" link2="camera_link" reason="Never" />
+				<disable_collisions link1="link_6" link2="camera_link" reason="Never" />
+				<disable_collisions link1="link_7" link2="camera_link" reason="Never" />
+				<disable_collisions link1="link_8" link2="camera_link" reason="Never" />
+			</xacro:if>
+			<xacro:if value="${camera == 'realsense' and end_effector == 'none'}">
+				<disable_collisions link1="camera_mount" link2="camera_link" reason="Adjacent" />
+				<disable_collisions link1="link_5" link2="camera_link" reason="Never" />
+				<disable_collisions link1="link_6" link2="camera_link" reason="Never" />
+				<disable_collisions link1="link_7" link2="camera_link" reason="Never" />
+				<disable_collisions link1="link_8" link2="camera_link" reason="Never" />
+			</xacro:if>
+			<xacro:if value="${camera == 'none' and end_effector == 'soft_gripper'}">
+				<disable_collisions link1="camera_mount" link2="soft_gripper_link" reason="Adjacent" />
+				<disable_collisions link1="camera_mount" link2="soft_gripper_mount" reason="Adjacent" />
+				<disable_collisions link1="link_2" link2="soft_gripper_link" reason="Never" />
+				<disable_collisions link1="link_2" link2="soft_gripper_mount" reason="Never" />
+				<disable_collisions link1="link_5" link2="soft_gripper_link" reason="Never" />
+				<disable_collisions link1="link_5" link2="soft_gripper_mount" reason="Never" />
+				<disable_collisions link1="link_6" link2="soft_gripper_link" reason="Never" />
+				<disable_collisions link1="link_6" link2="soft_gripper_mount" reason="Never" />
+				<disable_collisions link1="link_7" link2="soft_gripper_link" reason="Never" />
+				<disable_collisions link1="link_7" link2="soft_gripper_mount" reason="Never" />
+				<disable_collisions link1="link_8" link2="soft_gripper_link" reason="Never" />
+				<disable_collisions link1="link_8" link2="soft_gripper_mount" reason="Never" />
+				<disable_collisions link1="camera_mount" link2="camera_link" reason="Adjacent" />
+				<disable_collisions link1="link_7" link2="camera_mount" reason="Adjacent" />
+				<disable_collisions link1="link_8" link2="camera_mount" reason="Adjacent" />
+				<disable_collisions link1="soft_gripper_mount" link2="soft_gripper_link"
+					reason="Adjacent" />
+			</xacro:if>
+			<xacro:if value="${camera == 'oakd' and end_effector == 'soft_gripper'}">
+				<disable_collisions link1="camera_link" link2="soft_gripper_mount" reason="Never" />
+				<disable_collisions link1="camera_link" link2="soft_gripper_link" reason="Never" />
+				<disable_collisions link1="camera_mount" link2="camera_link" reason="Adjacent" />
+				<disable_collisions link1="camera_mount" link2="soft_gripper_link" reason="Adjacent" />
+				<disable_collisions link1="camera_mount" link2="soft_gripper_mount" reason="Adjacent" />
+				<disable_collisions link1="link_2" link2="soft_gripper_link" reason="Never" />
+				<disable_collisions link1="link_2" link2="soft_gripper_mount" reason="Never" />
+				<disable_collisions link1="link_5" link2="camera_link" reason="Never" />
+				<disable_collisions link1="link_5" link2="camera_mount" reason="Never" />
+				<disable_collisions link1="link_5" link2="soft_gripper_link" reason="Never" />
+				<disable_collisions link1="link_5" link2="soft_gripper_mount" reason="Never" />
+				<disable_collisions link1="link_6" link2="camera_link" reason="Never" />
+				<disable_collisions link1="link_6" link2="camera_mount" reason="Never" />
+				<disable_collisions link1="link_6" link2="soft_gripper_link" reason="Never" />
+				<disable_collisions link1="link_6" link2="soft_gripper_mount" reason="Never" />
+				<disable_collisions link1="link_7" link2="camera_link" reason="Never" />
+				<disable_collisions link1="link_7" link2="camera_mount" reason="Never" />
+				<disable_collisions link1="link_7" link2="soft_gripper_link" reason="Never" />
+				<disable_collisions link1="link_7" link2="soft_gripper_mount" reason="Never" />
+				<disable_collisions link1="link_8" link2="camera_link" reason="Never" />
+				<disable_collisions link1="link_8" link2="camera_mount" reason="Adjacent" />
+				<disable_collisions link1="link_8" link2="soft_gripper_link" reason="Never" />
+				<disable_collisions link1="link_8" link2="soft_gripper_mount" reason="Never" />
+				<disable_collisions link1="soft_gripper_mount" link2="soft_gripper_link"
+					reason="Adjacent" />
 			</xacro:if>
 			<xacro:if value="${camera == 'realsense' and end_effector == 'soft_gripper'}">
